File: Welder PSU/Welder_PSU.brd (EAGLE design)
At the start: 382 x 220 mm, 216 parts, among them IC101 UCC28951PWR, IC102 UCC21542DWK, IC103 UCC21542DWK, IC104 UCC27524DGNVSS, IC105 MCP6001UT, IC106 UCC27524DGNVSS, IC107 MCP6001UT, IC108 MCP6001UT, IC201 NCP1014AP065G, IC202 AP63301WU-7, IC203 LD1117S33TR, IC204 LM317AEMP, J301 TE_282841-2TE_282841-2_0_0, J401 TE_282841-2TE_282841-2_0_0, K301 PANASONIC_ALFG2PF09PANASONIC_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, Q101 BSS123TA, Q201 PS2501L-1-ARENESAS_ELECTRONIC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, T101 SIHG039N60EF, T102 SIHG039N60EF, T103 SIHG039N60EF, T104 SIHG039N60EF, T105 SIHG039N60EF, T106 SIHG039N60EF, T107 SIHG039N60EF, T108 SIHG039N60EF, U201 TL431AQDBZR,215NEXPERIA_TL431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, X1 726386-2TE_726386-2, X103 726386-2TE_726386-2, X104 726386-2TE_726386-2, X2 726386-2TE_726386-2, X3 7461061, X4 7461061

Commit message: HW00.00
Layout finalization
Routing:
- net GND: vias 294 -> 371
Changed lines of the file:
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@@
 <setting verticaltext="up"/>
 </settings>
-<grid distance="25" unitdist="mil" unit="mil" style="lines" multiple="1" display="yes" altdistance="100" altunitdist="mil" altunit="mil"/>
+<grid distance="100" unitdist="mil" unit="mil" style="lines" multiple="1" display="yes" altdistance="100" altunitdist="mil" altunit="mil"/>
 <layers>
 <layer number="1" name="Top" color="4" fill="1" visible="yes" active="yes"/>
@@
 <via x="114.3" y="7.62" extent="1-16" drill="0.35"/>
 <via x="114.3" y="5.08" extent="1-16" drill="0.35"/>
-<via x="20.32" y="2.54" extent="1-16" drill="0.35"/>
-<via x="3.81" y="15.24" extent="1-16" drill="0.35"/>
+<via x="45.72" y="-5.08" extent="1-16" drill="0.35"/>
+<via x="5.08" y="15.24" extent="1-16" drill="0.35"/>
 <via x="50.8" y="45.72" extent="1-16" drill="0.35"/>
 <via x="76.2" y="50.8" extent="1-16" drill="0.35"/>
@@
 <wire x1="342.673675" y1="17.875" x2="344.82216875" y2="17.875" width="0.508" layer="1"/>
 <wire x1="344.82216875" y1="17.875" x2="348.44666875" y2="21.4995" width="0.508" layer="1"/>
+<via x="53.34" y="86.36" extent="1-16" drill="0.35"/>
+<via x="58.42" y="86.36" extent="1-16" drill="0.35"/>
+<via x="63.5" y="86.36" extent="1-16" drill="0.35"/>
+<via x="68.58" y="86.36" extent="1-16" drill="0.35"/>
+<via x="73.66" y="86.36" extent="1-16" drill="0.35"/>
+<via x="78.74" y="86.36" extent="1-16" drill="0.35"/>
+<via x="5.08" y="86.36" extent="1-16" drill="0.35"/>
+<via x="5.08" y="81.28" extent="1-16" drill="0.35"/>
+<via x="5.08" y="76.2" extent="1-16" drill="0.35"/>
+<via x="5.08" y="71.12" extent="1-16" drill="0.35"/>
+<via x="5.08" y="66.04" extent="1-16" drill="0.35"/>
+<via x="5.08" y="60.96" extent="1-16" drill="0.35"/>
+<via x="5.08" y="55.88" extent="1-16" drill="0.35"/>
+<via x="5.08" y="50.8" extent="1-16" drill="0.35"/>
+<via x="5.08" y="45.72" extent="1-16" drill="0.35"/>
+<via x="5.08" y="40.64" extent="1-16" drill="0.35"/>
+<via x="5.08" y="35.56" extent="1-16" drill="0.35"/>
+<via x="5.08" y="30.48" extent="1-16" drill="0.35"/>
+<via x="5.08" y="25.4" extent="1-16" drill="0.35"/>
+<via x="5.08" y="20.32" extent="1-16" drill="0.35"/>
+<via x="5.08" y="10.16" extent="1-16" drill="0.35"/>
+<via x="5.08" y="5.08" extent="1-16" drill="0.35"/>
+<via x="5.08" y="0" extent="1-16" drill="0.35"/>
+<via x="5.08" y="-5.08" extent="1-16" drill="0.35"/>
+<via x="10.16" y="-5.08" extent="1-16" drill="0.35"/>
+<via x="15.24" y="-5.08" extent="1-16" drill="0.35"/>
+<via x="20.32" y="-5.08" extent="1-16" drill="0.35"/>
+<via x="25.4" y="-5.08" extent="1-16" drill="0.35"/>
+<via x="30.48" y="-5.08" extent="1-16" drill="0.35"/>
+<via x="35.56" y="-5.08" extent="1-16" drill="0.35"/>
+<via x="40.64" y="-5.08" extent="1-16" drill="0.35"/>
+<via x="93.98" y="50.8" extent="1-16" drill="0.35"/>
+<via x="93.98" y="53.34" extent="1-16" drill="0.35"/>
+<via x="93.98" y="55.88" extent="1-16" drill="0.35"/>
+<via x="93.98" y="45.72" extent="1-16" drill="0.35"/>
+<via x="93.98" y="43.18" extent="1-16" drill="0.35"/>
+<via x="93.98" y="40.64" extent="1-16" drill="0.35"/>
+<via x="93.98" y="38.1" extent="1-16" drill="0.35"/>
+<via x="121.92" y="50.8" extent="1-16" drill="0.35"/>
+<via x="121.92" y="48.26" extent="1-16" drill="0.35"/>
+<via x="121.92" y="45.72" extent="1-16" drill="0.35"/>
+<via x="121.92" y="43.18" extent="1-16" drill="0.35"/>
+<via x="121.92" y="40.64" extent="1-16" drill="0.35"/>
+<via x="121.92" y="38.1" extent="1-16" drill="0.35"/>
+<via x="129.54" y="63.5" extent="1-16" drill="0.35"/>
+<via x="129.54" y="58.42" extent="1-16" drill="0.35"/>
+<via x="106.68" y="76.2" extent="1-16" drill="0.35"/>
+<via x="106.68" y="71.12" extent="1-16" drill="0.35"/>
+<via x="106.68" y="66.04" extent="1-16" drill="0.35"/>
+<via x="104.14" y="68.58" extent="1-16" drill="0.35"/>
+<via x="104.14" y="73.66" extent="1-16" drill="0.35"/>
+<via x="104.14" y="78.74" extent="1-16" drill="0.35"/>
+<via x="104.14" y="83.82" extent="1-16" drill="0.35"/>
+<via x="109.22" y="83.82" extent="1-16" drill="0.35"/>
+<via x="109.22" y="78.74" extent="1-16" drill="0.35"/>
+<via x="109.22" y="73.66" extent="1-16" drill="0.35"/>
+<via x="109.22" y="68.58" extent="1-16" drill="0.35"/>
+<via x="129.54" y="76.2" extent="1-16" drill="0.35"/>
+<via x="134.62" y="71.12" extent="1-16" drill="0.35"/>
+<via x="129.54" y="71.12" extent="1-16" drill="0.35"/>
+<via x="129.54" y="81.28" extent="1-16" drill="0.35"/>
+<via x="134.62" y="76.2" extent="1-16" drill="0.35"/>
+<via x="134.62" y="81.28" extent="1-16" drill="0.35"/>
+<via x="38.1" y="78.74" extent="1-16" drill="0.35"/>
+<via x="27.94" y="60.96" extent="1-16" drill="0.35"/>
+<via x="40.64" y="66.04" extent="1-16" drill="0.35"/>
+<via x="53.34" y="68.58" extent="1-16" drill="0.35"/>
+<via x="53.34" y="66.04" extent="1-16" drill="0.35"/>
+<via x="53.34" y="63.5" extent="1-16" drill="0.35"/>
+<via x="50.8" y="71.12" extent="1-16" drill="0.35"/>
+<via x="45.72" y="71.12" extent="1-16" drill="0.35"/>
+<via x="43.18" y="71.12" extent="1-16" drill="0.35"/>
+<via x="40.64" y="68.58" extent="1-16" drill="0.35"/>
+<via x="50.8" y="55.88" extent="1-16" drill="0.35"/>
+<via x="50.8" y="50.8" extent="1-16" drill="0.35"/>
+<via x="50.8" y="53.34" extent="1-16" drill="0.35"/>
+<via x="50.8" y="48.26" extent="1-16" drill="0.35"/>
 <wire x1="28.26" y1="53.975" x2="24.765" y2="53.61" width="0" layer="19" extent="1-1"/>
 <wire x1="115.33689375" y1="74.842" x2="119.611846875" y2="74.842" width="0" layer="19" extent="1-1"/>
