File: Callisto/Callisto_v1p0.brd (EAGLE design)
At the start: 100 x 105 mm, 101 parts, among them J1 4-pos, J10 20-pos, J11 2-pos, J12 USB-A, J15 4-pos, J2 2-pos, J3 2-pos, J4 20-pos, J5 10-pos, J6 2-pos, J7 2-pos, J8 2-pos, J9 10-pos, U3 AD8495ARMZ, U6 AD8495ARMZ

Commit message: Updated Board Design
Parts:
- removed J#1, J#3, J15: 4-pos, 3D_MIG_Controller:1X4_3.81MM_PITCH
- removed J#2, J#5: (no value), 3D_MIG_Controller:1X4_3.81MM_PITCH
- removed RXS10, RXS2, RXS4, RXS8, RYS11, RYS12, RYS3, RYS4, RYS5, RYS6, RYS7, RYS8, RZS2, RZS3, RZS4, RZS6, U$14, U$15, U$16, U$17, U$22, U$23, U$25, U$26, U$3, U$31, U$32, U$33, U$34, U$4, U$5, U$6: (no value), 3D_MIG_Controller:0402
- added 130, R120, R121, R131: 100, 3D_MIG_Controller:0402
- added R1, R10, R11, R12, R13, R14, R15, R16, R17, R18, R19, R2, R20, R21, R22, R23, R24, R25, R26, R27, R28, R29, R3, R30, R31, R32: (no value), 3D_MIG_Controller:0402
- added R122, R132: 1M, 3D_MIG_Controller:0402
- J1: value 4-pos -> RJ45_TH_VERT; device 3D_MIG_Controller:1X4_3.81MM_PITCH -> 3D_MIG_Controller:ASSMANN_A-2014-2S-4-N-R
- J10: value 20-pos -> 2-pos; device 3D_MIG_Controller:2_X_10_.1_INCH -> 3D_MIG_Controller:2_3.81MM_PITCH
- J11: value 2-pos -> 20-pos; device 3D_MIG_Controller:2_3.81MM_PITCH -> 3D_MIG_Controller:2_X_10_.1_INCH
- J12: value USB-A -> 10-pos; device 3D_MIG_Controller:USB_A_SMT -> 3D_MIG_Controller:2X5
- J2, J3: value 2-pos -> RJ45_TH_VERT; device 3D_MIG_Controller:2_3.81MM_PITCH -> 3D_MIG_Controller:ASSMANN_A-2014-2S-4-N-R
- J4: value 20-pos -> RJ45_TH_VERT; device 3D_MIG_Controller:2_X_10_.1_INCH -> 3D_MIG_Controller:ASSMANN_A-2014-2S-4-N-R
- J5, J9: value 10-pos -> 2-pos; device 3D_MIG_Controller:2X5 -> 3D_MIG_Controller:2_3.81MM_PITCH
- R4, R5, R7, R8: value 100 -> (none)
- R6, R9: value 1M -> (none)
- moved J12 131.3 mm to (147.5, 59.5), turned to 270 degrees
- moved R9 104.3 mm to (21.4, 10.8), turned to 0 degrees
- moved J11 101.3 mm to (93.6, 27.0), turned to 270 degrees
- moved R8 94.4 mm to (6.22, 35.2), turned to 90 degrees
- moved R7 89.9 mm to (7.96, 35.8)
- moved J5 86.5 mm to (24.5, 101.1), turned to 180 degrees
- moved R6 83.7 mm to (10.8, 35.2)
- moved J3 83.0 mm to (13.0, 50.0), turned to 0 degrees
- moved J2 81.9 mm to (35.0, 25.0), turned to 0 degrees
- moved R5 80.2 mm to (12.5, 35.8)
- moved R4 76.6 mm to (15.2, 35.2), turned to 90 degrees
- moved J4 66.3 mm to (35.0, 50.0), turned to 0 degrees
- moved U19 52.1 mm to (19.7, 12.6), turned to 0 degrees
- moved U20 47.2 mm to (15.2, 12.6), turned to 0 degrees
- moved U28 46.4 mm to (19.7, 37.6), turned to 0 degrees
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- renumbered RXS1 to R105, RXS3 to R103, RXS5 to R101, RXS6 to R107, U$10 to R102, U$12 to R100, U$24 to R106, U$8 to R104
Connections:
- removed net F0_IN: RXS10.P$1, RXS2.P$1, RXS4.P$1, RXS8.P$1
- removed net F0_OUT: J#1.P$1, J#2.P$1, J#3.P$1, J#5.P$1, U14.3, U19.3, U28.3, U4.3
- removed net F1_IN: RYS11.P$1, RYS3.P$1, RYS5.P$1, RYS7.P$1
- removed net F1_OUT: J#1.P$2, J#2.P$2, J#3.P$2, J#5.P$2, U15.3, U20.3, U29.3, U5.3
- removed net F2_IN: RZS2.P$1, RZS3.P$1, RZS4.P$1, RZS6.P$1
- removed net F2_OUT: J#1.P$3, J#2.P$3, J#3.P$3, J#5.P$3, U13.3, U18.3, U2.3, U27.3
- removed net F3_IN: RYS12.P$1, RYS4.P$1, RYS6.P$1, RYS8.P$1
- removed net F3_OUT: J#1.P$4, J#2.P$4, J#3.P$4, J#5.P$4, U16.3, U21.3, U30.3, U7.3
- removed net GNDE: J1.P$4
- removed net INT_AI_LS_0: J15.P$1
- removed net INT_AI_LS_1: J15.P$2
- removed net INT_AI_LS_2: J15.P$3
- removed net INT_AI_LS_3: J15.P$4
- removed net N$40: RYS12.P$2, U$34.P$1, U30.1
- removed net P0_02: J5.1
- removed net P0_03: J5.3
- removed net P0_04: J5.5
- removed net P0_05: J5.7
- removed net P0_06: J5.9
- removed net P0_07: J5.10
- removed net P0_08: J5.8
- removed net P0_09: J5.6
- removed net P0_14: J5.4
- removed net P0_15: J5.2
- removed net P2_00: J10.P$13
- removed net P2_01: J10.P$14
- removed net P2_02: J10.P$19
- removed net P3_03: J10.P$2
- removed net P3_04: J10.P$4
- removed net P3_05: J10.P$6
- removed net P3_06: J10.P$1
- removed net P3_07: J10.P$3
- removed net P3_09: J10.P$5
- removed net P3_10: J10.P$7
- removed net P3_11: J10.P$8
- removed net P3_12: J10.P$9
- removed net P3_13: J10.P$20
- removed net P3_14: J10.P$17
- removed net P3_15: J10.P$18
- removed net P4_02: J4.P$9
- removed net P4_08: J4.P$20
- removed net P4_09: J4.P$19
- removed net P4_10: J4.P$18
- removed net P4_11: J4.P$17
- removed net P4_12: J4.P$16
- removed net P4_13: J4.P$15
- removed net P4_14: J4.P$14
- removed net P4_15: J4.P$13
- removed net P9_00: J10.P$16
- removed net P9_01: J10.P$15
- removed net P9_05: J10.P$10
- removed net P9_06: J10.P$11
- removed net P9_07: J10.P$12
- removed net PB_00: J4.P$12
- removed net VBUS: J12.VBUS
- removed net VDDIN: J1.P$2
- removed net V_KT: U3.5, U3.6, U6.5, U6.6
- new net INT_AL_LS_0: J11.P$9
- new net INT_AL_LS_1: J11.P$20
- new net M0_DIR: J11.P$16, R9.P$1
- new net M0_DIR_IN: J1.2, U19.3
- new net M0_STEP: J11.P$12, R1.P$1
- new net M0_STEP_IN: J3.2, U28.3
- new net M1_DIR: J11.P$17, R11.P$1
- new net M1_DIR_IN: J1.4, U20.3
- new net M1_STEP: J11.P$13, R3.P$1
- new net M1_STEP_IN: J3.4, U29.3
- new net M2_DIR: J11.P$18, R13.P$1
- new net M2_DIR_IN: J1.6, U18.3
- new net M2_STEP: J11.P$14, R5.P$1
- new net M2_STEP_IN: J3.6, U27.3
- new net M3_DIR_1: J11.P$19, R15.P$1
- new net M3_DIR_IN: J1.8, U21.3
- new net M3_STEP: J11.P$15, R7.P$1
- new net M3_STEP_IN: J3.8, U30.3
- new net M4_DIR: R25.P$1
- new net M4_DIR_IN: J4.2, U14.3
- new net M4_STEP: R17.P$1
- new net M4_STEP_IN: J2.2, U4.3
- new net M5_DIR: R27.P$1
- new net M5_DIR_IN: J4.4, U15.3
- new net M5_STEP: R19.P$1
- new net M5_STEP_IN: J2.4, U5.3
- new net M6_DIR: R29.P$1
- new net M6_DIR_IN: J4.6, U13.3
- new net M6_STEP: R21.P$1
- new net M6_STEP_IN: J2.6, U2.3
- new net M7_DIR: R31.P$1
- new net M7_DIR_IN: J4.8, U16.3
- new net M7_STEP: R23.P$1
- new net M7_STEP_IN: J2.8, U7.3
- new net STEP_4: R7.P$2, R8.P$1, U30.1
- net GND: now also J12.10, J12.2, J12.4, J12.6, J12.8, R10.P$2, R12.P$2, R122.P$1, R132.P$1, R14.P$2, R16.P$2, R18.P$2, R2.P$2, R20.P$2, R22.P$2, R24.P$2, R26.P$2, R28.P$2, R30.P$2, R32.P$2, R4.P$2, R6.P$2, R8.P$2; no longer J1.P$1, J12.GND, J9.10, J9.2, J9.4, J9.6, J9.8, R6.P$1, R9.P$1, U$14.P$2, U$15.P$2, U$16.P$2, U$17.P$2, U$22.P$2, U$23.P$2, U$25.P$2, U$26.P$2, U$3.P$2, U$31.P$2, U$32.P$2, U$33.P$2, U$34.P$2, U$4.P$2, U$5.P$2, U$6.P$2
- net IN+: now also 130.P$2, R120.P$2; no longer R4.P$2, R7.P$2
- net IN-: now also R121.P$2, R131.P$2; no longer R5.P$2, R8.P$2
- net N$1: now also J8.P$2; no longer J6.P$2
- net N$12: now also R29.P$2, R30.P$1; no longer RZS4.P$2, U$14.P$1
- net N$13: now also R25.P$2, R26.P$1; no longer RXS4.P$2, U$15.P$1
- net N$14: now also R27.P$2, R28.P$1; no longer RYS7.P$2, U$16.P$1
- net N$15: now also R31.P$2, R32.P$1; no longer RYS8.P$2, U$17.P$1
- net N$17: now also J6.P$2; no longer J8.P$2
- net N$18: now also J6.P$1; no longer J8.P$1
- net N$2: now also R21.P$2, R22.P$1; no longer RZS2.P$2, U$3.P$1
- net N$21: now also J5.P$2; no longer J11.P$2
- net N$23: now also J5.P$1; no longer J11.P$1
- net N$29: now also R13.P$2, R14.P$1; no longer RZS3.P$2, U$22.P$1
- net N$3: now also R17.P$2, R18.P$1; no longer RXS2.P$2, U$4.P$1
- net N$30: now also R10.P$1, R9.P$2; no longer RXS8.P$2, U$23.P$1
- net N$31: now also R11.P$2, R12.P$1; no longer RYS5.P$2, U$25.P$1
- net N$32: now also R15.P$2, R16.P$1; no longer RYS6.P$2, U$26.P$1
- net N$37: now also R5.P$2, R6.P$1; no longer RZS6.P$2, U$31.P$1
- net N$38: now also R1.P$2, R2.P$1; no longer RXS10.P$2, U$32.P$1
- net N$39: now also R3.P$2, R4.P$1; no longer RYS11.P$2, U$33.P$1
- net N$4: now also J8.P$1; no longer J6.P$1
- net N$6: now also R19.P$2, R20.P$1; no longer RYS3.P$2, U$5.P$1
- net N$7: now also R23.P$2, R24.P$1; no longer RYS4.P$2, U$6.P$1
- net P0_00: now also J11.P$2, U6.5, U6.6; no longer J4.P$2
- net P0_01: now also J11.P$1, U3.5, U3.6; no longer J4.P$1
- net P2_03: now also J12.1; no longer J9.1
- net P2_04: now also J12.3; no longer J9.3
- net P2_05: now also J12.5; no longer J9.5
- net P2_06: now also J12.7; no longer J9.7
- net P2_07: now also J12.9; no longer J9.9
- net P4_00: now also J11.P$7; no longer J4.P$7
- net P4_01: now also J11.P$8; no longer J4.P$8
- net P5_11: now also J11.P$6; no longer J4.P$6
- net P5_12: now also J11.P$5; no longer J4.P$5
- net P5_13: now also J11.P$4; no longer J4.P$4
- net P7_06: now also J11.P$10; no longer J4.P$10
- net P7_07: now also J11.P$11; no longer J4.P$11
- net P8_05: now also J11.P$3; no longer J4.P$3
- net RED-: now also J10.P$1, J9.P$1, R121.P$1, R122.P$2, R131.P$1, R132.P$2; no longer J2.P$1, J3.P$1, R5.P$1, R6.P$2, R8.P$1, R9.P$2
- net VDD5: now also J1.1, J1.3, J1.5, J1.7, J2.1, J2.3, J2.5, J2.7, J3.1, J3.3, J3.5, J3.7, J4.1, J4.3, J4.5, J4.7; no longer J1.P$3
- net YLW+: now also 130.P$1, J10.P$2, J9.P$2, R120.P$1; no longer J2.P$2, J3.P$2, R4.P$1, R7.P$1
Routing:
- net M3_DIR_1: track 0.00 -> 86.6 mm, vias 0 -> 2
- net P0_01: track 0.00 -> 70.8 mm, vias 0 -> 1
- net P0_00: track 0.00 -> 61.4 mm, vias 0 -> 1
- net V_KT: track 4.52 -> 0.00 mm, vias 2 -> 0
- net N$11: track 0.00 -> 4.30 mm
- net F1_OUT: track 3.94 -> 0.00 mm
- net F3_OUT: track 3.94 -> 0.00 mm
- net F0_OUT: track 3.93 -> 0.00 mm
- net F2_OUT: track 3.92 -> 0.00 mm
- net N$24: track 0.00 -> 3.90 mm
- net N$19: track 0.00 -> 3.70 mm
- net N$8: track 0.00 -> 3.60 mm
- net N$40: track 3.28 -> 0.00 mm
- net N$20: track 0.00 -> 3.04 mm
- net N$16: track 0.00 -> 2.84 mm
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Other:
- board text removed: "#####"
- board text removed: "0"
- board text removed: "1"
- board text removed: "2"
- board text removed: "3"

Commit message: Updated.
Parts:
- removed J10, J5, J6, J7, J8, J9: 2-pos, 3D_MIG_Controller:2_3.81MM_PITCH
- removed J11: 20-pos, 3D_MIG_Controller:2_X_10_.1_INCH
- removed J4: RJ45_TH_VERT, 3D_MIG_Controller:ASSMANN_A-2014-2S-4-N-R
- removed R1, R10, R100, R101, R102, R103, R104, R105, R106, R107, R11, R12, R13, R14, R15, R16, R17, R18, R19, R2, R20, R21, R22, R23, R24, R25, R26, R27, R28, R29, R3, R30, R31, R32, R4, R5, R6, R7, R8, R9: (no value), 3D_MIG_Controller:0402
- removed U$11, U$13, U$7, U$9: RELAY_KYOTO_KF0604D, 3D_MIG_Controller:RELAY_KYOTO_KF0604D
- removed U1, U13, U14, U15, U16, U18, U19, U2, U20, U21, U24, U27, U28, U29, U30, U4, U5, U7, U8, U9: (no value), 3D_MIG_Controller:SOT323
- J1: value RJ45_TH_VERT -> 20-pos; device 3D_MIG_Controller:ASSMANN_A-2014-2S-4-N-R -> 3D_MIG_Controller:2_X_10_.1_INCH
- J2, J3: value RJ45_TH_VERT -> 2-pos; device 3D_MIG_Controller:ASSMANN_A-2014-2S-4-N-R -> 3D_MIG_Controller:2_3.81MM_PITCH
- moved J2 65.5 mm to (51.2, 88.5), turned to 180 degrees
- moved J3 45.9 mm to (38.1, 88.5), turned to 180 degrees
- moved J1 45.7 mm to (55.0, 43.0), turned to 270 degrees
- moved U$2 36.1 mm to (54.0, 2.00)
- moved C10 30.0 mm to (32.5, 78.6)
- moved R121 30.0 mm to (38.1, 83.6)
- moved U3 30.0 mm to (36.7, 79.3)
- moved 130 30.0 mm to (47.3, 83.6)
- moved C13 30.0 mm to (45.6, 83.1)
- moved C6 30.0 mm to (36.2, 83.7)
- moved C7 30.0 mm to (40.1, 83.0)
- moved C11 30.0 mm to (49.3, 83.6)
- moved C12 30.0 mm to (53.2, 82.9)
- moved C8 30.0 mm to (32.5, 83.2)
- moved C9 30.0 mm to (32.5, 79.6)
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Connections:
- removed net INT_AL_LS_0: J11.P$9
- removed net INT_AL_LS_1: J11.P$20
- removed net M0_DIR_IN: J1.2, U19.3
- removed net M0_STEP: J11.P$12, R1.P$1
- removed net M0_STEP_IN: J3.2, U28.3
- removed net M1_DIR_IN: J1.4, U20.3
- removed net M1_STEP: J11.P$13, R3.P$1
- removed net M1_STEP_IN: J3.4, U29.3
- removed net M2_DIR_IN: J1.6, U18.3
- removed net M2_STEP_IN: J3.6, U27.3
- removed net M3_DIR_IN: J1.8, U21.3
- removed net M3_STEP_IN: J3.8, U30.3
- removed net M4_DIR: R25.P$1
- removed net M4_DIR_IN: J4.2, U14.3
- removed net M4_STEP: R17.P$1
- removed net M4_STEP_IN: J2.2, U4.3
- removed net M5_DIR: R27.P$1
- removed net M5_DIR_IN: J4.4, U15.3
- removed net M5_STEP: R19.P$1
- removed net M5_STEP_IN: J2.4, U5.3
- removed net M6_DIR: R29.P$1
- removed net M6_DIR_IN: J4.6, U13.3
- removed net M6_STEP: R21.P$1
- removed net M6_STEP_IN: J2.6, U2.3
- removed net M7_DIR: R31.P$1
- removed net M7_DIR_IN: J4.8, U16.3
- removed net M7_STEP: R23.P$1
- removed net M7_STEP_IN: J2.8, U7.3
- removed net N$1: J8.P$2, U$7.P$3
- removed net N$10: J7.P$1, U$9.P$4
- removed net N$11: U$9.P$2, U1.3
- removed net N$12: R29.P$2, R30.P$1, U13.1
- removed net N$13: R25.P$2, R26.P$1, U14.1
- removed net N$14: R27.P$2, R28.P$1, U15.1
- removed net N$15: R31.P$2, R32.P$1, U16.1
- removed net N$16: R102.P$1, R103.P$2, U8.1
- removed net N$17: J6.P$2, U$11.P$3
- removed net N$18: J6.P$1, U$11.P$4
- removed net N$19: U$11.P$2, U8.3
- removed net N$20: R100.P$1, R101.P$2, U9.1
- removed net N$21: J5.P$2, U$13.P$3
- removed net N$22: R106.P$1, R107.P$2, U24.1
- removed net N$23: J5.P$1, U$13.P$4
- removed net N$24: U$13.P$2, U9.3
- removed net N$29: R13.P$2, R14.P$1, U18.1
- removed net N$30: R10.P$1, R9.P$2, U19.1
- removed net N$31: R11.P$2, R12.P$1, U20.1
- removed net N$32: R15.P$2, R16.P$1, U21.1
- removed net N$37: R5.P$2, R6.P$1, U27.1
- removed net N$38: R1.P$2, R2.P$1, U28.1
- removed net N$39: R3.P$2, R4.P$1, U29.1
- removed net N$4: J8.P$1, U$7.P$4
- removed net N$5: R104.P$1, R105.P$2, U1.1
- removed net N$6: R19.P$2, R20.P$1, U5.1
- removed net N$7: R23.P$2, R24.P$1, U7.1
- removed net N$8: U$7.P$2, U24.3
- removed net N$9: J7.P$2, U$9.P$3
- removed net P0_00: J11.P$2, U6.5, U6.6
- removed net P0_01: J11.P$1, U3.5, U3.6
- removed net P5_13: J11.P$4
- removed net P8_05: J11.P$3
- removed net RELAY_01: R107.P$1
- removed net RELAY_02: R105.P$1
- removed net RELAY_03: R103.P$1
- removed net RELAY_04: R101.P$1
- removed net STEP_4: R7.P$2, R8.P$1, U30.1
- removed net VDD5: J1.1, J1.3, J1.5, J1.7, J2.1, J2.3, J2.5, J2.7, J3.1, J3.3, J3.5, J3.7, J4.1, J4.3, J4.5, J4.7, U$11.P$1, U$13.P$1, U$7.P$1, U$9.P$1
- new net INT_00: J1.P$9
- new net IN_01: J1.P$20
- new net OUT_00: J1.P$4
- new net OUT_01: J1.P$3
- new net TC_0: J1.P$2, U6.5, U6.6
- new net TC_1: J1.P$1, U3.5, U3.6
- net GND: no longer R10.P$2, R100.P$2, R102.P$2, R104.P$2, R106.P$2, R12.P$2, R14.P$2, R16.P$2, R18.P$2, R2.P$2, R20.P$2, R22.P$2, R24.P$2, R26.P$2, R28.P$2, R30.P$2, R32.P$2, R4.P$2, R6.P$2, R8.P$2, U1.2, U13.2, U14.2, U15.2, U16.2, U18.2, U19.2, U2.2, U20.2, U21.2, U24.2, U27.2, U28.2, U29.2, U30.2, U4.2, U5.2, U7.2, U8.2, U9.2
- net M0_DIR: now also J1.P$16; no longer J11.P$16, R9.P$1
- net M1_DIR: now also J1.P$17; no longer J11.P$17, R11.P$1
- net M2_DIR: now also J1.P$18; no longer J11.P$18, R13.P$1
- net M2_STEP: now also J1.P$14; no longer J11.P$14, R5.P$1
- net M3_DIR_1: now also J1.P$19; no longer J11.P$19, R15.P$1
- net M3_STEP: now also J1.P$15; no longer J11.P$15, R7.P$1
- net N$2: now also J1.P$12; no longer R21.P$2, R22.P$1, U2.1
- net N$3: now also J1.P$13; no longer R17.P$2, R18.P$1, U4.1
- net P4_00: now also J1.P$7; no longer J11.P$7
- net P4_01: now also J1.P$8; no longer J11.P$8
- net P5_11: now also J1.P$6; no longer J11.P$6
- net P5_12: now also J1.P$5; no longer J11.P$5
- net P7_06: now also J1.P$10; no longer J11.P$10
- net P7_07: now also J1.P$11; no longer J11.P$11
- net RED-: now also J2.P$1, J3.P$1; no longer J10.P$1, J9.P$1
- net YLW+: now also J2.P$2, J3.P$2; no longer J10.P$2, J9.P$2
Routing:
- net M3_DIR_1: track 86.6 -> 0.00 mm, vias 2 -> 0
- net P0_01: track 70.8 -> 0.00 mm, vias 1 -> 0
- net P0_00: track 61.4 -> 0.00 mm, vias 1 -> 0
- net TC_1: track 0.00 -> 42.5 mm, vias 0 -> 1
- net TC_0: track 0.00 -> 30.8 mm, vias 0 -> 1
- net N$11: track 4.30 -> 0.00 mm
- net N$24: track 3.90 -> 0.00 mm
- net N$19: track 3.70 -> 0.00 mm
- net N$8: track 3.60 -> 0.00 mm
- net N$20: track 3.04 -> 0.00 mm
- net N$16: track 2.84 -> 0.00 mm
- net N$22: track 2.81 -> 0.00 mm
- net N$2: track 2.73 -> 0.00 mm
- net N$12: track 2.73 -> 0.00 mm
- net N$5: track 2.71 -> 0.00 mm
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Other:
- board size 100 x 105 mm -> 60 x 92.4 mm

Commit message: Updated Callisto.
Parts:
- added J10, J11, J13, J14, J15, J16, J17, J18, J19, J20, J21, J22, J23, J24, J25, J5, J6, J7, J8, J9: RJ45_TH_VERT, 3D_MIG_Controller:ASSMANN_A-2014-2S-4-N-R
- added J4: 4-pos, 3D_MIG_Controller:1X4_3.81MM_PITCH
- added R10, R13, R14, R17, R18, R21, R22, R25, R26, R33, R34, R37, R38, R5, R6, R9: 1K, 3D_MIG_Controller:0402
- added R11, R12, R15, R16, R19, R20, R23, R24, R27, R28, R35, R36, R39, R40, R7, R8: 10K, 3D_MIG_Controller:0402
- added U1, U10, U11, U12, U13, U14, U17, U18, U19, U2, U20, U4, U5, U7, U8, U9: (no value), 3D_MIG_Controller:SOT323
- moved J1 103.0 mm to (154.0, 71.4)
- moved 130 97.3 mm to (140.6, 111.1)
- moved C13 97.3 mm to (138.9, 110.6)
- moved C14 97.3 mm to (138.9, 107.0)
- moved C15 97.3 mm to (138.9, 106.0)
- moved C7 97.3 mm to (133.4, 110.5)
- moved J2 97.3 mm to (144.5, 116.0)
- moved J3 97.3 mm to (131.4, 116.0)
- moved R121 97.3 mm to (131.4, 111.1)
- moved R131 97.3 mm to (144.5, 111.0)
- moved U3 97.3 mm to (130.0, 106.8)
- moved U6 97.3 mm to (143.1, 106.7)
- moved C10 97.3 mm to (125.8, 106.1)
- moved C11 97.3 mm to (142.6, 111.1)
- moved C12 97.3 mm to (146.5, 110.4)
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Connections:
- removed net IN_01: J1.P$20
- removed net M0_DIR: J1.P$16
- removed net M1_DIR: J1.P$17
- removed net M2_DIR: J1.P$18
- removed net M2_STEP: J1.P$14
- removed net M3_DIR_1: J1.P$19
- removed net M3_STEP: J1.P$15
- removed net N$2: J1.P$12
- removed net N$3: J1.P$13
- removed net OUT_00: J1.P$4
- removed net OUT_01: J1.P$3
- new net INT_01: J1.P$20, J19.2
- new net IN_DIR_M_0: J5.4, U2.3
- new net IN_DIR_M_1: J7.4, U8.3
- new net IN_DIR_M_2: J9.4, U12.3
- new net IN_DIR_M_3: J6.4, U5.3
- new net IN_DIR_M_4: J10.4, U14.3
- new net IN_DIR_M_5: J13.4, U18.3
- new net IN_DIR_M_6: J8.4, U10.3
- new net IN_DIR_M_7: J14.4, U20.3
- new net IN_STEP_M_0: J5.2, U1.3
- new net IN_STEP_M_1: J7.2, U7.3
- new net IN_STEP_M_2: J9.2, U11.3
- new net IN_STEP_M_3: J6.2, U4.3
- new net IN_STEP_M_4: J10.2, U13.3
- new net IN_STEP_M_5: J13.2, U17.3
- new net IN_STEP_M_6: J8.2, U9.3
- new net IN_STEP_M_7: J14.2, U19.3
- new net IO_SIGNAL: J11.2, J15.2, J16.2, J17.2, J20.2, J21.2, J22.2, J23.2, J24.2, J25.2
- new net N$1: R5.P$2, R7.P$1, U1.1
- new net N$10: R18.P$2, R20.P$1, U10.1
- new net N$11: R21.P$2, R23.P$1, U11.1
- new net N$12: R22.P$2, R24.P$1, U12.1
- new net N$13: R25.P$2, R27.P$1, U13.1
- new net N$14: R26.P$2, R28.P$1, U14.1
- new net N$17: R33.P$2, R35.P$1, U17.1
- new net N$18: R34.P$2, R36.P$1, U18.1
- new net N$19: R37.P$2, R39.P$1, U19.1
- new net N$20: R38.P$2, R40.P$1, U20.1
- new net N$4: R6.P$2, R8.P$1, U2.1
- new net N$5: R11.P$1, R9.P$2, U4.1
- new net N$6: R10.P$2, R12.P$1, U5.1
- new net N$7: R13.P$2, R15.P$1, U7.1
- new net N$8: R14.P$2, R16.P$1, U8.1
- new net N$9: R17.P$2, R19.P$1, U9.1
- new net P4_09: J1.P$19, R26.P$1
- new net P4_10: J1.P$18, R25.P$1
- new net P4_11: J1.P$17, R34.P$1
- new net P4_12: J1.P$16, R33.P$1
- new net P4_13: J1.P$15, R18.P$1
- new net P4_14: J1.P$14, R17.P$1
- new net P4_15: J1.P$13, R38.P$1
- new net P5_13: J1.P$4, R6.P$1
- new net P8_05: J1.P$3, R5.P$1
- new net PB_00: J1.P$12, R37.P$1
- new net VDD: J10.5, J11.5, J13.5, J14.5, J15.5, J16.5, J17.5, J18.5, J19.5, J20.5, J21.5, J22.5, J23.5, J24.5, J25.5, J4.P$2, J5.5, J6.5, J7.5, J8.5, J9.5
- new net VDD-12: J10.7, J11.7, J13.7, J14.7, J15.7, J16.7, J17.7, J18.7, J19.7, J20.7, J21.7, J22.7, J23.7, J24.7, J25.7, J5.7, J6.7, J7.7, J8.7, J9.7
- new net VDD12: J10.3, J11.3, J13.3, J14.3, J15.3, J16.3, J17.3, J18.3, J19.3, J20.3, J21.3, J22.3, J23.3, J24.3, J25.3, J4.P$4, J5.3, J6.3, J7.3, J8.3, J9.3
- new net VDD5: J10.8, J11.8, J13.8, J14.8, J15.8, J16.8, J17.8, J18.8, J19.8, J20.8, J21.8, J22.8, J23.8, J24.8, J25.8, J4.P$3, J5.8, J6.8, J7.8, J8.8, J9.8
- net GND: now also J10.1, J10.6, J11.1, J11.4, J11.6, J13.1, J13.6, J14.1, J14.6, J15.1, J15.4, J15.6, J16.1, J16.4, J16.6, J17.1, J17.4, J17.6, J18.1, J18.4, J18.6, J19.1, J19.4, J19.6, J20.1, J20.4, J20.6, J21.1, J21.4, J21.6, J22.1, J22.4, J22.6, J23.1, J23.4, J23.6, J24.1, J24.4, J24.6, J25.1, J25.4, J25.6, J4.P$1, J5.1, J5.6, J6.1, J6.6, J7.1, J7.6, J8.1, J8.6, J9.1, J9.6, R11.P$2, R12.P$2, R15.P$2, R16.P$2, R19.P$2, R20.P$2, R23.P$2, R24.P$2, R27.P$2, R28.P$2, R35.P$2, R36.P$2, R39.P$2, R40.P$2, R7.P$2, R8.P$2, U1.2, U10.2, U11.2, U12.2, U13.2, U14.2, U17.2, U18.2, U19.2, U2.2, U20.2, U4.2, U5.2, U7.2, U8.2, U9.2
- net INT_00: now also J18.2
- net P4_00: now also R21.P$1
- net P4_01: now also R22.P$1
- net P5_11: now also R14.P$1
- net P5_12: now also R13.P$1
- net P7_06: now also R9.P$1
- net P7_07: now also R10.P$1
Routing:
- net VDD12: track 0.00 -> 874.1 mm, vias 0 -> 33
- net VDD5: track 0.00 -> 867.7 mm, vias 0 -> 7
- net VDD: track 0.00 -> 806.9 mm, vias 0 -> 33
- net P5_13: track 0.00 -> 147.9 mm, vias 0 -> 2
- net P4_09: track 0.00 -> 136.1 mm
- net P8_05: track 0.00 -> 135.3 mm, vias 0 -> 2
- net P4_10: track 0.00 -> 129.3 mm
- net P5_11: track 0.00 -> 124.3 mm, vias 0 -> 2
- net P4_11: track 0.00 -> 111.9 mm
- net P5_12: track 0.00 -> 111.6 mm, vias 0 -> 2
- net P4_12: track 0.00 -> 105.1 mm
- net P4_01: track 0.00 -> 100.5 mm, vias 0 -> 2
- net P4_00: track 0.00 -> 87.9 mm, vias 0 -> 2
- net P4_13: track 0.00 -> 87.6 mm
- net P4_14: track 0.00 -> 81.0 mm
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Other:
- board size 60 x 92.4 mm -> 160 x 120 mm

Commit message: Updated Board
Parts:
- removed J12: 10-pos, 3D_MIG_Controller:2X5
- removed J15, J16, J17, J20, J21, J22, J23, J24, J25: RJ45_TH_VERT, 3D_MIG_Controller:ASSMANN_A-2014-2S-4-N-R
- J11: value RJ45_TH_VERT -> 2-pos; device 3D_MIG_Controller:ASSMANN_A-2014-2S-4-N-R -> 3D_MIG_Controller:2_3.81MM_PITCH
- moved J18 89.7 mm to (28.3, 71.9)
- moved J19 87.4 mm to (53.8, 71.6)
- moved J4 78.5 mm to (41.2, 88.5)
- moved J3 65.5 mm to (72.0, 88.5)
- moved R121 65.5 mm to (72.0, 83.6)
- moved 130 65.5 mm to (81.2, 83.6)
- moved C12 65.5 mm to (87.1, 82.9)
- moved C13 65.5 mm to (79.5, 83.1)
- moved C14 65.5 mm to (79.5, 79.5)
- moved C15 65.5 mm to (79.5, 78.5)
- moved C6 65.5 mm to (70.1, 83.7)
- moved C7 65.5 mm to (74.0, 83.0)
- moved J2 65.5 mm to (85.1, 88.5)
- moved R131 65.5 mm to (85.1, 83.5)
- moved U3 65.5 mm to (70.6, 79.3)
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Connections:
- removed net IO_SIGNAL: J11.2, J15.2, J16.2, J17.2, J20.2, J21.2, J22.2, J23.2, J24.2, J25.2
- removed net P2_03: J12.1
- removed net P2_04: J12.3
- removed net P2_05: J12.5
- removed net P2_06: J12.7
- removed net P2_07: J12.9
- removed net VDD+: C10.P$1, C14.P$1, C15.P$1, C9.P$1, U3.7, U6.7
- net GND: now also J11.P$1; no longer J11.1, J11.4, J11.6, J12.10, J12.2, J12.4, J12.6, J12.8, J15.1, J15.4, J15.6, J16.1, J16.4, J16.6, J17.1, J17.4, J17.6, J20.1, J20.4, J20.6, J21.1, J21.4, J21.6, J22.1, J22.4, J22.6, J23.1, J23.4, J23.6, J24.1, J24.4, J24.6, J25.1, J25.4, J25.6
- net P4_09: now also R9.P$1; no longer R26.P$1
- net P4_10: now also R10.P$1; no longer R25.P$1
- net P4_11: now also R37.P$1; no longer R34.P$1
- net P4_12: now also R38.P$1; no longer R33.P$1
- net P4_13: now also R17.P$1; no longer R18.P$1
- net P4_14: now also R18.P$1; no longer R17.P$1
- net P4_15: now also R33.P$1; no longer R38.P$1
- net P7_06: now also R26.P$1; no longer R9.P$1
- net P7_07: now also R25.P$1; no longer R10.P$1
- net PB_00: now also R34.P$1; no longer R37.P$1
- net VDD: no longer J11.5, J15.5, J16.5, J17.5, J20.5, J21.5, J22.5, J23.5, J24.5, J25.5
- net VDD-12: now also J11.P$2; no longer J11.7, J15.7, J16.7, J17.7, J20.7, J21.7, J22.7, J23.7, J24.7, J25.7
- net VDD12: no longer J11.3, J15.3, J16.3, J17.3, J20.3, J21.3, J22.3, J23.3, J24.3, J25.3
- net VDD5: now also C10.P$1, C14.P$1, C15.P$1, C9.P$1, U3.7, U6.7; no longer J11.8, J15.8, J16.8, J17.8, J20.8, J21.8, J22.8, J23.8, J24.8, J25.8
Routing:
- net VDD12: track 874.1 -> 385.5 mm, vias 33 -> 14
- net VDD: track 806.9 -> 366.4 mm, vias 33 -> 14
- net VDD5: track 867.7 -> 445.8 mm, vias 7 -> 5
- net VDD-12: track 0.00 -> 350.9 mm, vias 0 -> 13
- net P4_09: track 136.1 -> 27.1 mm
- net P4_10: track 129.3 -> 40.9 mm
- net P7_06: track 61.1 -> 130.3 mm, vias 0 -> 2
- net PB_00: track 56.4 -> 106.3 mm, vias 0 -> 2
- net P7_07: track 69.3 -> 117.3 mm, vias 0 -> 2
- net P5_11: track 124.3 -> 84.6 mm
- net P5_12: track 111.6 -> 72.0 mm
- net P8_05: track 135.3 -> 100.4 mm
- net P4_11: track 111.9 -> 78.1 mm, vias 0 -> 2
- net P5_13: track 147.9 -> 114.2 mm
- net P4_15: track 63.2 -> 92.4 mm, vias 0 -> 2
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- added copper zone on layer 1, net GND
- added copper zone on layer 16, net GND
Other:
- board size 160 x 120 mm -> 105 x 92.4 mm

Commit message: Updated Callisto board.
Parts:
- moved J19 0.40 mm to (53.8, 72.0)
- moved J18 0.10 mm to (28.3, 72.0)
Routing:
- net VDD5: track 445.8 -> 498.0 mm, vias 5 -> 7
- net VDD12: track 385.5 -> 437.4 mm, vias 14 -> 17
- net VDD: track 366.4 -> 412.3 mm, vias 14 -> 17
- net VDD-12: track 350.9 -> 387.7 mm, vias 13 -> 15
- net INT_00: track 68.3 -> 77.5 mm, vias 0 -> 2
- net P5_13: track 114.2 -> 110.7 mm
- net P7_06: track 130.3 -> 127.7 mm
- net P7_07: track 117.3 -> 115.0 mm
- net P4_00: track 83.9 -> 85.9 mm
- net P8_05: track 100.4 -> 98.4 mm
- net P4_01: track 80.5 -> 82.2 mm
- net P5_12: track 72.0 -> 73.4 mm
- net P5_11: track 84.6 -> 85.7 mm

Commit message: Updated Callisto boards.
Parts:
- U1, U10, U11, U12, U13, U14, U17, U18, U19, U2, U20, U4, U5, U7, U8, U9: value (none) -> NPN
- moved J1 1.70 mm to (99.1, 66.0)
Routing:
- net P4_12: track 77.0 -> 79.2 mm
- net P4_00: track 85.9 -> 84.0 mm
- net P4_01: track 82.2 -> 80.4 mm
- net P5_12: track 73.4 -> 71.8 mm
- net P4_09: track 27.1 -> 28.7 mm
- net P4_11: track 78.1 -> 79.7 mm
- net PB_00: track 106.3 -> 104.8 mm
- net P5_11: track 85.7 -> 84.2 mm
- net P4_10: track 40.9 -> 42.1 mm
- net P8_05: track 98.4 -> 97.2 mm
- net P4_15: track 92.4 -> 91.2 mm
- net INT_00: track 77.5 -> 76.5 mm
- net TC_1: track 32.2 -> 33.1 mm
- net P4_13: track 69.9 -> 70.8 mm
- net P5_13: track 110.7 -> 109.8 mm
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