File: Callisto/Callisto_v1p0.brd (EAGLE design)
At the start: 105 x 92.4 mm, 83 parts, among them J1 20-pos, J10 RJ45_TH_VERT, J11 2-pos, J13 RJ45_TH_VERT, J14 RJ45_TH_VERT, J18 RJ45_TH_VERT, J19 RJ45_TH_VERT, J2 2-pos, J3 2-pos, J4 4-pos, J5 RJ45_TH_VERT, J6 RJ45_TH_VERT, J7 RJ45_TH_VERT, J8 RJ45_TH_VERT, J9 RJ45_TH_VERT, U1 NPN, U10 NPN, U11 NPN, U12 NPN, U13 NPN, U14 NPN, U17 NPN, U18 NPN, U19 NPN, U2 NPN, U20 NPN, U3 AD8495ARMZ, U4 NPN, U5 NPN, U6 AD8495ARMZ, U7 NPN, U8 NPN, U9 NPN

Commit message: Updated Callisto board
Parts:
- removed R11, R12, R15, R16, R19, R20, R23, R24, R27, R28, R35, R36, R39, R40, R7, R8: 10K, 3D_MIG_Controller:0402
- moved U14 103.7 mm to (100.6, 66.5), flipped to the top
- moved R26 98.7 mm to (97.6, 67.2), flipped to the top, turned to 90 degrees
- moved U2 95.2 mm to (100.6, 74.2), flipped to the top
- moved R6 89.6 mm to (97.6, 74.8), flipped to the top, turned to 90 degrees
- moved U13 83.5 mm to (85.1, 65.3), flipped to the top, turned to 90 degrees
- moved U18 83.3 mm to (100.6, 64.0), flipped to the top
- moved R25 82.6 mm to (88.2, 64.6), flipped to the top, turned to 270 degrees
- moved R34 79.1 mm to (97.6, 64.6), flipped to the top, turned to 90 degrees
- moved U1 74.3 mm to (85.1, 75.4), flipped to the top, turned to 90 degrees
- moved R5 73.5 mm to (88.2, 74.8), flipped to the top, turned to 270 degrees
- moved U8 73.1 mm to (100.6, 71.6), flipped to the top
- moved R14 68.0 mm to (97.6, 72.3), flipped to the top, turned to 90 degrees
- moved U17 66.2 mm to (85.1, 62.8), flipped to the top, turned to 90 degrees
- moved U10 65.7 mm to (100.6, 61.5), flipped to the top
- moved R33 65.3 mm to (88.2, 62.1), flipped to the top, turned to 270 degrees
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Connections:
- net GND: no longer R11.P$2, R12.P$2, R15.P$2, R16.P$2, R19.P$2, R20.P$2, R23.P$2, R24.P$2, R27.P$2, R28.P$2, R35.P$2, R36.P$2, R39.P$2, R40.P$2, R7.P$2, R8.P$2
- net N$1: no longer R7.P$1
- net N$10: no longer R20.P$1
- net N$11: no longer R23.P$1
- net N$12: no longer R24.P$1
- net N$13: no longer R27.P$1
- net N$14: no longer R28.P$1
- net N$17: no longer R35.P$1
- net N$18: no longer R36.P$1
- net N$19: no longer R39.P$1
- net N$20: no longer R40.P$1
- net N$4: no longer R8.P$1
- net N$5: no longer R11.P$1
- net N$6: no longer R12.P$1
- net N$7: no longer R15.P$1
- net N$8: no longer R16.P$1
- net N$9: no longer R19.P$1
Routing:
- net IN_DIR_M_4: track 8.85 -> 136.7 mm, vias 0 -> 3
- net P7_06: track 128.4 -> 2.83 mm, vias 2 -> 1
- net P7_07: track 115.5 -> 2.83 mm, vias 2 -> 1
- net IN_STEP_M_4: track 3.04 -> 112.8 mm, vias 0 -> 3
- net IN_DIR_M_1: track 8.85 -> 116.2 mm, vias 0 -> 3
- net P5_13: track 109.8 -> 2.82 mm, vias 2 -> 1
- net IN_DIR_M_0: track 8.85 -> 113.1 mm, vias 0 -> 1
- net IN_DIR_M_5: track 8.85 -> 112.8 mm, vias 0 -> 3
- net PB_00: track 104.8 -> 2.83 mm, vias 2 -> 1
- net P8_05: track 97.2 -> 2.81 mm, vias 2 -> 1
- net IN_STEP_M_1: track 3.04 -> 92.9 mm, vias 0 -> 1
- net P4_15: track 91.2 -> 2.82 mm, vias 2 -> 1
- net IN_STEP_M_5: track 3.04 -> 90.6 mm, vias 0 -> 3
- net IN_STEP_M_0: track 3.04 -> 90.4 mm, vias 0 -> 1
- net P5_11: track 84.2 -> 2.81 mm, vias 2 -> 1
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
Commit message: Updated Callisto
Parts:
- removed J18, J19: RJ45_TH_VERT, 3D_MIG_Controller:ASSMANN_A-2014-2S-4-N-R
- added J12, J15: RJ45_TH_VERT, 3D_MIG_Controller:ASSMANN_A-2014-2S-4-N-R
- J11: value 2-pos -> RJ45_TH_VERT; device 3D_MIG_Controller:2_3.81MM_PITCH -> 3D_MIG_Controller:ASSMANN_A-2014-2S-4-N-R
- J4: value 4-pos -> 2-pos; device 3D_MIG_Controller:1X4_3.81MM_PITCH -> 3D_MIG_Controller:2_3.81MM_PITCH
- J5: value RJ45_TH_VERT -> 4-pos; device 3D_MIG_Controller:ASSMANN_A-2014-2S-4-N-R -> 3D_MIG_Controller:1X4_3.81MM_PITCH
- moved J6 71.0 mm to (28.3, 72.0)
- moved J11 61.3 mm to (93.5, 43.4), turned to 0 degrees
- moved J8 54.2 mm to (20.9, 43.4)
- moved J10 53.9 mm to (69.1, 43.4)
- moved J5 49.5 mm to (41.2, 88.5), turned to 180 degrees
- moved J7 30.0 mm to (53.8, 72.0)
- moved J14 24.6 mm to (69.1, 18.8)
- moved J9 23.9 mm to (45.0, 43.4)
- moved J4 10.8 mm to (52.0, 88.5)
- moved J13 0.20 mm to (45.0, 18.8)
Connections:
- new net NC: J6.4, J7.4
- net GND: now also J11.1, J11.6, J12.1, J12.6, J15.1, J15.6, J5.P$1; no longer J11.P$1, J18.1, J18.4, J18.6, J19.1, J19.4, J19.6, J5.1, J5.6
- net INT_00: now also J6.2; no longer J18.2
- net INT_01: now also J7.2; no longer J19.2
- net IN_DIR_M_0: now also J8.4; no longer J5.4
- net IN_DIR_M_1: now also J9.4; no longer J7.4
- net IN_DIR_M_2: now also J10.4; no longer J9.4
- net IN_DIR_M_3: now also J11.4; no longer J6.4
- net IN_DIR_M_4: now also J12.4; no longer J10.4
- net IN_DIR_M_6: now also J14.4; no longer J8.4
- net IN_DIR_M_7: now also J15.4; no longer J14.4
- net IN_STEP_M_0: now also J8.2; no longer J5.2
- net IN_STEP_M_1: now also J9.2; no longer J7.2
- net IN_STEP_M_2: now also J10.2; no longer J9.2
- net IN_STEP_M_3: now also J11.2; no longer J6.2
- net IN_STEP_M_4: now also J12.2; no longer J10.2
- net IN_STEP_M_6: now also J14.2; no longer J8.2
- net IN_STEP_M_7: now also J15.2; no longer J14.2
- net VDD: now also J11.5, J12.5, J15.5, J5.P$2; no longer J18.5, J19.5, J4.P$2, J5.5
- net VDD-12: now also J11.7, J12.7, J15.7, J4.P$2; no longer J11.P$2, J18.7, J19.7, J5.7
- net VDD12: now also J11.3, J12.3, J15.3, J5.P$4; no longer J18.3, J19.3, J4.P$4, J5.3
- net VDD5: now also J11.8, J12.8, J15.8, J5.P$3; no longer J18.8, J19.8, J4.P$3, J5.8
Routing:
- net IN_DIR_M_6: track 88.8 -> 89.6 mm
- net IN_DIR_M_2: track 89.3 -> 90.0 mm
- net IN_DIR_M_7: track 89.3 -> 89.9 mm
- net IN_DIR_M_4: track 136.7 -> 137.3 mm
- net TC_0: track 15.4 -> 15.2 mm, vias 1 -> 0
- net IN_STEP_M_2: track 67.5 -> 67.6 mm, vias 2 -> 1
- net TC_1: vias 1 -> 0
Other:
- board text added: "+12V"
- board text added: "+3.3V"
- board text added: "+5V"
- board text added: "-12V"
- board text added: "Callisto J4"
- board text added: "GND"
- board text added: "Interrupt 0"
- board text added: "Interrupt 1"
- board text added: "RED-"
- board text added: "TC 1"
- board text added: "TC 2"
- board text added: "Type K"
- board text added: "YLW+"
- board text added: "vs 1p00"
