File: Callisto/Callisto_v1p0.sch (EAGLE design)
At the start: 101 parts, among them J1 4-pos, J10 20-pos, J11 2-pos, J12 USB-A, J15 4-pos, J2 2-pos, J3 2-pos, J4 20-pos, J5 10-pos, J6 2-pos, J7 2-pos, J8 2-pos, J9 10-pos, U3 AD8495ARMZ, U6 AD8495ARMZ

Commit message: Updated Board Design
Parts:
- removed J#1, J#3, J15: 4-pos, 3D_MIG_Controller:3.81MM_1_X_4_RT_ANGLE_PLUG_HEADER
- removed J#2, J#5: (no value), 3D_MIG_Controller:3.81MM_1_X_4_RT_ANGLE_PLUG_HEADER
- removed RXS2, RXS4, RXS8, RYS12, RYS3, RYS4, RYS5, RYS6, RYS7, RYS8, RZS2, RZS3, RZS4, RZS6, U$14, U$15, U$16, U$17, U$22, U$23, U$25, U$26, U$3, U$31, U$33, U$34, U$4, U$5, U$6: (no value), 3D_MIG_Controller:R_0402
- added 130, R120, R121, R131: 100, 3D_MIG_Controller:R_0402
- added R10, R11, R12, R13, R14, R15, R16, R17, R18, R19, R20, R21, R22, R23, R24, R25, R26, R27, R28, R29, R30, R31, R32: (no value), 3D_MIG_Controller:R_0402
- added R122, R132: 1M, 3D_MIG_Controller:R_0402
- J1: value 4-pos -> RJ45_TH_VERT; device 3D_MIG_Controller:3.81MM_1_X_4_RT_ANGLE_PLUG_HEADER -> 3D_MIG_Controller:RJ45_TH_VERT
- J10: value 20-pos -> 2-pos; device 3D_MIG_Controller:2_X_10_HEADER_GENERIC -> 3D_MIG_Controller:3.81MM_1_X_2_RT_ANGLE_PLUG_HEADER
- J11: value 2-pos -> 20-pos; device 3D_MIG_Controller:3.81MM_1_X_2_RT_ANGLE_PLUG_HEADER -> 3D_MIG_Controller:2_X_10_HEADER_GENERIC
- J12: value USB-A -> 10-pos; device 3D_MIG_Controller:USB_A -> 3D_MIG_Controller:CONN_05X2_RAPTH
- J2, J3: value 2-pos -> RJ45_TH_VERT; device 3D_MIG_Controller:3.81MM_1_X_2_RT_ANGLE_PLUG_HEADER -> 3D_MIG_Controller:RJ45_TH_VERT
- J4: value 20-pos -> RJ45_TH_VERT; device 3D_MIG_Controller:2_X_10_HEADER_GENERIC -> 3D_MIG_Controller:RJ45_TH_VERT
- J5, J9: value 10-pos -> 2-pos; device 3D_MIG_Controller:CONN_05X2_RAPTH -> 3D_MIG_Controller:3.81MM_1_X_2_RT_ANGLE_PLUG_HEADER
- R4, R5, R7, R8: value 100 -> (none)
- R6, R9: value 1M -> (none)
- renumbered RXS1 to R105, RXS10 to R1, RXS3 to R103, RXS5 to R101, RXS6 to R107, RYS11 to R3, U$10 to R102, U$12 to R100, U$24 to R106, U$32 to R2, U$8 to R104
Connections:
- removed net F0_IN: R1.1, RXS2.1, RXS4.1, RXS8.1
- removed net F0_OUT: J#1.P$1, J#2.P$1, J#3.P$1, J#5.P$1, U14.C(3), U19.C(3), U28.C(3), U4.C(3)
- removed net F1_IN: R3.1, RYS3.1, RYS5.1, RYS7.1
- removed net F1_OUT: J#1.P$2, J#2.P$2, J#3.P$2, J#5.P$2, U15.C(3), U20.C(3), U29.C(3), U5.C(3)
- removed net F2_IN: RZS2.1, RZS3.1, RZS4.1, RZS6.1
- removed net F2_OUT: J#1.P$3, J#2.P$3, J#3.P$3, J#5.P$3, U13.C(3), U18.C(3), U2.C(3), U27.C(3)
- removed net F3_IN: RYS12.1, RYS4.1, RYS6.1, RYS8.1
- removed net F3_OUT: J#1.P$4, J#2.P$4, J#3.P$4, J#5.P$4, U16.C(3), U21.C(3), U30.C(3), U7.C(3)
- removed net GNDE: J1.P$4
- removed net INT_AI_LS_0: J15.P$1
- removed net INT_AI_LS_1: J15.P$2
- removed net INT_AI_LS_2: J15.P$3
- removed net INT_AI_LS_3: J15.P$4
- removed net N$40: RYS12.2, U$34.1, U30.B(2)
- removed net P0_02: J5.1
- removed net P0_03: J5.3
- removed net P0_04: J5.5
- removed net P0_05: J5.7
- removed net P0_06: J5.9
- removed net P0_07: J5.10
- removed net P0_08: J5.8
- removed net P0_09: J5.6
- removed net P0_14: J5.4
- removed net P0_15: J5.2
- removed net P2_00: J10.P$13
- removed net P2_01: J10.P$14
- removed net P2_02: J10.P$19
- removed net P3_03: J10.P$2
- removed net P3_04: J10.P$4
- removed net P3_05: J10.P$6
- removed net P3_06: J10.P$1
- removed net P3_07: J10.P$3
- removed net P3_09: J10.P$5
- removed net P3_10: J10.P$7
- removed net P3_11: J10.P$8
- removed net P3_12: J10.P$9
- removed net P3_13: J10.P$20
- removed net P3_14: J10.P$17
- removed net P3_15: J10.P$18
- removed net P4_02: J4.P$9
- removed net P4_08: J4.P$20
- removed net P4_09: J4.P$19
- removed net P4_10: J4.P$18
- removed net P4_11: J4.P$17
- removed net P4_12: J4.P$16
- removed net P4_13: J4.P$15
- removed net P4_14: J4.P$14
- removed net P4_15: J4.P$13
- removed net P9_00: J10.P$16
- removed net P9_01: J10.P$15
- removed net P9_05: J10.P$10
- removed net P9_06: J10.P$11
- removed net P9_07: J10.P$12
- removed net PB_00: J4.P$12
- removed net VDDIN: J1.P$2
- removed net V_KT: U3.OUT, U3.SENSE, U6.OUT, U6.SENSE
- new net INT_AL_LS_0: J11.P$9
- new net INT_AL_LS_1: J11.P$20
- new net M0_DIR: J11.P$16, R9.1
- new net M0_DIR_IN: J1.2, U19.C(3)
- new net M0_STEP: J11.P$12, R1.1
- new net M0_STEP_IN: J3.2, U28.C(3)
- new net M1_DIR: J11.P$17, R11.1
- new net M1_DIR_IN: J1.4, U20.C(3)
- new net M1_STEP: J11.P$13, R3.1
- new net M1_STEP_IN: J3.4, U29.C(3)
- new net M2_DIR: J11.P$18, R13.1
- new net M2_DIR_IN: J1.6, U18.C(3)
- new net M2_STEP: J11.P$14, R5.1
- new net M2_STEP_IN: J3.6, U27.C(3)
- new net M3_DIR_1: J11.P$19, R15.1
- new net M3_DIR_IN: J1.8, U21.C(3)
- new net M3_STEP: J11.P$15, R7.1
- new net M3_STEP_IN: J3.8, U30.C(3)
- new net M4_DIR: R25.1
- new net M4_DIR_IN: J4.2, U14.C(3)
- new net M4_STEP: R17.1
- new net M4_STEP_IN: J2.2, U4.C(3)
- new net M5_DIR: R27.1
- new net M5_DIR_IN: J4.4, U15.C(3)
- new net M5_STEP: R19.1
- new net M5_STEP_IN: J2.4, U5.C(3)
- new net M6_DIR: R29.1
- new net M6_DIR_IN: J4.6, U13.C(3)
- new net M6_STEP: R21.1
- new net M6_STEP_IN: J2.6, U2.C(3)
- new net M7_DIR: R31.1
- new net M7_DIR_IN: J4.8, U16.C(3)
- new net M7_STEP: R23.1
- new net M7_STEP_IN: J2.8, U7.C(3)
- new net STEP_4: R7.2, R8.1, U30.B(2)
- net GND: now also J12.10, J12.2, J12.4, J12.6, J12.8, R10.2, R12.2, R122.1, R132.1, R14.2, R16.2, R18.2, R20.2, R22.2, R24.2, R26.2, R28.2, R30.2, R32.2, R4.2, R6.2, R8.2; no longer J1.P$1, J9.10, J9.2, J9.4, J9.6, J9.8, R6.1, R9.1, U$14.2, U$15.2, U$16.2, U$17.2, U$22.2, U$23.2, U$25.2, U$26.2, U$3.2, U$31.2, U$33.2, U$34.2, U$4.2, U$5.2, U$6.2
- net IN+: now also 130.2, R120.2; no longer R4.2, R7.2
- net IN-: now also R121.2, R131.2; no longer R5.2, R8.2
- net N$1: now also J8.P$2; no longer J6.P$2
- net N$12: now also R29.2, R30.1; no longer RZS4.2, U$14.1
- net N$13: now also R25.2, R26.1; no longer RXS4.2, U$15.1
- net N$14: now also R27.2, R28.1; no longer RYS7.2, U$16.1
- net N$15: now also R31.2, R32.1; no longer RYS8.2, U$17.1
- net N$17: now also J6.P$2; no longer J8.P$2
- net N$18: now also J6.P$1; no longer J8.P$1
- net N$2: now also R21.2, R22.1; no longer RZS2.2, U$3.1
- net N$21: now also J5.P$2; no longer J11.P$2
- net N$23: now also J5.P$1; no longer J11.P$1
- net N$29: now also R13.2, R14.1; no longer RZS3.2, U$22.1
- net N$3: now also R17.2, R18.1; no longer RXS2.2, U$4.1
- net N$30: now also R10.1, R9.2; no longer RXS8.2, U$23.1
- net N$31: now also R11.2, R12.1; no longer RYS5.2, U$25.1
- net N$32: now also R15.2, R16.1; no longer RYS6.2, U$26.1
- net N$37: now also R5.2, R6.1; no longer RZS6.2, U$31.1
- net N$39: now also R4.1; no longer U$33.1
- net N$4: now also J8.P$1; no longer J6.P$1
- net N$6: now also R19.2, R20.1; no longer RYS3.2, U$5.1
- net N$7: now also R23.2, R24.1; no longer RYS4.2, U$6.1
- net P0_00: now also J11.P$2, U6.OUT, U6.SENSE; no longer J4.P$2
- net P0_01: now also J11.P$1, U3.OUT, U3.SENSE; no longer J4.P$1
- net P2_03: now also J12.1; no longer J9.1
- net P2_04: now also J12.3; no longer J9.3
- net P2_05: now also J12.5; no longer J9.5
- net P2_06: now also J12.7; no longer J9.7
- net P2_07: now also J12.9; no longer J9.9
- net P4_00: now also J11.P$7; no longer J4.P$7
- net P4_01: now also J11.P$8; no longer J4.P$8
- net P5_11: now also J11.P$6; no longer J4.P$6
- net P5_12: now also J11.P$5; no longer J4.P$5
- net P5_13: now also J11.P$4; no longer J4.P$4
- net P7_06: now also J11.P$10; no longer J4.P$10
- net P7_07: now also J11.P$11; no longer J4.P$11
- net P8_05: now also J11.P$3; no longer J4.P$3
- net RED-: now also J10.P$1, J9.P$1, R121.1, R122.2, R131.1, R132.2; no longer J2.P$1, J3.P$1, R5.1, R6.2, R8.1, R9.2
- net VDD5: now also J1.1, J1.3, J1.5, J1.7, J2.1, J2.3, J2.5, J2.7, J3.1, J3.3, J3.5, J3.7, J4.1, J4.3, J4.5, J4.7; no longer J1.P$3
- net YLW+: now also 130.1, J10.P$2, J9.P$2, R120.1; no longer J2.P$2, J3.P$2, R4.1, R7.1

Commit message: Updated.
Parts:
- removed J10, J5, J6, J7, J8, J9: 2-pos, 3D_MIG_Controller:3.81MM_1_X_2_RT_ANGLE_PLUG_HEADER
- removed J11: 20-pos, 3D_MIG_Controller:2_X_10_HEADER_GENERIC
- removed J4: RJ45_TH_VERT, 3D_MIG_Controller:RJ45_TH_VERT
- removed R1, R10, R100, R101, R102, R103, R104, R105, R106, R107, R11, R12, R13, R14, R15, R16, R17, R18, R19, R2, R20, R21, R22, R23, R24, R25, R26, R27, R28, R29, R3, R30, R31, R32, R4, R5, R6, R7, R8, R9: (no value), 3D_MIG_Controller:R_0402
- removed U$11, U$13, U$7, U$9: RELAY_KYOTO_KF0604D, 3D_MIG_Controller:RELAY_KYOTO_KF0604D
- removed U1, U13, U14, U15, U16, U18, U19, U2, U20, U21, U24, U27, U28, U29, U30, U4, U5, U7, U8, U9: (no value), 3D_MIG_Controller:BC846BW
- J1: value RJ45_TH_VERT -> 20-pos; device 3D_MIG_Controller:RJ45_TH_VERT -> 3D_MIG_Controller:2_X_10_HEADER_GENERIC
- J2, J3: value RJ45_TH_VERT -> 2-pos; device 3D_MIG_Controller:RJ45_TH_VERT -> 3D_MIG_Controller:3.81MM_1_X_2_RT_ANGLE_PLUG_HEADER
Connections:
- removed net INT_AL_LS_0: J11.P$9
- removed net INT_AL_LS_1: J11.P$20
- removed net M0_DIR_IN: J1.2, U19.C(3)
- removed net M0_STEP: J11.P$12, R1.1
- removed net M0_STEP_IN: J3.2, U28.C(3)
- removed net M1_DIR_IN: J1.4, U20.C(3)
- removed net M1_STEP: J11.P$13, R3.1
- removed net M1_STEP_IN: J3.4, U29.C(3)
- removed net M2_DIR_IN: J1.6, U18.C(3)
- removed net M2_STEP_IN: J3.6, U27.C(3)
- removed net M3_DIR_IN: J1.8, U21.C(3)
- removed net M3_STEP_IN: J3.8, U30.C(3)
- removed net M4_DIR: R25.1
- removed net M4_DIR_IN: J4.2, U14.C(3)
- removed net M4_STEP: R17.1
- removed net M4_STEP_IN: J2.2, U4.C(3)
- removed net M5_DIR: R27.1
- removed net M5_DIR_IN: J4.4, U15.C(3)
- removed net M5_STEP: R19.1
- removed net M5_STEP_IN: J2.4, U5.C(3)
- removed net M6_DIR: R29.1
- removed net M6_DIR_IN: J4.6, U13.C(3)
- removed net M6_STEP: R21.1
- removed net M6_STEP_IN: J2.6, U2.C(3)
- removed net M7_DIR: R31.1
- removed net M7_DIR_IN: J4.8, U16.C(3)
- removed net M7_STEP: R23.1
- removed net M7_STEP_IN: J2.8, U7.C(3)
- removed net N$1: J8.P$2, U$7.VO+
- removed net N$10: J7.P$1, U$9.VO-
- removed net N$11: U$9.VC-, U1.C(3)
- removed net N$12: R29.2, R30.1, U13.B(2)
- removed net N$13: R25.2, R26.1, U14.B(2)
- removed net N$14: R27.2, R28.1, U15.B(2)
- removed net N$15: R31.2, R32.1, U16.B(2)
- removed net N$16: R102.1, R103.2, U8.B(2)
- removed net N$17: J6.P$2, U$11.VO+
- removed net N$18: J6.P$1, U$11.VO-
- removed net N$19: U$11.VC-, U8.C(3)
- removed net N$20: R100.1, R101.2, U9.B(2)
- removed net N$21: J5.P$2, U$13.VO+
- removed net N$22: R106.1, R107.2, U24.B(2)
- removed net N$23: J5.P$1, U$13.VO-
- removed net N$24: U$13.VC-, U9.C(3)
- removed net N$29: R13.2, R14.1, U18.B(2)
- removed net N$30: R10.1, R9.2, U19.B(2)
- removed net N$31: R11.2, R12.1, U20.B(2)
- removed net N$32: R15.2, R16.1, U21.B(2)
- removed net N$37: R5.2, R6.1, U27.B(2)
- removed net N$38: R1.2, R2.1, U28.B(2)
- removed net N$39: R3.2, R4.1, U29.B(2)
- removed net N$4: J8.P$1, U$7.VO-
- removed net N$5: R104.1, R105.2, U1.B(2)
- removed net N$6: R19.2, R20.1, U5.B(2)
- removed net N$7: R23.2, R24.1, U7.B(2)
- removed net N$8: U$7.VC-, U24.C(3)
- removed net N$9: J7.P$2, U$9.VO+
- removed net P0_00: J11.P$2, U6.OUT, U6.SENSE
- removed net P0_01: J11.P$1, U3.OUT, U3.SENSE
- removed net P5_13: J11.P$4
- removed net P8_05: J11.P$3
- removed net RELAY_01: R107.1
- removed net RELAY_02: R105.1
- removed net RELAY_03: R103.1
- removed net RELAY_04: R101.1
- removed net STEP_4: R7.2, R8.1, U30.B(2)
- removed net VDD5: J1.1, J1.3, J1.5, J1.7, J2.1, J2.3, J2.5, J2.7, J3.1, J3.3, J3.5, J3.7, J4.1, J4.3, J4.5, J4.7, U$11.VC+, U$13.VC+, U$7.VC+, U$9.VC+
- new net INT_00: J1.P$9
- new net IN_01: J1.P$20
- new net OUT_00: J1.P$4
- new net OUT_01: J1.P$3
- new net TC_0: J1.P$2, U6.OUT, U6.SENSE
- new net TC_1: J1.P$1, U3.OUT, U3.SENSE
- net GND: no longer R10.2, R100.2, R102.2, R104.2, R106.2, R12.2, R14.2, R16.2, R18.2, R2.2, R20.2, R22.2, R24.2, R26.2, R28.2, R30.2, R32.2, R4.2, R6.2, R8.2, U1.E(1), U13.E(1), U14.E(1), U15.E(1), U16.E(1), U18.E(1), U19.E(1), U2.E(1), U20.E(1), U21.E(1), U24.E(1), U27.E(1), U28.E(1), U29.E(1), U30.E(1), U4.E(1), U5.E(1), U7.E(1), U8.E(1), U9.E(1)
- net M0_DIR: now also J1.P$16; no longer J11.P$16, R9.1
- net M1_DIR: now also J1.P$17; no longer J11.P$17, R11.1
- net M2_DIR: now also J1.P$18; no longer J11.P$18, R13.1
- net M2_STEP: now also J1.P$14; no longer J11.P$14, R5.1
- net M3_DIR_1: now also J1.P$19; no longer J11.P$19, R15.1
- net M3_STEP: now also J1.P$15; no longer J11.P$15, R7.1
- net N$2: now also J1.P$12; no longer R21.2, R22.1, U2.B(2)
- net N$3: now also J1.P$13; no longer R17.2, R18.1, U4.B(2)
- net P4_00: now also J1.P$7; no longer J11.P$7
- net P4_01: now also J1.P$8; no longer J11.P$8
- net P5_11: now also J1.P$6; no longer J11.P$6
- net P5_12: now also J1.P$5; no longer J11.P$5
- net P7_06: now also J1.P$10; no longer J11.P$10
- net P7_07: now also J1.P$11; no longer J11.P$11
- net RED-: now also J2.P$1, J3.P$1; no longer J10.P$1, J9.P$1
- net YLW+: now also J2.P$2, J3.P$2; no longer J10.P$2, J9.P$2

Commit message: Updated Callisto.
Parts:
- added J10, J11, J13, J14, J15, J16, J17, J18, J19, J20, J21, J22, J23, J24, J25, J5, J6, J7, J8, J9: RJ45_TH_VERT, 3D_MIG_Controller:RJ45_TH_VERT
- added J4: 4-pos, 3D_MIG_Controller:3.81MM_1_X_4_RT_ANGLE_PLUG_HEADER
- added R10, R13, R14, R17, R18, R21, R22, R25, R26, R33, R34, R37, R38, R5, R6, R9: 1K, 3D_MIG_Controller:R_0402
- added R11, R12, R15, R16, R19, R20, R23, R24, R27, R28, R35, R36, R39, R40, R7, R8: 10K, 3D_MIG_Controller:R_0402
- added U1, U10, U11, U12, U13, U14, U17, U18, U19, U2, U20, U4, U5, U7, U8, U9: (no value), 3D_MIG_Controller:BC846BW
Connections:
- removed net IN_01: J1.P$20
- removed net M0_DIR: J1.P$16
- removed net M1_DIR: J1.P$17
- removed net M2_DIR: J1.P$18
- removed net M2_STEP: J1.P$14
- removed net M3_DIR_1: J1.P$19
- removed net M3_STEP: J1.P$15
- removed net N$2: J1.P$12
- removed net N$3: J1.P$13
- removed net OUT_00: J1.P$4
- removed net OUT_01: J1.P$3
- new net INT_01: J1.P$20, J19.2
- new net IN_DIR_M_0: J5.4, U2.C(3)
- new net IN_DIR_M_1: J7.4, U8.C(3)
- new net IN_DIR_M_2: J9.4, U12.C(3)
- new net IN_DIR_M_3: J6.4, U5.C(3)
- new net IN_DIR_M_4: J10.4, U14.C(3)
- new net IN_DIR_M_5: J13.4, U18.C(3)
- new net IN_DIR_M_6: J8.4, U10.C(3)
- new net IN_DIR_M_7: J14.4, U20.C(3)
- new net IN_STEP_M_0: J5.2, U1.C(3)
- new net IN_STEP_M_1: J7.2, U7.C(3)
- new net IN_STEP_M_2: J9.2, U11.C(3)
- new net IN_STEP_M_3: J6.2, U4.C(3)
- new net IN_STEP_M_4: J10.2, U13.C(3)
- new net IN_STEP_M_5: J13.2, U17.C(3)
- new net IN_STEP_M_6: J8.2, U9.C(3)
- new net IN_STEP_M_7: J14.2, U19.C(3)
- new net IO_SIGNAL: J11.2, J15.2, J16.2, J17.2, J20.2, J21.2, J22.2, J23.2, J24.2, J25.2
- new net N$1: R5.2, R7.1, U1.B(2)
- new net N$10: R18.2, R20.1, U10.B(2)
- new net N$11: R21.2, R23.1, U11.B(2)
- new net N$12: R22.2, R24.1, U12.B(2)
- new net N$13: R25.2, R27.1, U13.B(2)
- new net N$14: R26.2, R28.1, U14.B(2)
- new net N$17: R33.2, R35.1, U17.B(2)
- new net N$18: R34.2, R36.1, U18.B(2)
- new net N$19: R37.2, R39.1, U19.B(2)
- new net N$20: R38.2, R40.1, U20.B(2)
- new net N$4: R6.2, R8.1, U2.B(2)
- new net N$5: R11.1, R9.2, U4.B(2)
- new net N$6: R10.2, R12.1, U5.B(2)
- new net N$7: R13.2, R15.1, U7.B(2)
- new net N$8: R14.2, R16.1, U8.B(2)
- new net N$9: R17.2, R19.1, U9.B(2)
- new net P4_09: J1.P$19, R26.1
- new net P4_10: J1.P$18, R25.1
- new net P4_11: J1.P$17, R34.1
- new net P4_12: J1.P$16, R33.1
- new net P4_13: J1.P$15, R18.1
- new net P4_14: J1.P$14, R17.1
- new net P4_15: J1.P$13, R38.1
- new net P5_13: J1.P$4, R6.1
- new net P8_05: J1.P$3, R5.1
- new net PB_00: J1.P$12, R37.1
- new net VDD: J10.5, J11.5, J13.5, J14.5, J15.5, J16.5, J17.5, J18.5, J19.5, J20.5, J21.5, J22.5, J23.5, J24.5, J25.5, J4.P$2, J5.5, J6.5, J7.5, J8.5, J9.5
- new net VDD-12: J10.7, J11.7, J13.7, J14.7, J15.7, J16.7, J17.7, J18.7, J19.7, J20.7, J21.7, J22.7, J23.7, J24.7, J25.7, J5.7, J6.7, J7.7, J8.7, J9.7
- new net VDD12: J10.3, J11.3, J13.3, J14.3, J15.3, J16.3, J17.3, J18.3, J19.3, J20.3, J21.3, J22.3, J23.3, J24.3, J25.3, J4.P$4, J5.3, J6.3, J7.3, J8.3, J9.3
- new net VDD5: J10.8, J11.8, J13.8, J14.8, J15.8, J16.8, J17.8, J18.8, J19.8, J20.8, J21.8, J22.8, J23.8, J24.8, J25.8, J4.P$3, J5.8, J6.8, J7.8, J8.8, J9.8
- net GND: now also J10.1, J10.6, J11.1, J11.4, J11.6, J13.1, J13.6, J14.1, J14.6, J15.1, J15.4, J15.6, J16.1, J16.4, J16.6, J17.1, J17.4, J17.6, J18.1, J18.4, J18.6, J19.1, J19.4, J19.6, J20.1, J20.4, J20.6, J21.1, J21.4, J21.6, J22.1, J22.4, J22.6, J23.1, J23.4, J23.6, J24.1, J24.4, J24.6, J25.1, J25.4, J25.6, J4.P$1, J5.1, J5.6, J6.1, J6.6, J7.1, J7.6, J8.1, J8.6, J9.1, J9.6, R11.2, R12.2, R15.2, R16.2, R19.2, R20.2, R23.2, R24.2, R27.2, R28.2, R35.2, R36.2, R39.2, R40.2, R7.2, R8.2, U1.E(1), U10.E(1), U11.E(1), U12.E(1), U13.E(1), U14.E(1), U17.E(1), U18.E(1), U19.E(1), U2.E(1), U20.E(1), U4.E(1), U5.E(1), U7.E(1), U8.E(1), U9.E(1)
- net INT_00: now also J18.2
- net P4_00: now also R21.1
- net P4_01: now also R22.1
- net P5_11: now also R14.1
- net P5_12: now also R13.1
- net P7_06: now also R9.1
- net P7_07: now also R10.1

Commit message: Updated Board
Parts:
- removed J12: 10-pos, 3D_MIG_Controller:CONN_05X2_RAPTH
- removed J15, J16, J17, J20, J21, J22, J23, J24, J25: RJ45_TH_VERT, 3D_MIG_Controller:RJ45_TH_VERT
- J11: value RJ45_TH_VERT -> 2-pos; device 3D_MIG_Controller:RJ45_TH_VERT -> 3D_MIG_Controller:3.81MM_1_X_2_RT_ANGLE_PLUG_HEADER
Connections:
- removed net IO_SIGNAL: J11.2, J15.2, J16.2, J17.2, J20.2, J21.2, J22.2, J23.2, J24.2, J25.2
- removed net P2_03: J12.1
- removed net P2_04: J12.3
- removed net P2_05: J12.5
- removed net P2_06: J12.7
- removed net P2_07: J12.9
- removed net VDD+: C10.1, C14.1, C15.1, C9.1, U3.+VS, U6.+VS
- net GND: now also J11.P$1; no longer J11.1, J11.4, J11.6, J12.10, J12.2, J12.4, J12.6, J12.8, J15.1, J15.4, J15.6, J16.1, J16.4, J16.6, J17.1, J17.4, J17.6, J20.1, J20.4, J20.6, J21.1, J21.4, J21.6, J22.1, J22.4, J22.6, J23.1, J23.4, J23.6, J24.1, J24.4, J24.6, J25.1, J25.4, J25.6
- net P4_09: now also R9.1; no longer R26.1
- net P4_10: now also R10.1; no longer R25.1
- net P4_11: now also R37.1; no longer R34.1
- net P4_12: now also R38.1; no longer R33.1
- net P4_13: now also R17.1; no longer R18.1
- net P4_14: now also R18.1; no longer R17.1
- net P4_15: now also R33.1; no longer R38.1
- net P7_06: now also R26.1; no longer R9.1
- net P7_07: now also R25.1; no longer R10.1
- net PB_00: now also R34.1; no longer R37.1
- net VDD: no longer J11.5, J15.5, J16.5, J17.5, J20.5, J21.5, J22.5, J23.5, J24.5, J25.5
- net VDD-12: now also J11.P$2; no longer J11.7, J15.7, J16.7, J17.7, J20.7, J21.7, J22.7, J23.7, J24.7, J25.7
- net VDD12: no longer J11.3, J15.3, J16.3, J17.3, J20.3, J21.3, J22.3, J23.3, J24.3, J25.3
- net VDD5: now also C10.1, C14.1, C15.1, C9.1, U3.+VS, U6.+VS; no longer J11.8, J15.8, J16.8, J17.8, J20.8, J21.8, J22.8, J23.8, J24.8, J25.8

Commit message: Updated Callisto boards.
Parts:
- U1, U10, U11, U12, U13, U14, U17, U18, U19, U2, U20, U4, U5, U7, U8, U9: value (none) -> NPN
Changed lines of the file:
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@@
 <part name="R7" library="3D_MIG_Controller" deviceset="R_0402" device="" value="10K"/>
 <part name="R8" library="3D_MIG_Controller" deviceset="R_0402" device="" value="10K"/>
-<part name="U1" library="3D_MIG_Controller" deviceset="BC846BW" device=""/>
-<part name="U2" library="3D_MIG_Controller" deviceset="BC846BW" device=""/>
+<part name="U1" library="3D_MIG_Controller" deviceset="BC846BW" device="" value="NPN"/>
+<part name="U2" library="3D_MIG_Controller" deviceset="BC846BW" device="" value="NPN"/>
 <part name="J5" library="3D_MIG_Controller" deviceset="RJ45_TH_VERT" device=""/>
 <part name="R13" library="3D_MIG_Controller" deviceset="R_0402" device="" value="1K"/>
@@
 <part name="R15" library="3D_MIG_Controller" deviceset="R_0402" device="" value="10K"/>
 <part name="R16" library="3D_MIG_Controller" deviceset="R_0402" device="" value="10K"/>
-<part name="U7" library="3D_MIG_Controller" deviceset="BC846BW" device=""/>
-<part name="U8" library="3D_MIG_Controller" deviceset="BC846BW" device=""/>
+<part name="U7" library="3D_MIG_Controller" deviceset="BC846BW" device="" value="NPN"/>
+<part name="U8" library="3D_MIG_Controller" deviceset="BC846BW" device="" value="NPN"/>
 <part name="J7" library="3D_MIG_Controller" deviceset="RJ45_TH_VERT" device=""/>
 <part name="R21" library="3D_MIG_Controller" deviceset="R_0402" device="" value="1K"/>
@@
 <part name="R23" library="3D_MIG_Controller" deviceset="R_0402" device="" value="10K"/>
 <part name="R24" library="3D_MIG_Controller" deviceset="R_0402" device="" value="10K"/>
-<part name="U11" library="3D_MIG_Controller" deviceset="BC846BW" device=""/>
-<part name="U12" library="3D_MIG_Controller" deviceset="BC846BW" device=""/>
+<part name="U11" library="3D_MIG_Controller" deviceset="BC846BW" device="" value="NPN"/>
+<part name="U12" library="3D_MIG_Controller" deviceset="BC846BW" device="" value="NPN"/>
 <part name="J9" library="3D_MIG_Controller" deviceset="RJ45_TH_VERT" device=""/>
 <part name="R9" library="3D_MIG_Controller" deviceset="R_0402" device="" value="1K"/>
@@
 <part name="R11" library="3D_MIG_Controller" deviceset="R_0402" device="" value="10K"/>
 <part name="R12" library="3D_MIG_Controller" deviceset="R_0402" device="" value="10K"/>
-<part name="U4" library="3D_MIG_Controller" deviceset="BC846BW" device=""/>
-<part name="U5" library="3D_MIG_Controller" deviceset="BC846BW" device=""/>
+<part name="U4" library="3D_MIG_Controller" deviceset="BC846BW" device="" value="NPN"/>
+<part name="U5" library="3D_MIG_Controller" deviceset="BC846BW" device="" value="NPN"/>
 <part name="J6" library="3D_MIG_Controller" deviceset="RJ45_TH_VERT" device=""/>
 <part name="R25" library="3D_MIG_Controller" deviceset="R_0402" device="" value="1K"/>
@@
 <part name="R27" library="3D_MIG_Controller" deviceset="R_0402" device="" value="10K"/>
 <part name="R28" library="3D_MIG_Controller" deviceset="R_0402" device="" value="10K"/>
-<part name="U13" library="3D_MIG_Controller" deviceset="BC846BW" device=""/>
-<part name="U14" library="3D_MIG_Controller" deviceset="BC846BW" device=""/>
+<part name="U13" library="3D_MIG_Controller" deviceset="BC846BW" device="" value="NPN"/>
+<part name="U14" library="3D_MIG_Controller" deviceset="BC846BW" device="" value="NPN"/>
 <part name="J10" library="3D_MIG_Controller" deviceset="RJ45_TH_VERT" device=""/>
 <part name="R33" library="3D_MIG_Controller" deviceset="R_0402" device="" value="1K"/>
@@
 <part name="R35" library="3D_MIG_Controller" deviceset="R_0402" device="" value="10K"/>
 <part name="R36" library="3D_MIG_Controller" deviceset="R_0402" device="" value="10K"/>
-<part name="U17" library="3D_MIG_Controller" deviceset="BC846BW" device=""/>
-<part name="U18" library="3D_MIG_Controller" deviceset="BC846BW" device=""/>
+<part name="U17" library="3D_MIG_Controller" deviceset="BC846BW" device="" value="NPN"/>
+<part name="U18" library="3D_MIG_Controller" deviceset="BC846BW" device="" value="NPN"/>
 <part name="J13" library="3D_MIG_Controller" deviceset="RJ45_TH_VERT" device=""/>
 <part name="R17" library="3D_MIG_Controller" deviceset="R_0402" device="" value="1K"/>
@@
 <part name="R19" library="3D_MIG_Controller" deviceset="R_0402" device="" value="10K"/>
 <part name="R20" library="3D_MIG_Controller" deviceset="R_0402" device="" value="10K"/>
-<part name="U9" library="3D_MIG_Controller" deviceset="BC846BW" device=""/>
-<part name="U10" library="3D_MIG_Controller" deviceset="BC846BW" device=""/>
+<part name="U9" library="3D_MIG_Controller" deviceset="BC846BW" device="" value="NPN"/>
+<part name="U10" library="3D_MIG_Controller" deviceset="BC846BW" device="" value="NPN"/>
 <part name="J8" library="3D_MIG_Controller" deviceset="RJ45_TH_VERT" device=""/>
 <part name="R37" library="3D_MIG_Controller" deviceset="R_0402" device="" value="1K"/>
@@
 <part name="R39" library="3D_MIG_Controller" deviceset="R_0402" device="" value="10K"/>
 <part name="R40" library="3D_MIG_Controller" deviceset="R_0402" device="" value="10K"/>
-<part name="U19" library="3D_MIG_Controller" deviceset="BC846BW" device=""/>
-<part name="U20" library="3D_MIG_Controller" deviceset="BC846BW" device=""/>
+<part name="U19" library="3D_MIG_Controller" deviceset="BC846BW" device="" value="NPN"/>
+<part name="U20" library="3D_MIG_Controller" deviceset="BC846BW" device="" value="NPN"/>
 <part name="J14" library="3D_MIG_Controller" deviceset="RJ45_TH_VERT" device=""/>
 <part name="J18" library="3D_MIG_Controller" deviceset="RJ45_TH_VERT" device=""/>

Commit message: Updated Callisto board
Parts:
- removed R11, R12, R15, R16, R19, R20, R23, R24, R27, R28, R35, R36, R39, R40, R7, R8: 10K, 3D_MIG_Controller:R_0402
Connections:
- net GND: no longer R11.2, R12.2, R15.2, R16.2, R19.2, R20.2, R23.2, R24.2, R27.2, R28.2, R35.2, R36.2, R39.2, R40.2, R7.2, R8.2
- net N$1: no longer R7.1
- net N$10: no longer R20.1
- net N$11: no longer R23.1
- net N$12: no longer R24.1
- net N$13: no longer R27.1
- net N$14: no longer R28.1
- net N$17: no longer R35.1
- net N$18: no longer R36.1
- net N$19: no longer R39.1
- net N$20: no longer R40.1
- net N$4: no longer R8.1
- net N$5: no longer R11.1
- net N$6: no longer R12.1
- net N$7: no longer R15.1
- net N$8: no longer R16.1
- net N$9: no longer R19.1
