File: Callisto/Callisto_v1p0.sch (EAGLE design)
At the start: 67 parts, among them J1 20-pos, J10 RJ45_TH_VERT, J11 2-pos, J13 RJ45_TH_VERT, J14 RJ45_TH_VERT, J18 RJ45_TH_VERT, J19 RJ45_TH_VERT, J2 2-pos, J3 2-pos, J4 4-pos, J5 RJ45_TH_VERT, J6 RJ45_TH_VERT, J7 RJ45_TH_VERT, J8 RJ45_TH_VERT, J9 RJ45_TH_VERT, U1 NPN, U10 NPN, U11 NPN, U12 NPN, U13 NPN, U14 NPN, U17 NPN, U18 NPN, U19 NPN, U2 NPN, U20 NPN, U3 AD8495ARMZ, U4 NPN, U5 NPN, U6 AD8495ARMZ, U7 NPN, U8 NPN, U9 NPN

Commit message: Updated Callisto
Parts:
- removed J18, J19: RJ45_TH_VERT, 3D_MIG_Controller:RJ45_TH_VERT
- added J12, J15: RJ45_TH_VERT, 3D_MIG_Controller:RJ45_TH_VERT
- J11: value 2-pos -> RJ45_TH_VERT; device 3D_MIG_Controller:3.81MM_1_X_2_RT_ANGLE_PLUG_HEADER -> 3D_MIG_Controller:RJ45_TH_VERT
- J4: value 4-pos -> 2-pos; device 3D_MIG_Controller:3.81MM_1_X_4_RT_ANGLE_PLUG_HEADER -> 3D_MIG_Controller:3.81MM_1_X_2_RT_ANGLE_PLUG_HEADER
- J5: value RJ45_TH_VERT -> 4-pos; device 3D_MIG_Controller:RJ45_TH_VERT -> 3D_MIG_Controller:3.81MM_1_X_4_RT_ANGLE_PLUG_HEADER
Connections:
- new net NC: J6.4, J7.4
- net GND: now also J11.1, J11.6, J12.1, J12.6, J15.1, J15.6, J5.P$1; no longer J11.P$1, J18.1, J18.4, J18.6, J19.1, J19.4, J19.6, J5.1, J5.6
- net INT_00: now also J6.2; no longer J18.2
- net INT_01: now also J7.2; no longer J19.2
- net IN_DIR_M_0: now also J8.4; no longer J5.4
- net IN_DIR_M_1: now also J9.4; no longer J7.4
- net IN_DIR_M_2: now also J10.4; no longer J9.4
- net IN_DIR_M_3: now also J11.4; no longer J6.4
- net IN_DIR_M_4: now also J12.4; no longer J10.4
- net IN_DIR_M_6: now also J14.4; no longer J8.4
- net IN_DIR_M_7: now also J15.4; no longer J14.4
- net IN_STEP_M_0: now also J8.2; no longer J5.2
- net IN_STEP_M_1: now also J9.2; no longer J7.2
- net IN_STEP_M_2: now also J10.2; no longer J9.2
- net IN_STEP_M_3: now also J11.2; no longer J6.2
- net IN_STEP_M_4: now also J12.2; no longer J10.2
- net IN_STEP_M_6: now also J14.2; no longer J8.2
- net IN_STEP_M_7: now also J15.2; no longer J14.2
- net VDD: now also J11.5, J12.5, J15.5, J5.P$2; no longer J18.5, J19.5, J4.P$2, J5.5
- net VDD-12: now also J11.7, J12.7, J15.7, J4.P$2; no longer J11.P$2, J18.7, J19.7, J5.7
- net VDD12: now also J11.3, J12.3, J15.3, J5.P$4; no longer J18.3, J19.3, J4.P$4, J5.3
- net VDD5: now also J11.8, J12.8, J15.8, J5.P$3; no longer J18.8, J19.8, J4.P$3, J5.8
Other:
- moved on the sheet: J10, J14, J6, J7, J8, J9
