File: Callisto_Relays/Callisto_Minor_2_Relays_v1p0.sch (EAGLE design)
At the start: 11 parts, among them J1 2-pos, J2 RJ45_TH_VERT, J5 2-pos, U2 NPN, U3 NPN

Commit message: Updated Callisto
Parts:
- removed J5: 2-pos, 3D_MIG_Controller:3.81MM_1_X_2_RT_ANGLE_PLUG_HEADER
- removed R3: 500R0, 3D_MIG_Controller:R_0402
- removed U2, U3: NPN, 3D_MIG_Controller:BC846BW
- added J3: RJ45_TH_VERT, 3D_MIG_Controller:RJ45_TH_VERT
- added LED1, LED2: Green, 3D_MIG_Controller:LED_0805_GREEN
- added R2: 470R0, 3D_MIG_Controller:R_0402_470R0
- J2: value RJ45_TH_VERT -> 2-pos; device 3D_MIG_Controller:RJ45_TH_VERT -> 3D_MIG_Controller:3.81MM_1_X_2_RT_ANGLE_PLUG_HEADER
- R1: value 500R0 -> 470R0; device 3D_MIG_Controller:R_0402 -> 3D_MIG_Controller:R_0402_470R0
Connections:
- removed net N$2: R1.2, U2.B(2)
- removed net N$3: U$3.VC-, U2.C(3)
- removed net N$5: R3.2, U3.B(2)
- removed net N$6: U$5.VC-, U3.C(3)
- new net N$1: LED1.A, R1.1
- new net N$7: LED2.A, R2.1
- net GND: now also J3.1, J3.6; no longer J2.1, J2.6, U2.E(1), U3.E(1)
- net RELAY_1: now also J3.2, LED1.C, U$3.VC-; no longer J2.2, R1.1
- net RELAY_2: now also J3.4, LED2.C, U$5.VC-; no longer J2.4, R3.1
- net RO_NEG_2: now also J2.P$2; no longer J5.P$2
- net RO_POS_2: now also J2.P$1; no longer J5.P$1
- net VDD: now also J3.5; no longer J2.5
- net VDD-12: now also J3.7; no longer J2.7
- net VDD12: now also J3.3; no longer J2.3
- net VDD5: now also J3.8, R1.2, R2.2; no longer J2.8
Other:
- moved on the sheet: R1
