File: S7G2_3_Axis_plus_Ethernet/S7G7_footprint_simplified_w_ethernet_v1p23.brd (EAGLE design)
At the start: 100 x 100 mm, 147 parts, among them J9 SD_CARD_1140084168, U2 AP2141DWG-5, U3 KSZ8081RNACAQFN-24-M, X3 32.768KHZ, X4 24MHZ

Commit message: Updated Renesas processor references.
Parts:
- U4: value (none) -> S7G2LQFP176
Changed lines of the file:
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@@
 <layer number="115" name="ReferenceISLANDS" color="7" fill="1" visible="yes" active="yes"/>
 <layer number="116" name="Patch_BOT" color="9" fill="4" visible="yes" active="yes"/>
+<layer number="117" name="PM_Ref" color="7" fill="1" visible="yes" active="yes"/>
 <layer number="118" name="Rect_Pads" color="7" fill="1" visible="yes" active="yes"/>
+<layer number="119" name="PF_Ref" color="7" fill="1" visible="yes" active="yes"/>
+<layer number="120" name="WFL_Ref" color="7" fill="1" visible="yes" active="yes"/>
 <layer number="121" name="_tsilk" color="7" fill="1" visible="yes" active="yes"/>
 <layer number="122" name="_bsilk" color="7" fill="1" visible="yes" active="yes"/>
@@
 <attribute name="VALUE" x="55.558" y="1.15" size="0.381" layer="27" font="vector" ratio="10" rot="R90" align="top-left"/>
 </element>
-<element name="U4" library="3D_MIG_Controller" package="LQFP176_24X24" value="" x="60.5" y="52" smashed="yes" rot="R45">
+<element name="U4" library="3D_MIG_Controller" package="LQFP176_24X24" value="S7G2LQFP176" x="60.5" y="52" smashed="yes" rot="R45">
 <attribute name="NAME" x="78.7565625" y="52.599996875" size="1.27" layer="25"/>
+<attribute name="PARTNO" value="R7FS7G27H3A01CFC#AA0" x="60.5" y="52" size="1.778" layer="27" rot="R45" display="off"/>
+<attribute name="VALUE" value="S7G2LQFP176" x="60.5" y="52" size="1.778" layer="27" rot="R45" display="off"/>
 </element>
 <element name="C10" library="3D_MIG_Controller" package="0402" value="0.1uF" x="73.651728125" y="64.518171875" smashed="yes" rot="MR45"/>
