File: S7G2_3_Axis_plus_Ethernet/S7G7_footprint_simplified_w_ethernet_v1p23.sch (EAGLE design)
At the start: 147 parts, among them J9 SD_CARD_1140084168, U2 AP2141DWG-5, U3 KSZ8081RNACAQFN-24-M, X3 32.768KHZ, X4 24MHZ

Commit message: Updated Renesas processor references.
Parts:
- U4: value (none) -> S7G2LQFP176; device 3D_MIG_Controller:S7G2_X_176 -> 3D_MIG_Controller:RENESAS_S7G2_X_176
Changed lines of the file:
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@@
 <layer number="115" name="ReferenceISLANDS" color="7" fill="1" visible="yes" active="yes"/>
 <layer number="116" name="Patch_BOT" color="9" fill="4" visible="yes" active="yes"/>
+<layer number="117" name="PM_Ref" color="7" fill="1" visible="yes" active="yes"/>
 <layer number="118" name="Rect_Pads" color="7" fill="1" visible="yes" active="yes"/>
+<layer number="119" name="PF_Ref" color="7" fill="1" visible="yes" active="yes"/>
+<layer number="120" name="WFL_Ref" color="7" fill="1" visible="yes" active="yes"/>
 <layer number="121" name="_tsilk" color="7" fill="1" visible="yes" active="yes"/>
 <layer number="122" name="_bsilk" color="7" fill="1" visible="yes" active="yes"/>
@@
 <part name="GND46" library="3D_MIG_Controller" deviceset="GND" device=""/>
 <part name="J3" library="3D_MIG_Controller" deviceset="USB_A" device=""/>
-<part name="U4" library="3D_MIG_Controller" deviceset="S7G2_X_176" device=""/>
+<part name="U4" library="3D_MIG_Controller" deviceset="RENESAS_S7G2_X_176" device="" value="S7G2LQFP176"/>
 <part name="C10" library="3D_MIG_Controller" deviceset="C_0402" device="" value="0.1uF"/>
 <part name="C13" library="3D_MIG_Controller" deviceset="C_0402" device="" value="0.1uF"/>
