File: S7G2_Titan/Titan_v1p4.sch (EAGLE design)
At the start: 93 parts, among them J1 SD_CARD, J10 20-pos, J2 4-pos, J3 10-pos, J4 20-pos, J5 10-pos, J6 USB-A, J7 USB-B-Micro, J8 40-pos, J9 10-pos, U1 KSZ8081_QFN_24, U2 AP2151DWG-7, U3 S7G2LQFP176, X1 25MHz, X2 24MHz, X3 32.768KHz

Commit message: Updated Renesas processor references.
Parts:
- U3: device 3D_MIG_Controller:S7G2_X_176 -> 3D_MIG_Controller:RENESAS_S7G2_X_176
Changed lines of the file:
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@@
 <part name="GND46" library="3D_MIG_Controller" deviceset="GND" device=""/>
 <part name="J6" library="3D_MIG_Controller" deviceset="USB_A" device="" value="USB-A"/>
-<part name="U3" library="3D_MIG_Controller" deviceset="S7G2_X_176" device="" value="S7G2LQFP176"/>
+<part name="U3" library="3D_MIG_Controller" deviceset="RENESAS_S7G2_X_176" device="" value="S7G2LQFP176"/>
 <part name="C35" library="3D_MIG_Controller" deviceset="C_0402_0.1UF" device="" value="0.1uF"/>
 <part name="C38" library="3D_MIG_Controller" deviceset="C_0402_0.1UF" device="" value="0.1uF"/>
