File: S7G2_Titan/Titan_v1p6.brd (EAGLE design)
At the start: 60 x 92 mm, 93 parts, among them J1 SD_CARD, J10 20-pos, J2 4-pos, J3 10-pos, J4 20-pos, J5 10-pos, J6 USB-A, J7 USB-B-Micro, J8 40-pos, J9 10-pos, U1 KSZ8081_QFN_24, U2 AP2151DWG-7, U3 S7G2LQFP176, X1 25MHz, X2 24MHz, X3 32.768KHz

Commit message: Updated Titan USB
Parts:
- C31: value 10uF_Tant -> 100uF_Tant
Changed lines of the file:
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@@
 <attribute name="PARTNO" value="CL05F104ZO5NNNC" x="28.3" y="15.1" size="1.778" layer="27" rot="R270" display="off"/>
 </element>
-<element name="C31" library="3D_MIG_Controller" package="C1210" package3d_urn="urn:adsk.eagle:package:26139/1" value="10uF_Tant" x="28.9" y="17.7" smashed="yes" rot="R180">
-<attribute name="PARTNO" value="TPST106K016H0800" x="28.9" y="17.7" size="1.778" layer="27" rot="R180" display="off"/>
+<element name="C31" library="3D_MIG_Controller" package="C1210" package3d_urn="urn:adsk.eagle:package:26139/1" value="100uF_Tant" x="28.9" y="17.7" smashed="yes" rot="R180">
+<attribute name="PARTNO" value="TLJT107M010R0900" x="28.9" y="17.7" size="1.778" layer="27" rot="R180" display="off"/>
 </element>
 <element name="J6" library="3D_MIG_Controller" package="USB_A_SMT" value="USB-A" x="35" y="7.4" smashed="yes" rot="R90">
