File: S7G2_Titan/Titan_v1p7.sch (EAGLE design)
At the start: 172 parts, among them J1 SD_CARD, J10 20-pos, J2 4-pos, J3 10-pos, J4 20-pos, J5 10-pos, J6 USB-A, J7 USB-B-Micro, J9 10-pos, U1 KSZ8081_QFN_24, U10 NPN, U11 NPN, U12 NPN, U13 NPN, U14 NPN, U15 NPN, U16 NPN, U17 NPN, U18 NPN, U19 NPN, U2 AP2151DWG-7, U20 NPN, U21 NPN, U22 NPN, U23 NPN, U24 NPN, U25 NPN, U26 NPN, U27 NPN, U3 S7G2LQFP176, U34 NPN, U35 NPN, U36 NPN, U37 NPN, U38 NPN, U39 NPN, X1 25MHz, X2 24MHz, X3 32.768KHz

Commit message: Updated Titan Design
Parts:
- removed R53, R54, R57, R58, R59, R60: (no value), 3D_MIG_Controller:R_0805
- removed R55: 1k, 3D_MIG_Controller:R_0805
- removed R56: 33, 3D_MIG_Controller:R_0805
- removed U18, U19, U20, U21: NPN, 3D_MIG_Controller:BC846BW
- added J11, J12, J19, J20, J23, J24: 2-pos, 3D_MIG_Controller:3.81MM_1_X_2_RT_ANGLE_PLUG_HEADER
- added J25, J26, J29, J30, J33, J34: (no value), 3D_MIG_Controller:TEKNIC_8PIN_MOTOR
- added J8: 40-pos, 3D_MIG_Controller:HEADER_2_X_20_GENERIC
- added LED4, LED5, LED8, LED9: Green, 3D_MIG_Controller:LED_0805_GREEN
- added R109, R113, R114, R115, R119, R120, R133, R137, R138, R139, R143, R144, R157, R161, R162, R163, R167, R168: 1k, 3D_MIG_Controller:R_0805
- added R110, R111, R112, R116, R117, R118, R134, R135, R136, R140, R141, R142, R158, R159, R160, R164, R165, R166: 33, 3D_MIG_Controller:R_0805
- added R29, R30: 500R0, 3D_MIG_Controller:R_0402
- added R31, R32: 470R0, 3D_MIG_Controller:R_0402_470R0
- added U$1, U$2, U$7, U$8: RELAY_KYOTO_KF0604D, 3D_MIG_Controller:RELAY_KYOTO_KF0604D
- added U46, U47, U48, U49, U50, U51, U58, U59, U6, U60, U61, U62, U63, U7, U70, U71, U72, U73, U74, U75: NPN, 3D_MIG_Controller:BC846BW
- J15, J16: value (none) -> 2-pos; device 3D_MIG_Controller:TEKNIC_8PIN_MOTOR -> 3D_MIG_Controller:3.81MM_1_X_2_RT_ANGLE_PLUG_HEADER
- R39, R40, R45, R46, R63, R64, R69, R70, R87, R88, R93, R94: value (none) -> 33
- R41, R42, R47, R48, R65, R66, R71, R72, R89, R90, R95, R96: value (none) -> 1k
- R49: value 1k -> 500R0; device 3D_MIG_Controller:R_0805 -> 3D_MIG_Controller:R_0402
- R50: value 33 -> 500R0; device 3D_MIG_Controller:R_0805 -> 3D_MIG_Controller:R_0402
- R51, R52: value (none) -> 470R0; device 3D_MIG_Controller:R_0805 -> 3D_MIG_Controller:R_0402_470R0
Connections:
- net A_DIR_X renamed X_A_DIR
- net A_DIR_Y renamed Y_A_DIR
- net A_DIR_Z renamed Z_A_DIR
- net A_ENABLE_X renamed X_A_ENABLE
- net A_ENABLE_Y renamed Y_A_ENABLE
- net A_ENABLE_Z renamed Z_A_ENABLE
- net A_HLFB_OUT_X renamed X_A_HLFB_OUT
- net A_HLFB_OUT_Y renamed Y_A_HLFB_OUT
- net A_HLFB_OUT_Z renamed Z_A_HLFB_OUT
- net A_MI_DIR_X renamed X_A_MI_DIR
- net A_MI_DIR_Y renamed Y_A_MI_DIR
- net A_MI_DIR_Z renamed Z_A_MI_DIR
- net A_MI_ENABLE_X renamed X_A_MI_ENABLE
- net A_MI_ENABLE_Y renamed Y_A_MI_ENABLE
- net A_MI_ENABLE_Z renamed Z_A_MI_ENABLE
- net A_MI_STEP_X renamed X_A_MI_STEP
- net A_MI_STEP_Y renamed Y_A_MI_STEP
- net A_MI_STEP_Z renamed Z_A_MI_STEP
- net A_STEP_A renamed RELAY_4
- net A_STEP_X renamed X_A_STEP
- net A_STEP_Y renamed Y_A_STEP
- net A_STEP_Z renamed Z_A_STEP
- net B_DIR_X renamed X_B_DIR
- net B_DIR_Y renamed Y_B_DIR
- net B_DIR_Z renamed Z_B_DIR
- net B_ENABLE_X renamed X_B_ENABLE
- net B_ENABLE_Y renamed Y_B_ENABLE
- net B_ENABLE_Z renamed Z_B_ENABLE
- net B_HLFB_OUT_X renamed X_B_HLFB_OUT
- net B_HLFB_OUT_Y renamed Y_B_HLFB_OUT
- net B_HLFB_OUT_Z renamed Z_B_HLFB_OUT
- net B_MI_DIR_X renamed X_B_MI_DIR
- net B_MI_DIR_Y renamed Y_B_MI_DIR
- net B_MI_DIR_Z renamed Z_B_MI_DIR
- net B_MI_ENABLE_X renamed X_B_MI_ENABLE
- net B_MI_ENABLE_Y renamed Y_B_MI_ENABLE
- net B_MI_ENABLE_Z renamed Z_B_MI_ENABLE
- net B_MI_STEP_X renamed X_B_MI_STEP
- net B_MI_STEP_Y renamed Y_B_MI_STEP
- net B_MI_STEP_Z renamed Z_B_MI_STEP
- net B_STEP_X renamed X_B_STEP
- net B_STEP_Y renamed Y_B_STEP
- net B_STEP_Z renamed Z_B_STEP
- removed net A_DIR_A: R51.1
- removed net A_ENABLE_A: R52.1
- removed net A_HLFB_OUT_A: J15.5-HLFB-
- removed net A_MI_DIR_A: J15.7-INPUT_A-, R53.1, U17.C(3)
- removed net A_MI_ENABLE_A: J15.8-ENABLE-, R54.1, U18.C(3)
- removed net A_MI_STEP_A: J15.6-INPUT_B-, R49.1, U16.C(3)
- removed net B_DIR_A: R57.1
- removed net B_ENABLE_A: R58.1
- removed net B_HLFB_OUT_A: J16.5-HLFB-
- removed net B_MI_ENABLE_A: J16.8-ENABLE-, R60.1, U21.C(3)
- removed net B_MI_STEP_A: J16.6-INPUT_B-, R55.1, U19.C(3)
- removed net B_STEP_A: R56.1
- new net A_A_DIR: R111.1
- new net A_A_ENABLE: R112.1
- new net A_A_HLFB_OUT: J25.5-HLFB-
- new net A_A_MI_DIR: J25.7-INPUT_A-, R113.1, U47.C(3)
- new net A_A_MI_ENABLE: J25.8-ENABLE-, R114.1, U48.C(3)
- new net A_A_MI_STEP: J25.6-INPUT_B-, R109.1, U46.C(3)
- new net A_A_STEP: R110.1
- new net A_B_DIR: R117.1
- new net A_B_ENABLE: R118.1
- new net A_B_HLFB_OUT: J26.5-HLFB-
- new net A_B_MI_DIR: J26.7-INPUT_A-, R119.1, U50.C(3)
- new net A_B_MI_ENABLE: J26.8-ENABLE-, R120.1, U51.C(3)
- new net A_B_MI_STEP: J26.6-INPUT_B-, R115.1, U49.C(3)
- new net A_B_STEP: R116.1
- new net C_A_DIR: R135.1
- new net C_A_ENABLE: R136.1
- new net C_A_HLFB_OUT: J29.5-HLFB-
- new net C_A_MI_DIR: J29.7-INPUT_A-, R137.1, U59.C(3)
- new net C_A_MI_ENABLE: J29.8-ENABLE-, R138.1, U60.C(3)
- new net C_A_MI_STEP: J29.6-INPUT_B-, R133.1, U58.C(3)
- new net C_A_STEP: R134.1
- new net C_B_DIR: R141.1
- new net C_B_ENABLE: R142.1
- new net C_B_HLFB_OUT: J30.5-HLFB-
- new net C_B_MI_DIR: J30.7-INPUT_A-, R143.1, U62.C(3)
- new net C_B_MI_ENABLE: J30.8-ENABLE-, R144.1, U63.C(3)
- new net C_B_MI_STEP: J30.6-INPUT_B-, R139.1, U61.C(3)
- new net C_B_STEP: R140.1
- new net N$44: R49.2, U16.B(2)
- new net N$45: LED8.C, U$7.VC-, U16.C(3)
- new net N$46: R50.2, U17.B(2)
- new net N$47: LED9.C, U$8.VC-, U17.C(3)
- new net N$48: LED9.A, R51.1
- new net N$49: LED8.A, R52.1
- new net N$50: R111.2, U47.B(2)
- new net N$51: R112.2, U48.B(2)
- new net N$52: R110.2, U46.B(2)
- new net N$53: R117.2, U50.B(2)
- new net N$54: R118.2, U51.B(2)
- new net N$55: R116.2, U49.B(2)
- new net N$62: R135.2, U59.B(2)
- new net N$63: R136.2, U60.B(2)
- new net N$64: R134.2, U58.B(2)
- new net N$65: R141.2, U62.B(2)
- new net N$66: R142.2, U63.B(2)
- new net N$67: R140.2, U61.B(2)
- new net N$74: R159.2, U71.B(2)
- new net N$75: R160.2, U72.B(2)
- new net N$76: R158.2, U70.B(2)
- new net N$77: R165.2, U74.B(2)
- new net N$78: R166.2, U75.B(2)
- new net N$79: R164.2, U73.B(2)
- new net RELAY_1: R29.1
- new net RELAY_2: R30.1
- new net RELAY_3: R49.1
- new net RO_NEG_1: J15.P$2, U$1.VO-
- new net RO_NEG_2: J16.P$2, U$2.VO-
- new net RO_NEG_3: J23.P$2, U$7.VO-
- new net RO_NEG_4: J24.P$2, U$8.VO-
- new net RO_POS_1: J15.P$1, U$1.VO+
- new net RO_POS_2: J16.P$1, U$2.VO+
- new net RO_POS_3: J23.P$1, U$7.VO+
- new net RO_POS_4: J24.P$1, U$8.VO+
- new net WF_A_DIR: R159.1
- new net WF_A_ENABLE: R160.1
- new net WF_A_HLFB_OUT: J33.5-HLFB-
- new net WF_A_MI_DIR: J33.7-INPUT_A-, R161.1, U71.C(3)
- new net WF_A_MI_ENABLE: J33.8-ENABLE-, R162.1, U72.C(3)
- new net WF_A_MI_STEP: J33.6-INPUT_B-, R157.1, U70.C(3)
- new net WF_A_STEP: R158.1
- new net WF_B_DIR: R165.1
- new net WF_B_ENABLE: R166.1
- new net WF_B_HLFB_OUT: J34.5-HLFB-
- new net WF_B_MI_ENABLE: J34.8-ENABLE-, R168.1, U75.C(3)
- new net WF_B_MI_STEP: J34.6-INPUT_B-, R163.1, U73.C(3)
- new net WF_B_STEP: R164.1
- net B_MI_DIR: now also J34.7-INPUT_A-, R167.1, U74.C(3); no longer J16.7-INPUT_A-, R59.1, U20.C(3)
- net GND: now also J8.P$1, U46.E(1), U47.E(1), U48.E(1), U49.E(1), U50.E(1), U51.E(1), U58.E(1), U59.E(1), U6.E(1), U60.E(1), U61.E(1), U62.E(1), U63.E(1), U7.E(1), U70.E(1), U71.E(1), U72.E(1), U73.E(1), U74.E(1), U75.E(1); no longer U18.E(1), U19.E(1), U20.E(1), U21.E(1)
- net IIC_1_SCL: now also J8.P$5
- net IIC_1_SDA: now also J8.P$6
- net INT_MI_01: now also J8.P$39
- net INT_MI_02: now also J8.P$40
- net INT_MI_03: now also J8.P$9
- net INT_MI_04: now also J8.P$10
- net N$20: now also R29.2, U6.B(2); no longer R51.2, U17.B(2)
- net N$21: now also LED4.C, U$1.VC-, U6.C(3); no longer R52.2, U18.B(2)
- net N$22: now also R30.2, U7.B(2); no longer R50.2, U16.B(2)
- net N$23: now also LED5.C, U$2.VC-, U7.C(3); no longer R57.2, U20.B(2)
- net N$24: now also LED5.A, R31.1; no longer R58.2, U21.B(2)
- net N$25: now also LED4.A, R32.1; no longer R56.2, U19.B(2)
- net P1_02: now also J8.P$7
- net P1_03: now also J8.P$8
- net P1_06: now also J8.P$11
- net P1_07: now also J8.P$12
- net P1_11: now also J8.P$38
- net P1_12: now also J8.P$37
- net P1_13: now also J8.P$36
- net P1_14: now also J8.P$35
- net P1_15: now also J8.P$34
- net P6_00: now also J8.P$13
- net P6_01: now also J8.P$14
- net P6_02: now also J8.P$15
- net P6_03: now also J8.P$16
- net P6_04: now also J8.P$17
- net P6_05: now also J8.P$18
- net P6_06: now also J8.P$19
- net P6_07: now also J8.P$20
- net P6_08: now also J8.P$33
- net P6_09: now also J8.P$32
- net P6_10: now also J8.P$31
- net P6_11: now also J8.P$30
- net P6_12: now also J8.P$29
- net P6_13: now also J8.P$28
- net P6_14: now also J8.P$27
- net P6_15: now also J8.P$26
- net P8_00: now also J8.P$4
- net P8_01: now also J8.P$3
- net P8_02: now also J8.P$2
- net PA_00: now also J8.P$21
- net PA_01: now also J8.P$22
- net PA_08: now also J8.P$25
- net PA_09: now also J8.P$24
- net PA_10: now also J8.P$23
- net VDD12: now also J25.1-HLFB+, J25.2-INPUT_B+, J25.3-INPUT_A+, J25.4-ENABLE+, J26.1-HLFB+, J26.2-INPUT_B+, J26.3-INPUT_A+, J26.4-ENABLE+, J29.1-HLFB+, J29.2-INPUT_B+, J29.3-INPUT_A+, J29.4-ENABLE+, J30.1-HLFB+, J30.2-INPUT_B+, J30.3-INPUT_A+, J30.4-ENABLE+, J33.1-HLFB+, J33.2-INPUT_B+, J33.3-INPUT_A+, J33.4-ENABLE+, J34.1-HLFB+, J34.2-INPUT_B+, J34.3-INPUT_A+, J34.4-ENABLE+, R109.2, R113.2, R114.2, R115.2, R119.2, R120.2, R133.2, R137.2, R138.2, R139.2, R143.2, R144.2, R157.2, R161.2, R162.2, R163.2, R167.2, R168.2; no longer J15.1-HLFB+, J15.2-INPUT_B+, J15.3-INPUT_A+, J15.4-ENABLE+, J16.1-HLFB+, J16.2-INPUT_B+, J16.3-INPUT_A+, J16.4-ENABLE+, R49.2, R53.2, R54.2, R55.2, R59.2, R60.2
- net VDD5: now also R31.2, R32.2, R51.2, R52.2, U$1.VC+, U$2.VC+, U$7.VC+, U$8.VC+
Other:
- moved on the sheet: J13, J14, J17, J18, J21, J22, R37, R38, R39, R40, R41, R42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
