File: HIVDC_Startup_S3/HVDCS_S3A6_48_TQFP.brd (EAGLE design)
At the start: 35 x 35 mm, 15 parts, among them J3 10-pos, U1 NPN, U2 NPN, U3 NPN, U6 RENESAS_R7FS3A6783A01CFLAA0PL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

Commit message: Update HVDCS_S3A6_48_TQFP.brd
Parts:
- moved U$5 26.2 mm to (30.8, 4.60), turned to 0 degrees
- moved U1 23.1 mm to (6.00, 8.10)
- moved R1 22.7 mm to (5.00, 11.2), turned to 180 degrees
- moved U2 17.3 mm to (8.60, 8.10)
- moved R2 16.4 mm to (7.60, 11.1), turned to 180 degrees
- moved U3 11.5 mm to (11.1, 8.10)
- moved R3 10.9 mm to (10.2, 11.1), turned to 180 degrees
Routing:
- net VDD5: track 30.4 -> 19.9 mm
- net AC_L1_ONOFF: track 0.00 -> 3.92 mm
- net HVP_ONOFF: track 0.00 -> 3.91 mm
- net AC_L2_ONOFF: track 0.00 -> 3.89 mm
- net VDD: track 92.2 -> 94.3 mm
