File: AC-DC Supply Module 1/AC-DC-Supply-M1.sch (EAGLE design)
At the start: 3 parts, among them X1 726386-2, X2 726386-2, X3 MOLEX_206832-0601MOLEX_206832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

Commit message: HW02.02
Added -5V Output and voltage regulator
Connections:
- new net V_-5V0: X3B.6
- net GND: no longer X3B.6
