File: Aqua_system/Aqua_D_CTRL/Aqua_D_CTRL/Aqua_D_CTRL.brd (EAGLE design)
At the start: 150 x 120 mm, 233 parts, among them IC1 SN65HVD3082EDR, IC2 CSTNE8M00G520000R0, IC3 LT6106CS5#TRPBF, IC4 LT6106CS5#TRPBF, IC5 TPS54202DDCR, IC6 LD1117S33TR, IC8 LM317AEMP, J1 ESP32-PICO-KIT, K1 KB20C06A, K2 KB20C06A, Q1 DMP6185SEQ-13, Q10 BC817, Q11 2N7002, Q12 DMP6185SEQ-13, Q13 2N7002, Q14 DMP6185SEQ-13, Q15 2N7002, Q16 DMP6185SEQ-13, Q17 BC817, Q18 BC817, Q19 BC817, Q2 2N7002, Q20 BC817, Q21 BC817, Q22 BC817, Q23 BC817, Q3 DMP6185SEQ-13, Q4 2N7002, Q5 DMP6185SEQ-13, Q6 DMP6185SEQ-13, Q7 2N7002, Q8 DMP6185SEQ-13, Q9 2N7002, SW1 L101011MS02Q, U2 R7FA6M5BG3CFBLQFP_144_20X20_R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, X1 B2B-XH-AM(LF)(SN), X10 726386-2TE_726386-2, X11 282834-2, X12 RJ45-8L-B, X13 MICROMATCH-16, X14 RJ45-8L-B, X2 WF2549-2WS05S0B01, X3 282834-3, X4 282834-3, X5 726386-2TE_726386-2, X6 726386-2TE_726386-2, X7 726386-2TE_726386-2, X8 726386-2TE_726386-2, X9 726386-2TE_726386-2

Commit message: HW00.00 Ongoing
Finalizing Layout
Parts:
- R42: value 10K 1% -> 100R 1%
- moved D10 83.7 mm to (71.6, 31.6), turned to 0 degrees
- moved R42 82.5 mm to (71.5, 34.3), turned to 180 degrees
- moved R41 81.5 mm to (71.5, 38.4)
- moved R40 79.3 mm to (71.5, 36.3)
- moved R86 5.74 mm to (86.2, 98.7), turned to 180 degrees
- moved C66 1.40 mm to (71.5, 40.4)
- moved C44 0.51 mm to (81.5, 72.1)
- moved C41 0.51 mm to (87.5, 72.1)
- moved C53 0.51 mm to (89.5, 72.1)
- moved C55 0.51 mm to (83.6, 72.1)
- moved R84 0.51 mm to (85.6, 72.1)
Routing:
- net DO_ESP32_EN: track 3.09 -> 61.8 mm
- net DO_CONDUCTIV_SENSOR_ON: track 0.00 -> 24.5 mm, vias 0 -> 4
- net AI_24V0: track 12.3 -> 21.3 mm, vias 0 -> 2
- net VCC: track 374.3 -> 365.4 mm, vias 17 -> 20
- net V_24V0_P: track 196.2 -> 204.3 mm, vias 5 -> 6
- net GND: track 69.9 -> 63.0 mm
- net AI_I_SENSE_PH_SENSOR: track 36.0 -> 40.6 mm
- net DO_PH_SENSOR_ON: track 36.8 -> 33.9 mm, vias 2 -> 0
- net N$83: track 2.21 -> 0.00 mm
- net N$27: track 3.63 -> 5.47 mm
- net ESP32_TXD: track 60.5 -> 61.7 mm
- net DBG_SWDIO: track 15.9 -> 16.7 mm
- net NRST: track 37.6 -> 38.4 mm
- added copper zone on layer 1, net VCC
