File: Callisto_MSO_Teknic/Callisto_MSO_Teknic.sch (EAGLE design)
At the start: 12 parts, among them J2 4-pos, J3 4-pos, U1 NPN, U2 NPN, U3 NPN

Commit message: Updated Teknic MSO
Parts:
- removed J1: (no value), 3D_MIG_Controller:TEKNIC_8PIN_MOTOR
- removed J3: 4-pos, 3D_MIG_Controller:3.81MM_1_X_4_RT_ANGLE_PLUG_HEADER
- J2: value 4-pos -> (none); device 3D_MIG_Controller:3.81MM_1_X_4_RT_ANGLE_PLUG_HEADER -> 3D_MIG_Controller:TEKNIC_8PIN_MOTOR
- R1: value (none) -> 1k
- R4: value (none) -> 33
Connections:
- net N$1 renamed R1_IN
- removed net DIR: J3.P$1, R4.1
- removed net ENABLE: J3.P$3, R6.1
- removed net ENABLE-: J1.8-ENABLE-, R3.1, U3.C(3)
- removed net INPUT_A-: J1.7-INPUT_A-, R2.1, U2.C(3)
- removed net INPUT_B-: J1.6-INPUT_B-, R1.1, U1.C(3)
- removed net STEP: J3.P$2, R5.1
- new net DIR1: R5.1
- new net ENABLE1: R6.1
- new net HLFB_OUT_1: J2.5-HLFB-
- new net MI_DIR1: J2.7-INPUT_A-, R2.1, U2.C(3)
- new net MI_ENABLE1: J2.8-ENABLE-, R3.1, U3.C(3)
- new net MI_STEP1: J2.6-INPUT_B-, R1.1, U1.C(3)
- new net STEP1: R4.1
- net GND: no longer J2.P$1
- net VDD12: now also J2.1-HLFB+, J2.2-INPUT_B+, J2.3-INPUT_A+, J2.4-ENABLE+; no longer J1.2-INPUT_B+, J1.3-INPUT_A+, J1.4-ENABLE+, J2.P$2
Other:
- moved on the sheet: R3
