File: Callisto_MSO_Teknic/Callisto_MSO_Teknic_v1p00.brd (EAGLE design)
At the start: 115 x 60 mm, 102 parts, among them J7 4-pos, U1 NPN, U13 NPN, U14 NPN, U15 NPN, U16 NPN, U17 NPN, U18 NPN, U2 NPN, U25 NPN, U26 NPN, U27 NPN, U28 NPN, U29 NPN, U3 NPN, U30 NPN, U37 NPN, U38 NPN, U39 NPN, U4 NPN, U40 NPN, U41 NPN, U42 NPN, U49 NPN, U5 NPN, U50 NPN, U51 NPN, U52 NPN, U53 NPN, U54 NPN, U6 NPN

Commit message: Update Callisto
Routing:
- net ENABLE: vias 10 -> 2
Changed lines of the file:
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@@
 <via x="89.9" y="21.1" extent="1-16" drill="0.35"/>
 <via x="43" y="42.5" extent="1-16" drill="0.35"/>
+<via x="90.8" y="45.4" extent="1-16" drill="0.35"/>
 </signal>
 <signal name="VDD12">
@@
 <wire x1="7.1" y1="47.6" x2="7.2" y2="39.95" width="0.508" layer="16"/>
 <wire x1="7.2" y1="39.95" x2="7.05" y2="39.8" width="0.508" layer="16"/>
-<via x="29.6" y="47.6" extent="1-16" drill="0.35"/>
 <wire x1="29.6" y1="47.6" x2="29.6" y2="39.85" width="0.508" layer="16"/>
 <wire x1="29.6" y1="39.85" x2="29.45" y2="39.7" width="0.508" layer="16"/>
-<via x="51.3" y="47.6" extent="1-16" drill="0.35"/>
 <wire x1="51.35" y1="41.75" x2="51.35" y2="39.7" width="0.508" layer="16"/>
-<via x="73.9" y="47.6" extent="1-16" drill="0.35"/>
 <wire x1="73.9" y1="47.6" x2="73.9" y2="39.85" width="0.508" layer="16"/>
 <wire x1="73.9" y1="39.85" x2="73.85" y2="39.8" width="0.508" layer="16"/>
-<via x="96.6" y="47.6" extent="1-16" drill="0.35"/>
 <wire x1="96.6" y1="47.6" x2="96.6" y2="39.75" width="0.508" layer="16"/>
 <wire x1="96.6" y1="39.75" x2="96.55" y2="39.7" width="0.508" layer="16"/>
@@
 <wire x1="7.1" y1="25" x2="7.1" y2="22.25" width="0.508" layer="16"/>
 <wire x1="7.1" y1="22.25" x2="7.05" y2="22.2" width="0.508" layer="16"/>
-<via x="29.5" y="25" extent="1-16" drill="0.35"/>
 <wire x1="29.5" y1="25" x2="29.5" y2="22.15" width="0.508" layer="16"/>
 <wire x1="29.5" y1="22.15" x2="29.45" y2="22.1" width="0.508" layer="16"/>
-<via x="51.4" y="25" extent="1-16" drill="0.35"/>
 <wire x1="51.4" y1="25" x2="51.4" y2="22.15" width="0.508" layer="16"/>
 <wire x1="51.4" y1="22.15" x2="51.35" y2="22.1" width="0.508" layer="16"/>
-<via x="73.8" y="25" extent="1-16" drill="0.35"/>
 <wire x1="73.8" y1="25" x2="73.85" y2="24.25" width="0.508" layer="16"/>
 <wire x1="73.85" y1="24.25" x2="73.85" y2="22.2" width="0.508" layer="16"/>
-<via x="96.6" y="25" extent="1-16" drill="0.35"/>
 <wire x1="96.6" y1="25" x2="96.6" y2="22.15" width="0.508" layer="16"/>
 <wire x1="96.6" y1="22.15" x2="96.55" y2="22.1" width="0.508" layer="16"/>
@@
 <wire x1="85.1" y1="42.1" x2="100" y2="42.1" width="0.254" layer="1"/>
 </signal>
-<signal name="N$10">
-<via x="90.7" y="42.8" extent="1-16" drill="0.35"/>
-</signal>
 </signals>

Commit message: Updated MSO Teknic
Parts:
- R10, R101, R102, R107, R108, R11, R12, R29, R30, R35, R36, R53, R54, R59, R60, R77, R78, R83, R84, R9: value (none) -> 1k
- R100, R105, R106, R2, R27, R28, R3, R33, R34, R5, R51, R52, R57, R58, R6, R75, R76, R81, R82, R99: value (none) -> 33
