File: Callisto_MSO_Teknic/Callisto_MSO_Teknic_v1p00.sch (EAGLE design)
At the start: 102 parts, among them J7 4-pos, U1 NPN, U13 NPN, U14 NPN, U15 NPN, U16 NPN, U17 NPN, U18 NPN, U2 NPN, U25 NPN, U26 NPN, U27 NPN, U28 NPN, U29 NPN, U3 NPN, U30 NPN, U37 NPN, U38 NPN, U39 NPN, U4 NPN, U40 NPN, U41 NPN, U42 NPN, U49 NPN, U5 NPN, U50 NPN, U51 NPN, U52 NPN, U53 NPN, U54 NPN, U6 NPN

Commit message: Updated MSO Teknic
Parts:
- R10, R101, R102, R107, R108, R11, R12, R29, R30, R35, R36, R53, R54, R59, R60, R77, R78, R83, R84, R9: value (none) -> 1k
- R100, R105, R106, R2, R27, R28, R3, R33, R34, R5, R51, R52, R57, R58, R6, R75, R76, R81, R82, R99: value (none) -> 33
