File: Callisto_MSO_Teknic/Callisto_Teknic_MSO_LED_out.sch (EAGLE design)
At the start: 13 parts, among them J2 ATX24RH

Commit message: Updated DBs
Parts:
- removed LED1, LED2, LED3, LED4: Green, 3D_MIG_Controller:LED_0805_GREEN
- removed R1, R2, R3, R4: (no value), 3D_MIG_Controller:R_0805
- added J10, J13, J14, J17, J18, J3, J5, J6, J9: (no value), 3D_MIG_Controller:TEKNIC_MOTOR_SD_8PIN
- added LED10, LED11, LED12, LED17, LED18, LED19, LED20, LED21, LED22, LED23, LED24, LED33, LED34, LED35, LED36, LED37, LED38, LED39, LED40, LED49, LED50, LED51, LED52, LED53, LED54, LED55, LED56, LED65, LED66, LED67, LED68, LED69, LED7, LED70, LED71, LED72, LED8, LED9: Green, 3D_MIG_Controller:LED_0805_GREEN
- added R10, R11, R12, R17, R18, R19, R20, R21, R22, R23, R24, R33, R34, R35, R36, R37, R38, R39, R40, R49, R50, R51, R52, R53, R54, R55, R56, R65, R66, R67, R68, R69, R7, R70, R71, R72, R8, R9: (no value), 3D_MIG_Controller:R_0805
- J2: value ATX24RH -> (none); device 3D_MIG_Controller:ATX24RH -> 3D_MIG_Controller:TEKNIC_MOTOR_SD_8PIN
Connections:
- removed net DIR+: J2.12V@1, R2.2
- removed net DIR-: J2.5V@4, LED2.C
- removed net DIR2+: J2.GND@0, R5.2
- removed net DIR2-: J2.GND@3, LED5.C
- removed net ENABLE+: J2.3.3V@2, R1.2
- removed net ENABLE-: J2.GND@7, LED1.C
- removed net ENABLE2+: J2.5V@0, R4.2
- removed net ENABLE2-: J2.PS_ON, LED4.C
- removed net N$1: LED1.A, R1.1
- removed net N$2: LED2.A, R2.1
- removed net N$3: LED3.A, R3.1
- removed net N$4: LED4.A, R4.1
- removed net STEP+: J2.12V@0, R3.2
- removed net STEP-: J2.5V@3, LED3.C
- removed net STEP2+: J2.3.3V@1, R6.2
- removed net STEP2-: J2.-12V, LED6.C
- new net A_DIR+_A: J14.3-DIR+, R54.2
- new net A_DIR+_C: J18.3-DIR+, R70.2
- new net A_DIR+_X: J2.3-DIR+, R6.2
- new net A_DIR+_Y: J6.3-DIR+, R22.2
- new net A_DIR+_Z: J10.3-DIR+, R38.2
- new net A_DIR-A: J14.7-DIR-, LED54.C
- new net A_DIR-C: J18.7-DIR-, LED70.C
- new net A_DIR-X: J2.7-DIR-, LED6.C
- new net A_DIR-Y: J6.7-DIR-, LED22.C
- new net A_DIR-Z: J10.7-DIR-, LED38.C
- new net A_ENABLE+_A: J14.4-ENABLE+, R55.2
- new net A_ENABLE+_C: J18.4-ENABLE+, R71.2
- new net A_ENABLE+_X: J2.4-ENABLE+, R7.2
- new net A_ENABLE+_Y: J6.4-ENABLE+, R23.2
- new net A_ENABLE+_Z: J10.4-ENABLE+, R39.2
- new net A_ENABLE-_A: J14.8-ENABLE-, LED55.C
- new net A_ENABLE-_C: J18.8-ENABLE-, LED71.C
- new net A_ENABLE-_X: J2.8-ENABLE-, LED7.C
- new net A_ENABLE-_Y: J6.8-ENABLE-, LED23.C
- new net A_ENABLE-_Z: J10.8-ENABLE-, LED39.C
- new net A_HLFB+_A: J14.1-HLFB+, R56.2
- new net A_HLFB+_C: J18.1-HLFB+, R72.2
- new net A_HLFB+_X: J2.1-HLFB+, R8.2
- new net A_HLFB+_Y: J6.1-HLFB+, R24.2
- new net A_HLFB+_Z: J10.1-HLFB+, R40.2
- new net A_HLFB-_A: J14.5-HLFB-, LED56.C
- new net A_HLFB-_C: J18.5-HLFB-, LED72.C
- new net A_HLFB-_X: J2.5-HLFB-, LED8.C
- new net A_HLFB-_Y: J6.5-HLFB-, LED24.C
- new net A_HLFB-_Z: J10.5-HLFB-, LED40.C
- new net A_STEP+_A: J14.2-STEP+, R53.2
- new net A_STEP+_C: J18.2-STEP+, R69.2
- new net A_STEP+_X: J2.2-STEP+, R5.2
- new net A_STEP+_Y: J6.2-STEP+, R21.2
- new net A_STEP+_Z: J10.2-STEP+, R37.2
- new net A_STEP-_A: J14.6-STEP-, LED53.C
- new net A_STEP-_C: J18.6-STEP-, LED69.C
- new net A_STEP-_X: J2.6-STEP-, LED5.C
- new net A_STEP-_Y: J6.6-STEP-, LED21.C
- new net A_STEP-_Z: J10.6-STEP-, LED37.C
- new net B_DIR+_A: J13.3-DIR+, R50.2
- new net B_DIR+_WF: J17.3-DIR+, R66.2
- new net B_DIR+_X: J3.3-DIR+, R10.2
- new net B_DIR+_Y: J5.3-DIR+, R18.2
- new net B_DIR+_Z: J9.3-DIR+, R34.2
- new net B_DIR-X: J3.7-DIR-, LED10.C
- new net B_DIR-Y: J5.7-DIR-, LED18.C
- new net B_DIR-Z: J9.7-DIR-, LED34.C
- new net B_DIR-_A: J13.7-DIR-, LED50.C
- new net B_DIR-_WF: J17.7-DIR-, LED66.C
- new net B_ENABLE+_A: J13.4-ENABLE+, R51.2
- new net B_ENABLE+_WF: J17.4-ENABLE+, R67.2
- new net B_ENABLE+_X: J3.4-ENABLE+, R11.2
- new net B_ENABLE+_Y: J5.4-ENABLE+, R19.2
- new net B_ENABLE+_Z: J9.4-ENABLE+, R35.2
- new net B_ENABLE-_A: J13.8-ENABLE-, LED51.C
- new net B_ENABLE-_WF: J17.8-ENABLE-, LED67.C
- new net B_ENABLE-_X: J3.8-ENABLE-, LED11.C
- new net B_ENABLE-_Y: J5.8-ENABLE-, LED19.C
- new net B_ENABLE-_Z: J9.8-ENABLE-, LED35.C
- new net B_HLFB+_A: J13.1-HLFB+, R52.2
- new net B_HLFB+_WF: J17.1-HLFB+, R68.2
- new net B_HLFB+_X: J3.1-HLFB+, R12.2
- new net B_HLFB+_Y: J5.1-HLFB+, R20.2
- new net B_HLFB+_Z: J9.1-HLFB+, R36.2
- new net B_HLFB-_A: J13.5-HLFB-, LED52.C
- new net B_HLFB-_WF: J17.5-HLFB-, LED68.C
- new net B_HLFB-_X: J3.5-HLFB-, LED12.C
- new net B_HLFB-_Y: J5.5-HLFB-, LED20.C
- new net B_HLFB-_Z: J9.5-HLFB-, LED36.C
- new net B_STEP+_A: J13.2-STEP+, R49.2
- new net B_STEP+_WF: J17.2-STEP+, R65.2
- new net B_STEP+_X: J3.2-STEP+, R9.2
- new net B_STEP+_Y: J5.2-STEP+, R17.2
- new net B_STEP+_Z: J9.2-STEP+, R33.2
- new net B_STEP-_A: J13.6-STEP-, LED49.C
- new net B_STEP-_WF: J17.6-STEP-, LED65.C
- new net B_STEP-_X: J3.6-STEP-, LED9.C
- new net B_STEP-_Y: J5.6-STEP-, LED17.C
- new net B_STEP-_Z: J9.6-STEP-, LED33.C
- new net N$10: LED10.A, R10.1
- new net N$11: LED11.A, R11.1
- new net N$12: LED12.A, R12.1
- new net N$17: LED17.A, R17.1
- new net N$18: LED18.A, R18.1
- new net N$19: LED19.A, R19.1
- new net N$20: LED20.A, R20.1
- new net N$21: LED21.A, R21.1
- new net N$22: LED22.A, R22.1
- new net N$23: LED23.A, R23.1
- new net N$24: LED24.A, R24.1
- new net N$33: LED33.A, R33.1
- new net N$34: LED34.A, R34.1
- new net N$35: LED35.A, R35.1
- new net N$36: LED36.A, R36.1
- new net N$37: LED37.A, R37.1
- new net N$38: LED38.A, R38.1
- new net N$39: LED39.A, R39.1
- new net N$40: LED40.A, R40.1
- new net N$49: LED49.A, R49.1
- new net N$50: LED50.A, R50.1
- new net N$51: LED51.A, R51.1
- new net N$52: LED52.A, R52.1
- new net N$53: LED53.A, R53.1
- new net N$54: LED54.A, R54.1
- new net N$55: LED55.A, R55.1
- new net N$56: LED56.A, R56.1
- new net N$65: LED65.A, R65.1
- new net N$66: LED66.A, R66.1
- new net N$67: LED67.A, R67.1
- new net N$68: LED68.A, R68.1
- new net N$69: LED69.A, R69.1
- new net N$7: LED7.A, R7.1
- new net N$70: LED70.A, R70.1
- new net N$71: LED71.A, R71.1
- new net N$72: LED72.A, R72.1
- new net N$8: LED8.A, R8.1
- new net N$9: LED9.A, R9.1
Other:
- moved on the sheet: LED5, R5, R6

Commit message: Updated test board
Parts:
- added J1, J4: (no value), 3D_MIG_Controller:TEKNIC_MOTOR_SD_8PIN
- added LED1, LED13, LED14, LED15, LED16, LED2, LED3, LED4: Green, 3D_MIG_Controller:LED_0805_GREEN
- added R1, R13, R14, R15, R16, R2, R3, R4: (no value), 3D_MIG_Controller:R_0805
Connections:
- new net A_DIR+_WF: J4.3-DIR+, R14.2
- new net A_DIR-_WF: J4.7-DIR-, LED14.C
- new net A_ENABLE+_WF: J4.4-ENABLE+, R15.2
- new net A_ENABLE-_WF: J4.8-ENABLE-, LED15.C
- new net A_HLFB+_WF: J4.1-HLFB+, R16.2
- new net A_HLFB-_WF: J4.5-HLFB-, LED16.C
- new net A_STEP+_WF: J4.2-STEP+, R13.2
- new net A_STEP-_WF: J4.6-STEP-, LED13.C
- new net B_DIR+_C: J1.3-DIR+, R2.2
- new net B_DIR-C: J1.7-DIR-, LED2.C
- new net B_ENABLE+_C: J1.4-ENABLE+, R3.2
- new net B_ENABLE-_C: J1.8-ENABLE-, LED3.C
- new net B_HLFB+_C: J1.1-HLFB+, R4.2
- new net B_HLFB-_C: J1.5-HLFB-, LED4.C
- new net B_STEP+_C: J1.2-STEP+, R1.2
- new net B_STEP-_C: J1.6-STEP-, LED1.C
- new net N$1: LED1.A, R1.1
- new net N$13: LED13.A, R13.1
- new net N$14: LED14.A, R14.1
- new net N$15: LED15.A, R15.1
- new net N$16: LED16.A, R16.1
- new net N$2: LED2.A, R2.1
- new net N$3: LED3.A, R3.1
- new net N$4: LED4.A, R4.1
Other:
- moved on the sheet: J17, LED65, R65, R66, R67, R68

Commit message: Updated Boards
Parts:
- added J11, J19, J23, J27, J31, J35, J39, J43, J47, J51: (no value), 3D_MIG_Controller:CONN_530470310_PICOBLADE_X_3
- added J12, J20, J24, J28, J32, J36, J40, J44, J48, J52: 4-pos, 3D_MIG_Controller:3.81MM_1_X_4_RT_ANGLE_PLUG_HEADER
- added LED25, LED28, LED30, LED32, LED42, LED44, LED46, LED48, LED58, LED60: Green, 3D_MIG_Controller:LED_0805_GREEN
- added R100, R106, R27, R41, R47, R62, R76, R82, R88, R94: 2K2, 3D_MIG_Controller:R_0402
- added R101, R102, R107, R108, R28, R29, R42, R43, R48, R57, R63, R64, R77, R78, R83, R84, R89, R90, R95, R96: (no value), 3D_MIG_Controller:R_0402
- added SW10, SW12, SW14, SW16, SW18, SW2, SW20, SW4, SW6, SW8: PTS810SJG250SMTRLFS, 3D_MIG_Controller:PTS810SJG250SMTRLFS
- added U1, U11, U13, U15, U17, U20, U3, U5, U7, U9: NPN, 3D_MIG_Controller:BC846BW
Connections:
- new net BLACK_1: J11.2, J12.P$3, R28.1, R29.1
- new net BLACK_2: J19.2, J20.P$3, R42.1, R43.1
- new net BLACK_3: J23.2, J24.P$3, R48.1, R57.1
- new net BLACK_4: J27.2, J28.P$3, R63.1, R64.1
- new net BLACK_5: J31.2, J32.P$3, R77.1, R78.1
- new net BLACK_6: J35.2, J36.P$3, R83.1, R84.1
- new net BLACK_7: J39.2, J40.P$3, R89.1, R90.1
- new net BLACK_8: J43.2, J44.P$3, R95.1, R96.1
- new net BLACK_9: J47.2, J48.P$3, R101.1, R102.1
- new net BLACK_E_STOP: J51.2, J52.P$3, R107.1, R108.1
- new net BLUE: J11.1, J12.P$1, J12.P$2, J19.1, J20.P$1, J20.P$2, J23.1, J24.P$1, J24.P$2, J27.1, J28.P$1, J28.P$2, J31.1, J32.P$1, J32.P$2, J35.1, J36.P$1, J36.P$2, J39.1, J40.P$1, J40.P$2, J43.1, J44.P$1, J44.P$2, J47.1, J48.P$1, J48.P$2, J51.1, J52.P$1, J52.P$2, SW10.3, SW10.4, SW12.3, SW12.4, SW14.3, SW14.4, SW16.3, SW16.4, SW18.3, SW18.4, SW2.3, SW2.4, SW20.3, SW20.4, SW4.3, SW4.4, SW6.3, SW6.4, SW8.3, SW8.4
- new net BROWN: J11.3, J12.P$4, J19.3, J20.P$4, J23.3, J24.P$4, J27.3, J28.P$4, J31.3, J32.P$4, J35.3, J36.P$4, J39.3, J40.P$4, J43.3, J44.P$4, J47.3, J48.P$4, J51.3, J52.P$4, R100.1, R106.1, R27.1, R41.1, R47.1, R62.1, R76.1, R82.1, R88.1, R94.1, U1.C(3), U11.C(3), U13.C(3), U15.C(3), U17.C(3), U20.C(3), U3.C(3), U5.C(3), U7.C(3), U9.C(3)
- new net N$100: LED58.A, R100.2, U17.B(2)
- new net N$101: LED58.C, R102.2, SW18.1, SW18.2
- new net N$102: R101.2, U17.E(1)
- new net N$106: LED60.A, R106.2, U20.B(2)
- new net N$107: LED60.C, R108.2, SW20.1, SW20.2
- new net N$108: R107.2, U20.E(1)
- new net N$28: LED25.A, R27.2, U1.B(2)
- new net N$29: LED25.C, R29.2, SW2.1, SW2.2
- new net N$30: R28.2, U1.E(1)
- new net N$42: LED28.A, R41.2, U3.B(2)
- new net N$43: LED28.C, R43.2, SW4.1, SW4.2
- new net N$44: R42.2, U3.E(1)
- new net N$48: LED30.A, R47.2, U5.B(2)
- new net N$57: LED30.C, R57.2, SW6.1, SW6.2
- new net N$58: R48.2, U5.E(1)
- new net N$62: LED32.A, R62.2, U7.B(2)
- new net N$63: LED32.C, R64.2, SW8.1, SW8.2
- new net N$64: R63.2, U7.E(1)
- new net N$76: LED42.A, R76.2, U9.B(2)
- new net N$77: LED42.C, R78.2, SW10.1, SW10.2
- new net N$78: R77.2, U9.E(1)
- new net N$82: LED44.A, R82.2, U11.B(2)
- new net N$83: LED44.C, R84.2, SW12.1, SW12.2
- new net N$84: R83.2, U11.E(1)
- new net N$88: LED46.A, R88.2, U13.B(2)
- new net N$89: LED46.C, R90.2, SW14.1, SW14.2
- new net N$90: R89.2, U13.E(1)
- new net N$94: LED48.A, R94.2, U15.B(2)
- new net N$95: LED48.C, R96.2, SW16.1, SW16.2
- new net N$96: R95.2, U15.E(1)
