File: OutputIndicator/OutputIndicator_20_pins_v1p0.sch (EAGLE design)
At the start: 84 parts

Commit message: Updated Design added Output to 20 pin header
Connections:
- removed net IIC_1_SCL: RYS44.1
- removed net IIC_1_SDA: RYS3.1
- removed net INT_MI_03: RYS48.1
- removed net INT_MI_04: RYS7.1
- removed net INT_MI_05: RYS40.1
- removed net P1_02: RYS46.1
- removed net P1_03: RYS5.1
- removed net P1_06: RYS50.1
- removed net P1_07: RYS10.1
- removed net P6_00: RYS52.1
- removed net P6_01: RYS12.1
- removed net P6_02: RYS54.1
- removed net P6_03: RYS14.1
- removed net P6_04: RYS56.1
- removed net P6_05: RYS16.1
- removed net P6_06: RYS58.1
- removed net P6_07: RYS18.1
- removed net P8_00: RYS2.1
- removed net P8_01: RYS42.1
- removed net P8_02: RYS1.1
- new net P1: J2.P$1, RYS40.1
- new net P10: J2.P$10, RYS7.1
- new net P11: J2.P$11, RYS50.1
- new net P12: J2.P$12, RYS10.1
- new net P13: J2.P$13, RYS52.1
- new net P14: J2.P$14, RYS12.1
- new net P15: J2.P$15, RYS54.1
- new net P16: J2.P$16, RYS14.1
- new net P17: J2.P$17, RYS56.1
- new net P18: J2.P$18, RYS16.1
- new net P19: J2.P$19, RYS58.1
- new net P2: J2.P$2, RYS1.1
- new net P20: J2.P$20, RYS18.1
- new net P3: J2.P$3, RYS42.1
- new net P4: J2.P$4, RYS2.1
- new net P5: J2.P$5, RYS44.1
- new net P6: J2.P$6, RYS3.1
- new net P7: J2.P$7, RYS46.1
- new net P8: J2.P$8, RYS5.1
- new net P9: J2.P$9, RYS48.1
