File: S7G2_Titan_Teknic/Titan_v1p7.brd (EAGLE design)
At the start: 115 x 135 mm, 241 parts, among them J1 SD_CARD, J10 20-pos, J11 2-pos, J12 2-pos, J15 2-pos, J16 2-pos, J19 2-pos, J2 4-pos, J20 2-pos, J23 2-pos, J24 2-pos, J3 10-pos, J4 20-pos, J5 10-pos, J6 USB-A, J7 USB-B-Micro, J8 40-pos, J9 10-pos, U1 KSZ8081_QFN_24, U10 NPN, U11 NPN, U12 NPN, U13 NPN, U14 NPN, U15 NPN, U16 NPN, U17 NPN, U2 AP2151DWG-7, U22 NPN, U23 NPN, U24 NPN, U25 NPN, U26 NPN, U27 NPN, U3 S7G2LQFP176, U34 NPN, U35 NPN, U36 NPN, U37 NPN, U38 NPN, U39 NPN, U46 NPN, U47 NPN, U48 NPN, U49 NPN, U50 NPN, U51 NPN, U58 NPN, U59 NPN, U6 NPN, U60 NPN, U61 NPN, U62 NPN, U63 NPN, U7 NPN, U70 NPN, U71 NPN, U72 NPN, U73 NPN, U74 NPN, U75 NPN, X1 25MHz, X2 24MHz, X3 32.768KHz

Commit message: Update
Parts:
- removed J8: 40-pos, 3D_MIG_Controller:HEADER_2_X_20_.1_INCH
- added J27, J28, J31, J32, J35, J36, J37, J38: 2-pos, 3D_MIG_Controller:2_3.81MM_PITCH
- J10: value 20-pos -> 2-pos; device 3D_MIG_Controller:2_X_10_.1_INCH -> 3D_MIG_Controller:2_3.81MM_PITCH
- J9: value 10-pos -> 2-pos; device 3D_MIG_Controller:2X5 -> 3D_MIG_Controller:2_3.81MM_PITCH
- moved J10 102.1 mm to (106.6, 131.1), turned to 180 degrees
- moved J9 47.9 mm to (99.1, 4.00), turned to 0 degrees
- moved J12 5.40 mm to (69.1, 4.00)
- moved J19 5.40 mm to (79.1, 4.00)
- moved J20 5.40 mm to (89.1, 4.00)
- moved J11 5.40 mm to (59.1, 4.00)
- moved J3 3.69 mm to (56.8, 77.4)
- moved J16 3.21 mm to (111.2, 34.3)
- moved LED5 3.21 mm to (64.2, 37.5)
- moved R31 3.21 mm to (64.2, 34.0)
- moved R32 3.21 mm to (64.2, 45.8)
- moved U$1 3.21 mm to (71.1, 48.5)
- moved U$2 3.21 mm to (71.1, 37.0)
- moved U$7 3.21 mm to (71.1, 24.9)
- moved U6 3.21 mm to (62.9, 52.8)
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Connections:
- removed net P2_00: J10.P$13, U3.69
- removed net P2_01: J10.P$14, U3.68
- removed net P2_02: J4.P$9, U3.54
- removed net P2_03: J9.1, U3.53
- removed net P2_04: J9.3, U3.52
- removed net P2_05: J9.5, U3.51
- removed net P2_06: J9.7, U3.50
- removed net P2_07: J9.9, U3.49
- removed net P3_03: J10.P$2, U3.85
- removed net P3_04: J10.P$4, U3.82
- removed net P3_05: J10.P$6, U3.81
- removed net P3_06: J10.P$1, U3.80
- removed net P3_07: J10.P$3, U3.79
- removed net P3_09: J10.P$5, U3.77
- removed net P3_10: J10.P$7, U3.76
- removed net P3_11: J10.P$8, U3.75
- removed net P3_12: J10.P$9, U3.74
- removed net P3_13: J10.P$20, U3.55
- removed net P3_14: J10.P$17, U3.56
- removed net P3_15: J10.P$18, U3.57
- removed net P9_00: J10.P$16, U3.58
- removed net P9_01: J10.P$15, U3.59
- removed net P9_05: J10.P$10, U3.73
- removed net P9_06: J10.P$11, U3.72
- removed net P9_07: J10.P$12, U3.71
- removed net P9_08: U3.70
- new net ESTOP: J9.P$1, U3.69
- new net LS_01: J11.P$1, U3.50
- new net LS_02: J12.P$1, U3.51
- new net LS_03: J19.P$1, U3.53
- new net LS_04: J20.P$1, U3.54
- new net P$9: J4.P$9
- net A_A_DIR: now also U3.75
- net A_A_ENABLE: now also U3.74
- net A_A_HLFB_OUT: now also U3.77
- net A_A_STEP: now also U3.76
- net A_B_DIR: now also U3.80
- net A_B_ENABLE: now also U3.79
- net A_B_HLFB_OUT: now also U3.82
- net A_B_STEP: now also U3.81
- net C_A_DIR: now also U3.58
- net C_A_ENABLE: now also U3.57
- net C_A_HLFB_OUT: now also U3.68
- net C_A_STEP: now also U3.59
- net C_B_DIR: now also U3.71
- net C_B_ENABLE: now also U3.70
- net C_B_HLFB_OUT: now also U3.73
- net C_B_STEP: now also U3.72
- net GND: no longer J10.P$19, J8.P$1, J9.10, J9.2, J9.4, J9.6, J9.8
- net IIC_1_SCL: no longer J8.P$5
- net IIC_1_SDA: no longer J8.P$6
- net INT_MI_01: no longer J8.P$39
- net INT_MI_02: no longer J8.P$40
- net INT_MI_03: no longer J8.P$9
- net INT_MI_04: no longer J8.P$10
- net P1_02: no longer J8.P$7
- net P1_03: no longer J8.P$8
- net P1_06: no longer J8.P$11
- net P1_07: no longer J8.P$12
- net P1_11: no longer J8.P$38
- net P1_12: no longer J8.P$37
- net P1_13: no longer J8.P$36
- net P1_14: no longer J8.P$35
- net P1_15: no longer J8.P$34
- net P6_00: no longer J8.P$13
- net P6_01: no longer J8.P$14
- net P6_02: no longer J8.P$15
- net P6_03: no longer J8.P$16
- net P6_04: no longer J8.P$17
- net P6_05: no longer J8.P$18
- net P6_06: no longer J8.P$19
- net P6_07: no longer J8.P$20
- net P6_08: no longer J8.P$33
- net P6_09: no longer J8.P$32
- net P6_10: no longer J8.P$31
- net P6_11: no longer J8.P$30
- net P6_12: no longer J8.P$29
- net P6_13: no longer J8.P$28
- net P6_14: no longer J8.P$27
- net P6_15: no longer J8.P$26
- net P8_00: no longer J8.P$4
- net P8_01: no longer J8.P$3
- net P8_02: no longer J8.P$2
- net PA_00: no longer J8.P$21
- net PA_01: no longer J8.P$22
- net PA_08: no longer J8.P$25
- net PA_09: no longer J8.P$24
- net PA_10: no longer J8.P$23
- net RELAY_1: now also U3.56
- net RELAY_2: now also U3.55
- net RELAY_3: now also U3.52
- net RELAY_4: now also U3.49
- net VDD12: now also J10.P$1, J10.P$2, J11.P$2, J12.P$2, J19.P$2, J20.P$2, J9.P$2
Routing:
- net VDD12: track 271.1 -> 557.3 mm
- net ESTOP: track 0.00 -> 100.4 mm, vias 0 -> 2
- net LS_04: track 0.00 -> 85.7 mm
- net A_A_HLFB_OUT: track 0.00 -> 81.9 mm
- net A_A_STEP: track 0.00 -> 79.7 mm, vias 0 -> 1
- net A_A_DIR: track 0.00 -> 76.2 mm, vias 0 -> 1
- net LS_03: track 0.00 -> 75.4 mm
- net A_A_ENABLE: track 0.00 -> 74.3 mm, vias 0 -> 1
- net C_A_HLFB_OUT: track 0.00 -> 73.4 mm
- net C_A_STEP: track 0.00 -> 66.9 mm, vias 0 -> 1
- net C_A_DIR: track 0.00 -> 64.4 mm, vias 0 -> 1
- net A_B_HLFB_OUT: track 0.00 -> 63.6 mm
- net LS_02: track 0.00 -> 63.6 mm
- net A_B_STEP: track 0.00 -> 61.3 mm, vias 0 -> 1
- net C_A_ENABLE: track 0.00 -> 61.1 mm, vias 0 -> 1
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Other:
- board text removed: "39"
- board text removed: "40"
