File: S7G2_Titan_Teknic/Titan_Teknic_v1p00.brd (EAGLE design)
At the start: 115 x 135 mm, 303 parts, among them J1 SD_CARD, J10 2-pos, J11 2-pos, J12 2-pos, J15 2-pos, J16 2-pos, J19 2-pos, J2 4-pos, J20 2-pos, J23 2-pos, J24 2-pos, J27 2-pos, J28 2-pos, J3 10-pos, J31 2-pos, J32 2-pos, J35 2-pos, J36 2-pos, J37 2-pos, J38 2-pos, J4 20-pos, J5 10-pos, J6 USB-A, J7 USB-B-Micro, J9 2-pos, U1 KSZ8081_QFN_24, U10 NPN, U11 NPN, U12 NPN, U13 NPN, U14 NPN, U15 NPN, U16 NPN, U17 NPN, U18 NPN, U19 NPN, U2 AP2151DWG-7, U20 NPN, U21 NPN, U22 NPN, U23 NPN, U24 NPN, U25 NPN, U26 NPN, U27 NPN, U28 NPN, U29 NPN, U3 S7G2LQFP176, U30 NPN, U34 NPN, U35 NPN, U36 NPN, U37 NPN, U38 NPN, U39 NPN, U46 NPN, U47 NPN, U48 NPN, U49 NPN, U5 NPN, U50 NPN, U51 NPN, U58 NPN, U59 NPN, U6 NPN, U60 NPN, U61 NPN, U62 NPN, U63 NPN, U7 NPN, U70 NPN, U71 NPN, U72 NPN, U73 NPN, U74 NPN, U75 NPN, U8 NPN, U9 NPN, X1 25MHz, X2 24MHz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

Commit message: Updated design
Parts:
- removed J32, J35, J36, J37, J38: 2-pos, 3D_MIG_Controller:2_3.81MM_PITCH
- removed J5: 10-pos, 3D_MIG_Controller:2X5
- added J39: (no value), 3D_MIG_Controller:2_X_10_.1_INCH
- added R102, R103, R104, R105, R106, R107, R108, R25, R26, R27: 100K, 3D_MIG_Controller:0402
- moved J1 5.80 mm to (7.21, 91.0), flipped to the bottom, turned to 90 degrees
- moved J8 2.80 mm to (3.70, 110.9)
- moved J4 1.35 mm to (5.00, 40.0)
- moved C20 0.91 mm to (25.2, 64.8)
Connections:
- removed net N$72: J32.P$2
- removed net N$73: J32.P$1
- removed net N$87: J8.P$1
- removed net N$93: J8.P$10
- removed net N$94: J8.P$8
- removed net N$95: J8.P$6
- removed net N$96: J8.P$4
- removed net N$97: J8.P$2
- removed net P$9: J4.P$9
- net GND: now also J39.P$1, J39.P$11, J39.P$13, J39.P$15, J39.P$17, J39.P$19, J39.P$3, J39.P$5, J39.P$7, J39.P$9
- net IIC_1_SCL: now also J8.P$8; no longer J8.P$3
- net IIC_1_SDA: now also J8.P$7; no longer J8.P$5
- net NC: now also J8.P$6
- net P0_02: now also J39.P$20, R25.P$1; no longer J5.1
- net P0_03: now also J39.P$18, R26.P$1; no longer J5.3
- net P0_04: now also J39.P$16, R27.P$1; no longer J5.5
- net P0_05: now also J39.P$14, R102.P$1; no longer J5.7
- net P0_06: now also J39.P$12, R103.P$1; no longer J5.9
- net P0_07: now also J39.P$10, R104.P$1; no longer J5.10
- net P0_08: now also J39.P$8, R105.P$1; no longer J5.8
- net P0_09: now also J39.P$6, R106.P$1; no longer J5.6
- net P0_14: now also J39.P$4, R107.P$1; no longer J5.4
- net P0_15: now also J39.P$2, R108.P$1; no longer J5.2
- net P1_02: now also J8.P$10; no longer J8.P$7
- net P4_02: now also J4.P$9
- net P8_00: now also J8.P$5
- net P8_01: now also J8.P$3
- net P8_02: now also J8.P$4
- net P8_03: now also J8.P$1
- net P8_04: now also J8.P$2
- net VDD: now also R102.P$2, R103.P$2, R104.P$2, R105.P$2, R106.P$2, R107.P$2, R108.P$2, R25.P$2, R26.P$2, R27.P$2
- net VDD12: now also J13.1, J14.1, J17.1, J18.1, J21.1, J22.1, J25.1, J26.1, J29.1, J30.1, J33.1, J34.1
Routing:
- net VDD12: track 645.0 -> 598.5 mm
- net P8_00: track 0.00 -> 45.6 mm
- net P8_02: track 0.00 -> 45.5 mm
- net P8_04: track 0.00 -> 45.0 mm
- net P8_01: track 0.00 -> 43.3 mm
- net VDD: track 356.9 -> 399.5 mm
- net P8_03: track 0.00 -> 42.1 mm
- net P4_02: track 0.00 -> 22.8 mm
- net SD1_WP: track 24.8 -> 45.5 mm, vias 0 -> 1
- net P0_06: track 11.4 -> 29.9 mm
- net P0_07: track 14.1 -> 32.2 mm
- net P0_09: track 20.8 -> 36.7 mm, vias 1 -> 0
- net P0_08: track 19.1 -> 34.4 mm
- net P0_05: track 13.0 -> 27.9 mm
- net SD1_DAT2: track 35.5 -> 50.0 mm, vias 2 -> 1
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- added copper zone on layer 1, net GND
- added copper zone on layer 16, net GND

Commit message: Updated
Parts:
- U$1, U$2, U$7, U$8: value RELAY_KYOTO_KF0604D -> (none)
- moved R73 5.59 mm to (93.2, 12.4)
- moved R79 5.45 mm to (102.7, 12.3)
- moved R58 5.32 mm to (103.1, 104.6)
- moved R36 5.31 mm to (73.2, 12.3)
- moved R55 5.31 mm to (82.7, 12.3)
- moved R76 5.30 mm to (103.0, 114.3)
- moved R97 5.24 mm to (103.1, 123.7)
- moved R33 5.12 mm to (62.6, 12.2)
- moved R74 4.23 mm to (93.7, 14.5), turned to 270 degrees
- moved R80 4.23 mm to (103.3, 14.5), turned to 270 degrees
- moved R53 4.03 mm to (73.8, 14.5), turned to 270 degrees
- moved R77 4.01 mm to (101.0, 114.9), turned to 0 degrees
- moved R56 3.93 mm to (83.3, 14.4), turned to 270 degrees
- moved R98 3.83 mm to (101.0, 124.3), turned to 0 degrees
- moved R59 3.45 mm to (101.4, 105.2), turned to 0 degrees
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Routing:
- net LS_01_RET: track 12.5 -> 0.00 mm, vias 1 -> 0
- net LS_01: track 51.0 -> 43.8 mm, vias 1 -> 0
- net ESTOP: track 98.2 -> 91.7 mm, vias 3 -> 2
- net LS_04: track 85.2 -> 79.6 mm, vias 1 -> 0
- net LS_05: track 93.7 -> 88.1 mm
- net LS_03: track 73.8 -> 68.5 mm, vias 1 -> 0
- net LS_06: track 103.0 -> 97.7 mm
- net LS_02: track 61.7 -> 56.7 mm, vias 1 -> 0
- net LS_03_RET: track 12.1 -> 7.60 mm, vias 1 -> 0
- net LS_02_RET: track 12.2 -> 7.67 mm, vias 1 -> 0
- net LS_07: track 110.6 -> 106.2 mm
- net LS_04_RET: track 11.9 -> 7.60 mm, vias 1 -> 0
- net ESTOP_RET: track 11.9 -> 7.77 mm, vias 1 -> 0
- net N$11: track 1.56 -> 0.00 mm
- net N$10: track 1.31 -> 0.00 mm
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Other:
- board text added: "1,2"
- board text added: "E-Stop"
- board text added: "LS-1"
- board text added: "LS-2"
- board text added: "LS-3"
- board text added: "LS-4"
- board text added: "LS-5"
- board text added: "LS-6"
- board text added: "LS-7"
- board text added: "LS-8"
- board text added: "LS-9"
- board text added: "P0_01 , P0_00"
- board text added: "VDD5"
- board text removed: "+12V"
- board text removed: "1"
- board text removed: "10"
- board text removed: "19"
- board text removed: "2"
- board text removed: "20"
- board text removed: "3.3V"
- board text removed: "5V"
- board text removed: "9"
- board text removed: "Titan"
