File: Welder PSU/HW05.05/Welder_PSU_Backup.sch (EAGLE design)
At the start: 483 parts, among them IC1 UCC28951PWR, IC100 PC817, IC2 LMV641, IC301 LMV641, IC302 LMV641, IC306 UCC21710, IC307 UCC21710, IC308 MAX764CSA+, IC309 MAX764CSA+, IC310 UCC21710, IC311 UCC21710, IC312 LM317AEMP, IC313 LM317AEMP, IC401 CSTNE8M00G520000R0, IC500 SN65HVD3082EDR, K100 PANASONIC_ALFG2PF09PANASONIC_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, K101 PANASONIC_ALFG2PF09PANASONIC_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, Q1 2N7002, Q100 BC640TA, Q101 KSD1616AYTA, Q2 2N7002, Q300 2N7002, Q306 2N7002, Q307 2N7002, Q308 2N7002, Q309 2N7002, Q310 2N7002, Q500 DMP6185SEQ-13, Q501 BC817, Q502 DMP6185SEQ-13, Q503 BC817, Q504 DMP6185SEQ-13, Q505 BC817, Q506 BC817, Q507 BC817, T1 CST206-2A, T300 IHW20N120R5, T301 IHW20N120R5, T303 IHW20N120R5, T304 IHW20N120R5, T500 2N7002, T501 2N7002, T502 2N7002, U2 R7FA6M5BG3CFBLQFP-144-M, U300 PAD_3MMX6MM, U301 PAD_3MMX6MM, X1 WF2549-2WS05S0B01, X100 01020071Z, X101 01020071Z, X200 726386-2TE_726386-2, X201 726386-2TE_726386-2, X202 726386-2TE_726386-2, X203 726386-2TE_726386-2, X204 MOLEX_206832-0601MOLEX_206832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, X205 MOLEX_206832-0601MOLEX_206832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, X400 2304-6111-TP, X401 2304-6111-TP, X402 2304-6111-TP

Commit message: Welder PSU HW05.05 Altium -> Eagle Ongoing
Recreating schematic done, Netlisting Ongoing
Parts:
- removed C448: 1uF/35V, Labops_Lib_AH:C_0603EIA0603
- removed C449, C500, C501, C502, C503, C504, C505, C506: 100nF/50V, Labops_Lib_AH:C_0603EIA0603
- removed IC500: SN65HVD3082EDR, Labops_Lib_AH:SN65HVD3082EDR
- removed Q500, Q502, Q504: DMP6185SEQ-13, Labops_Lib_AH:DMP6185SEQ-13
- removed Q501, Q503, Q505, Q506, Q507: BC817, Labops_Lib_AH:BC817
- removed R500, R501, R503, R505, R507, R510, R512, R514, R515, R516, R519: 10K 1%, Labops_Lib_AH:R_0603
- removed R502, R506, R508, R511, R513, R517, R518, R521, R523, R524, R528: 100R 1%, Labops_Lib_AH:R_0603
- removed R504, R509: 1K 1%, Labops_Lib_AH:R_0603
- removed R520, R522, R525: 470R 1%, Labops_Lib_AH:R_0603
- removed R526, R527: 0R 1%, Labops_Lib_AH:R_0603
- removed T500, T501, T502: 2N7002, Labops_Lib_AH:2N7002
- removed V500, V501, V502, V503, V504: 0603ESDA-24NSMD, Labops_Lib_AH:0603ESDA-24NSMD
- removed X1: WF2549-2WS05S0B01, Labops_Lib_AH:WF2549-2WS05S0B01
Connections:
- net DGB_SWDCLK_TCK renamed N$124
- net DO_7SEG_BCD_D renamed N$120
- removed net /COMM_RX_EN: R520.2
- removed net BCD_A: C500.1, Q501.C
- removed net BCD_B: C501.1, Q503.C
- removed net BCD_C: C502.1, Q505.C
- removed net BCD_D: C506.1, Q507.C
- removed net COMM_TX_EN: R522.2
- removed net DBG_TDI: X1.1
- removed net DGB_SWDIO_TCK: X1.7
- removed net DGB_SWDIO_TDO: U2B.P109/TDO
- removed net DGB_SWDIO_TMS: U2B.P108/TMS/SWDIO, X1.5
- removed net DGB_SWO_TDO: X1.3
- removed net DISP1_VCC: Q504.DRAIN, V502.2
- removed net DISP2_VCC: Q502.DRAIN, V501.2
- removed net DISP3_VCC: Q500.DRAIN, V500.2
- removed net DO_7SEG_BCD_A: R504.2, U2A.P301
- removed net DO_7SEG_BCD_B: R509.2, U2A.P302
- removed net DO_7SEG_BCD_C: R513.2, U2A.P303
- removed net DO_7SEG_DISP1_EN: R517.2, U2A.P305
- removed net DO_7SEG_DISP2_EN: R508.2, U2A.P306
- removed net DO_7SEG_DISP3_EN: R502.2, U2A.P307
- removed net D_7SEG_BCD_D: R524.2
- removed net N$120 (its old number): Q506.B, R516.2
- removed net N$124 (its old number): Q501.E, R506.2
- removed net N$125: X1.8
- removed net N$127: IC500.DE, R522.1
- removed net N$128: IC500.D, R525.1
- removed net N$129: Q503.B, R509.1
- removed net N$131: Q503.E, R511.2
- removed net N$133: Q505.B, R513.1
- removed net N$135: Q505.E, R518.2
- removed net N$137: Q507.B, R524.1
- removed net N$139: Q507.E, R528.2
- removed net N$140: R508.1, R510.2, T501.G
- removed net N$141: R502.1, R503.2, T500.G
- removed net N$142: R501.1, T500.D
- removed net N$143: Q500.GATE, R500.1, R501.2
- removed net N$145: R507.1, T501.D
- removed net N$147: Q502.GATE, R505.1, R507.2
- removed net N$150: R517.1, R519.2, T502.G
- removed net N$151: R514.1, T502.D
- removed net N$152: Q504.GATE, R512.1, R514.2
- removed net RS485-A: IC500.A, R523.1, R527.1, V503.2
- removed net RS485-A-NEXT: R527.2
- removed net RS485-B: IC500.B, R521.1, R526.1, V504.2
- removed net RS485-B-NEXT: R526.2
- removed net UART_RX: Q506.C, R515.2
- removed net UART_TX: R525.2
- new net N$118: U2A.P306
- new net N$122: U2A.P302
- net GND: no longer C448.1, C449.1, C500.2, C501.2, C502.2, C503.1, C504.1, C505.1, C506.2, IC500.GND, R503.1, R506.1, R510.1, R511.1, R518.1, R519.1, R528.1, T500.S, T501.S, T502.S, V500.1, V501.1, V502.1, V503.1, V504.1, X1.10, X1.6
- net N$117: now also U2A.P307; no longer C505.2, R521.2, R523.2
- net N$119: now also U2A.P305; no longer IC500.R, Q506.E
- net N$121: now also U2A.P303; no longer Q501.B, R504.1
- net N$123: now also U2A.P301; no longer IC500./RE, R520.1
- net NRST: no longer X1.9
- net V_3V3: no longer C448.2, C449.2, C503.2, R515.1, R516.1, X1.2, X1.4
- net V_5V0: no longer C504.2, IC500.VCC, Q500.SOURCE, Q502.SOURCE, Q504.SOURCE, R500.2, R505.2, R512.2
