File: Callisto_Limit_Switch_PX/Callisto_Limit_Switch_PX.brd (EAGLE design)
At the start: 50 x 40 mm, 6 parts, among them J1 RJ45_TH_VERT, J2 4-pos, U1 NPN

Commit message: LS Update.
Connections:
- removed net IO_SIGNAL_2: J1.4
- removed net VDD5: J1.8
- net VDD: no longer J1.5
Routing:
- net VDD: track 14.0 -> 1.80 mm
Changed lines of the file:
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@@
 <wire x1="21.7" y1="26.7" x2="17.04" y2="22.04" width="0.8128" layer="16"/>
-</signal>
-<signal name="VDD5">
-<contactref element="J1" pad="8"/>
 </signal>
 <signal name="VDD-12">
@@
 </signal>
 <signal name="VDD">
-<contactref element="J1" pad="5"/>
 <contactref element="U1" pad="3"/>
-<wire x1="36.82" y1="20.635" x2="24.665" y2="20.635" width="0.254" layer="16"/>
 <wire x1="24.665" y1="20.635" x2="24.6" y2="20.7" width="0.254" layer="16"/>
 <via x="24.6" y="20.7" extent="1-16" drill="0.35"/>
@@
 <wire x1="24.61" y1="20.69" x2="24.61" y2="18.9963" width="0.254" layer="1"/>
 </signal>
-<signal name="IO_SIGNAL_2">
-<contactref element="J1" pad="4"/>
-</signal>
 <signal name="N$1">
