File: Callisto_Limit_Switch_PX/Callisto_Limit_Switch_PX.sch (EAGLE design)
At the start: 6 parts, among them J1 RJ45_TH_VERT, J2 4-pos, U1 NPN

Commit message: LS Update.
Connections:
- removed net IO_SIGNAL_2: J1.4
- removed net VDD5: J1.8
- net VDD: no longer J1.5
Changed lines of the file:
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@@
-</segment>
-</net>
-<net name="VDD5" class="0">
-<segment>
-<pinref part="J1" gate="G$1" pin="8"/>
-<wire x1="20.32" y1="25.4" x2="22.86" y2="25.4" width="0.1524" layer="91"/>
-<label x="22.86" y="25.4" size="1.016" layer="95" xref="yes"/>
 </segment>
 </net>
@@
 <net name="VDD" class="0">
 <segment>
-<pinref part="J1" gate="G$1" pin="5"/>
-<wire x1="20.32" y1="17.78" x2="22.86" y2="17.78" width="0.1524" layer="91"/>
-<label x="22.86" y="17.78" size="1.016" layer="95" xref="yes"/>
-</segment>
-<segment>
 <pinref part="U1" gate="A" pin="C(3)"/>
 <wire x1="76.2" y1="27.34" x2="76.2" y2="38.1" width="0.1524" layer="91"/>
@@
 </segment>
 </net>
-<net name="IO_SIGNAL_2" class="0">
-<segment>
-<pinref part="J1" gate="G$1" pin="4"/>
-<wire x1="20.32" y1="15.24" x2="22.86" y2="15.24" width="0.1524" layer="91"/>
-<label x="22.86" y="15.24" size="1.016" layer="95" xref="yes"/>
-</segment>
-</net>
