File: Teknic_motor_IO/Teknic_motor_io.brd (EAGLE design)
At the start: 60 x 45 mm, 26 parts, among them J1 4-pos, J2 4-pos, J3 10-pos, J4 4-pos, J5 10-pos, J8 10-pos, U10 NPN, U11 NPN, U12 NPN, U7 NPN, U8 NPN, U9 NPN

Commit message: Updated motor IO board.
Parts:
- removed J5: 10-pos, 3D_MIG_Controller:2X5
- removed J6: (no value), 3D_MIG_Controller:CON_39281083
- removed R13, R17, R18: 1k, 3D_MIG_Controller:0805
- removed R14, R15, R16: 33, 3D_MIG_Controller:0805
- removed U7, U8, U9: NPN, 3D_MIG_Controller:SOT323
- added J10, J12, J9: (no value), 3D_MIG_Controller:CON_39281083
- added R10, R11, R25, R29, R3, R30, R32, R41, R45, R46, R48, R49, R53, R54, R56, R57, R61, R62, R64, R7, R73, R77, R78, R8, R80: 1K0, 3D_MIG_Controller:0402
- added R12, R26, R27, R28, R31, R4, R42, R43, R44, R47, R5, R50, R51, R52, R55, R58, R59, R6, R60, R63, R74, R75, R76, R79, R9: 33R0, 3D_MIG_Controller:0402
- added U13, U14, U15, U16, U2, U21, U22, U23, U24, U25, U26, U27, U28, U29, U3, U30, U31, U32, U37, U38, U39, U4, U40, U5, U6: NPN, 3D_MIG_Controller:SOT323
- J2, J4: value 4-pos -> (none); device 3D_MIG_Controller:1X4_3.81MM_PITCH -> 3D_MIG_Controller:CON_39281083
- J3: value 10-pos -> (none); device 3D_MIG_Controller:2X5 -> 3D_MIG_Controller:CON_39281083
- J8: value 10-pos -> 40-pos; device 3D_MIG_Controller:2X5 -> 3D_MIG_Controller:HEADER_2_X_20_.1_INCH
- R19, R23: value 1k -> 33R0; device 3D_MIG_Controller:0805 -> 3D_MIG_Controller:0402
- R20: value 33 -> 33R0; device 3D_MIG_Controller:0805 -> 3D_MIG_Controller:0402
- R21, R22: value 33 -> 1K0; device 3D_MIG_Controller:0805 -> 3D_MIG_Controller:0402
- R24: value 1k -> 1K0; device 3D_MIG_Controller:0805 -> 3D_MIG_Controller:0402
- moved J8 75.9 mm to (30.0, 88.5), turned to 0 degrees
- moved J2 56.8 mm to (4.60, 60.5), turned to 90 degrees
- moved R20 56.1 mm to (42.2, 78.7), flipped to the top, turned to 0 degrees
- moved J3 54.5 mm to (34.6, 60.5), turned to 90 degrees
- moved U12 52.7 mm to (33.4, 78.1), turned to 180 degrees
- moved U10 51.7 mm to (38.9, 78.1), turned to 180 degrees
- moved U11 51.6 mm to (41.6, 78.1), turned to 180 degrees
- moved J1 49.9 mm to (9.20, 4.00), turned to 0 degrees
- moved R23 45.9 mm to (34.1, 78.7), flipped to the top
- moved R19 45.7 mm to (39.5, 78.7), flipped to the top
- moved J4 43.5 mm to (4.50, 37.4), turned to 90 degrees
- moved R21 41.9 mm to (37.0, 64.8), turned to 0 degrees
- moved R24 40.5 mm to (37.3, 73.0)
- moved R22 38.0 mm to (36.9, 60.3), turned to 0 degrees
- moved J7 25.7 mm to (19.5, 37.4), turned to 90 degrees
Connections:
- removed net A_DIR: J2.P$2, J3.3, J3.4, R15.1
- removed net A_ENABLE: J2.P$3, J3.5, J3.6, R16.1
- removed net A_HLFB_OUT: J6.5
- removed net A_MI_DIR: J6.7, R17.1, U8.3
- removed net A_MI_ENABLE: J6.8, R18.1, U9.3
- removed net A_MI_STEP: J6.6, R13.1, U7.3
- removed net A_STEP: J2.P$1, J3.1, J3.2, R14.1
- removed net B_DIR: J4.P$2, J5.3, J5.4, R21.1
- removed net B_ENABLE: J4.P$3, J5.5, J5.6, R22.1
- removed net B_HLFB_OUT: J7.5
- removed net B_MI_DIR: J7.7, R23.1, U11.3
- removed net B_MI_ENABLE: J7.8, R24.1, U12.3
- removed net B_MI_STEP: J7.6, R19.1, U10.3
- removed net B_STEP: J4.P$1, J5.1, J5.2, R20.1
- removed net N$10: R15.2, U8.1
- removed net N$11: R16.2, U9.1
- removed net N$12: R14.2, U7.1
- new net IIC_1_SCL: J8.P$5
- new net IIC_1_SDA: J8.P$6
- new net INT_MI_03: J8.P$9
- new net INT_MI_04: J8.P$10
- new net LS_07: J8.P$40
- new net LS_08: J8.P$39
- new net LS_09: J8.P$38
- new net M1_DIR: J8.P$15, R5.P$1
- new net M1_ENABLE: J8.P$16, R6.P$1
- new net M1_HLFB: R9.P$1
- new net M1_STEP: J8.P$14, R4.P$1
- new net M2_DIR: J8.P$18, R27.P$1
- new net M2_ENABLE: J8.P$19, R28.P$1
- new net M2_HLFB: R31.P$1
- new net M2_STEP: J8.P$17, R26.P$1
- new net M3_DIR: J8.P$21, R51.P$1
- new net M3_ENABLE: J8.P$22, R52.P$1
- new net M3_HLFB: R55.P$1
- new net M3_STEP: J8.P$20, R50.P$1
- new net M4_DIR: J8.P$24, R43.P$1
- new net M4_ENABLE: J8.P$25, R44.P$1
- new net M4_HLFB: R47.P$1
- new net M4_STEP: J8.P$23, R42.P$1
- new net M5_DIR: J8.P$27, R19.P$1
- new net M5_ENABLE: J8.P$28, R20.P$1
- new net M5_HLFB: R23.P$1
- new net M5_STEP: J8.P$26, R12.P$1
- new net M6_DIR: J8.P$30, R59.P$1
- new net M6_ENABLE: J8.P$31, R60.P$1
- new net M6_HLFB: R63.P$1
- new net M6_STEP: J8.P$29, R58.P$1
- new net M7_DIR: J8.P$33, R75.P$1
- new net M7_ENABLE: J8.P$34, R76.P$1
- new net M7_HLFB: R79.P$1
- new net M7_STEP: J8.P$32, R74.P$1
- new net M8_DIR: J8.P$36
- new net M8_ENABLE: J8.P$37
- new net M8_STEP: J8.P$35
- new net MR_DIR: J10.7, J12.7, J2.7, J3.7, J4.7, J7.7, J9.7, R21.P$1, R29.P$1, R45.P$1, R53.P$1, R61.P$1, R7.P$1, R77.P$1, U10.3, U14.3, U22.3, U26.3, U3.3, U30.3, U38.3
- new net MR_ENABLE: J10.8, J12.8, J2.8, J3.8, J4.8, J7.8, J9.8, R22.P$1, R30.P$1, R46.P$1, R54.P$1, R62.P$1, R78.P$1, R8.P$1, U11.3, U15.3, U23.3, U27.3, U31.3, U39.3, U4.3
- new net MR_HLFB: J10.5, J12.5, J2.5, J3.5, J4.5, J7.5, J9.5, R10.P$1, R24.P$1, R32.P$1, R48.P$1, R56.P$1, R64.P$1, R80.P$1, U12.3, U16.3, U24.3, U28.3, U32.3, U40.3, U5.3
- new net MR_STEP: J10.6, J12.6, J2.6, J3.6, J4.6, J7.6, J9.6, R11.P$1, R25.P$1, R3.P$1, R41.P$1, R49.P$1, R57.P$1, R73.P$1, U13.3, U2.3, U21.3, U25.3, U29.3, U37.3, U6.3
- new net N$16: R31.P$2, U16.1
- new net N$2: R5.P$2, U3.1
- new net N$21: R43.P$2, U22.1
- new net N$22: R44.P$2, U23.1
- new net N$23: R42.P$2, U21.1
- new net N$24: R47.P$2, U24.1
- new net N$25: R51.P$2, U26.1
- new net N$26: R52.P$2, U27.1
- new net N$27: R50.P$2, U25.1
- new net N$28: R55.P$2, U28.1
- new net N$29: R59.P$2, U30.1
- new net N$3: R6.P$2, U4.1
- new net N$30: R60.P$2, U31.1
- new net N$31: R58.P$2, U29.1
- new net N$32: R63.P$2, U32.1
- new net N$37: R75.P$2, U38.1
- new net N$38: R76.P$2, U39.1
- new net N$39: R74.P$2, U37.1
- new net N$4: R4.P$2, U2.1
- new net N$40: R79.P$2, U40.1
- new net N$5: R9.P$2, U5.1
- new net N$6: R19.P$2, U10.1
- new net N$7: R20.P$2, U11.1
- new net N$8: R12.P$2, U6.1
- new net N$9: R23.P$2, U12.1
- new net P1_02: J8.P$7
- new net P1_03: J8.P$8
- new net P1_06: J8.P$11
- new net P1_07: J8.P$12
- new net P6_00: J8.P$13
- new net P8_00: J8.P$4
- new net P8_01: J8.P$3
- new net P8_02: J8.P$2
- net GND: now also J8.P$1, U13.2, U14.2, U15.2, U16.2, U2.2, U21.2, U22.2, U23.2, U24.2, U25.2, U26.2, U27.2, U28.2, U29.2, U3.2, U30.2, U31.2, U32.2, U37.2, U38.2, U39.2, U4.2, U40.2, U5.2, U6.2; no longer J2.P$4, J3.10, J3.7, J3.8, J3.9, J4.P$4, J5.10, J5.7, J5.8, J5.9, U7.2, U8.2, U9.2
- net N$13: now also R27.P$2, U14.1; no longer R21.2, U11.1
- net N$14: now also R28.P$2, U15.1; no longer R22.2, U12.1
- net N$15: now also R26.P$2, U13.1; no longer R20.2, U10.1
- net VDD: no longer J8.1, J8.10, J8.2, J8.3, J8.4, J8.5, J8.6, J8.7, J8.8, J8.9
- net VDD12: now also J10.1, J10.2, J10.3, J10.4, J12.1, J12.2, J12.3, J12.4, J2.1, J2.2, J2.3, J2.4, J3.1, J3.2, J3.3, J3.4, J4.1, J4.2, J4.3, J4.4, J9.1, J9.2, J9.3, J9.4, R10.P$2, R11.P$2, R21.P$2, R22.P$2, R24.P$2, R25.P$2, R29.P$2, R3.P$2, R30.P$2, R32.P$2, R41.P$2, R45.P$2, R46.P$2, R48.P$2, R49.P$2, R53.P$2, R54.P$2, R56.P$2, R57.P$2, R61.P$2, R62.P$2, R64.P$2, R7.P$2, R73.P$2, R77.P$2, R78.P$2, R8.P$2, R80.P$2; no longer J6.1, J6.2, J6.3, J6.4, R13.2, R17.2, R18.2, R19.2, R23.2, R24.2
Routing:
- net VDD12: track 68.1 -> 305.6 mm, vias 0 -> 3
- net MR_ENABLE: track 0.00 -> 160.5 mm
- net MR_DIR: track 0.00 -> 135.6 mm
- net MR_STEP: track 0.00 -> 77.4 mm, vias 0 -> 14
- net MR_HLFB: track 0.00 -> 52.7 mm
- net M2_DIR: track 0.00 -> 46.9 mm
- net M2_STEP: track 0.00 -> 45.5 mm
- net M2_ENABLE: track 0.00 -> 42.0 mm
- net M4_DIR: track 0.00 -> 39.8 mm
- net M4_STEP: track 0.00 -> 38.0 mm
- net M6_DIR: track 0.00 -> 38.0 mm
- net VDD: track 38.0 -> 0.00 mm
- net M6_STEP: track 0.00 -> 36.9 mm
- net M4_ENABLE: track 0.00 -> 34.9 mm
- net M6_ENABLE: track 0.00 -> 32.9 mm
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- removed copper zone on layer 1, net GND
- removed copper zone on layer 16, net GND
Other:
- board size 60 x 45 mm -> 60 x 92 mm
- board text added: "A"
- board text added: "C"
- board text added: "W F"
- board text added: "X1"
- board text added: "Y"
- board text added: "Z"

Commit message: Updated headers.
Parts:
- added J11: (no value), 3D_MIG_Controller:CON_39281083
- added J5: 2-pos, 3D_MIG_Controller:2_3.81MM_PITCH
- added R33, R37, R38, R40, R65, R69, R70, R72: 1K0, 3D_MIG_Controller:0402
- added R34, R35, R36, R39, R66, R67, R68, R71: 33R0, 3D_MIG_Controller:0402
- added U17, U18, U19, U20, U33, U34, U35, U36: NPN, 3D_MIG_Controller:SOT323
- J1: value 4-pos -> (none); device 3D_MIG_Controller:1X4_3.81MM_PITCH -> 3D_MIG_Controller:CON_39281083
- moved J3 59.3 mm to (7.10, 8.00)
- moved J12 54.0 mm to (37.1, 8.00)
- moved R73 54.0 mm to (39.7, 16.5)
- moved R74 54.0 mm to (39.3, 26.2)
- moved R75 54.0 mm to (42.0, 26.2)
- moved R76 54.0 mm to (44.7, 26.2)
- moved R77 54.0 mm to (39.5, 12.3)
- moved R78 54.0 mm to (39.4, 7.80)
- moved R79 54.0 mm to (36.6, 26.2)
- moved R80 54.0 mm to (39.8, 20.5)
- moved U37 54.0 mm to (38.6, 25.6)
- moved U38 54.0 mm to (41.4, 25.6)
- moved U39 54.0 mm to (44.1, 25.6)
- moved U40 54.0 mm to (35.9, 25.6)
- moved J1 53.4 mm to (7.10, 57.4), turned to 90 degrees
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Connections:
- removed net IIC_1_SCL: J8.P$5
- removed net IIC_1_SDA: J8.P$6
- removed net INT_MI_03: J8.P$9
- removed net INT_MI_04: J8.P$10
- removed net LS_07: J8.P$40
- removed net LS_08: J8.P$39
- removed net LS_09: J8.P$38
- removed net P1_02: J8.P$7
- removed net P1_03: J8.P$8
- removed net P1_06: J8.P$11
- removed net P1_07: J8.P$12
- removed net P6_00: J8.P$13
- removed net P8_00: J8.P$4
- removed net P8_01: J8.P$3
- removed net P8_02: J8.P$2
- removed net VDD: J1.P$2
- removed net VDD5: J1.P$3
- new net M10_DIR: J8.P$29
- new net M10_ENABLE: J8.P$30
- new net M10_STEP: J8.P$28
- new net M11_DIR: J8.P$32
- new net M11_ENABLE: J8.P$33
- new net M11_STEP: J8.P$31
- new net M12_DIR: J8.P$35
- new net M12_ENABLE: J8.P$36
- new net M12_STEP: J8.P$34
- new net M8_HLFB: R71.P$1
- new net M9_DIR: J8.P$26, R75.P$1
- new net M9_ENABLE: J8.P$27, R76.P$1
- new net M9_HLFB: R79.P$1
- new net M9_STEP: J8.P$25, R74.P$1
- new net N$17: R35.P$2, U18.1
- new net N$18: R36.P$2, U19.1
- new net N$19: R34.P$2, U17.1
- new net N$20: R39.P$2, U20.1
- new net N$33: R67.P$2, U34.1
- new net N$34: R68.P$2, U35.1
- new net N$35: R66.P$2, U33.1
- new net N$36: R71.P$2, U36.1
- net GND: now also J5.P$1, J8.P$37, J8.P$38, J8.P$39, J8.P$40, U17.2, U18.2, U19.2, U20.2, U33.2, U34.2, U35.2, U36.2; no longer J1.P$1, J8.P$1
- net M1_DIR: now also J8.P$2; no longer J8.P$15
- net M1_ENABLE: now also J8.P$3; no longer J8.P$16
- net M1_STEP: now also J8.P$1; no longer J8.P$14
- net M2_DIR: now also J8.P$5, R19.P$1; no longer J8.P$18, R27.P$1
- net M2_ENABLE: now also J8.P$6, R20.P$1; no longer J8.P$19, R28.P$1
- net M2_HLFB: now also R23.P$1; no longer R31.P$1
- net M2_STEP: now also J8.P$4, R12.P$1; no longer J8.P$17, R26.P$1
- net M3_DIR: now also J8.P$8, R27.P$1; no longer J8.P$21, R51.P$1
- net M3_ENABLE: now also J8.P$9, R28.P$1; no longer J8.P$22, R52.P$1
- net M3_HLFB: now also R31.P$1; no longer R55.P$1
- net M3_STEP: now also J8.P$7, R26.P$1; no longer J8.P$20, R50.P$1
- net M4_DIR: now also J8.P$11, R35.P$1; no longer J8.P$24, R43.P$1
- net M4_ENABLE: now also J8.P$12, R36.P$1; no longer J8.P$25, R44.P$1
- net M4_HLFB: now also R39.P$1; no longer R47.P$1
- net M4_STEP: now also J8.P$10, R34.P$1; no longer J8.P$23, R42.P$1
- net M5_DIR: now also J8.P$14, R43.P$1; no longer J8.P$27, R19.P$1
- net M5_ENABLE: now also J8.P$15, R44.P$1; no longer J8.P$28, R20.P$1
- net M5_HLFB: now also R47.P$1; no longer R23.P$1
- net M5_STEP: now also J8.P$13, R42.P$1; no longer J8.P$26, R12.P$1
- net M6_DIR: now also J8.P$17, R51.P$1; no longer J8.P$30, R59.P$1
- net M6_ENABLE: now also J8.P$18, R52.P$1; no longer J8.P$31, R60.P$1
- net M6_HLFB: now also R55.P$1; no longer R63.P$1
- net M6_STEP: now also J8.P$16, R50.P$1; no longer J8.P$29, R58.P$1
- net M7_DIR: now also J8.P$20, R59.P$1; no longer J8.P$33, R75.P$1
- net M7_ENABLE: now also J8.P$21, R60.P$1; no longer J8.P$34, R76.P$1
- net M7_HLFB: now also R63.P$1; no longer R79.P$1
- net M7_STEP: now also J8.P$19, R58.P$1; no longer J8.P$32, R74.P$1
- net M8_DIR: now also J8.P$23, R67.P$1; no longer J8.P$36
- net M8_ENABLE: now also J8.P$24, R68.P$1; no longer J8.P$37
- net M8_STEP: now also J8.P$22, R66.P$1; no longer J8.P$35
- net MR_DIR: now also J1.7, J11.7, R37.P$1, R69.P$1, U18.3, U34.3
- net MR_ENABLE: now also J1.8, J11.8, R38.P$1, R70.P$1, U19.3, U35.3
- net MR_HLFB: now also J1.5, J11.5, R40.P$1, R72.P$1, U20.3, U36.3
- net MR_STEP: now also J1.6, J11.6, R33.P$1, R65.P$1, U17.3, U33.3
- net VDD12: now also J1.1, J1.2, J1.3, J1.4, J11.1, J11.2, J11.3, J11.4, J5.P$2, R33.P$2, R37.P$2, R38.P$2, R40.P$2, R65.P$2, R69.P$2, R70.P$2, R72.P$2; no longer J1.P$4
Routing:
- net VDD12: track 305.6 -> 117.3 mm, vias 3 -> 0
- net M9_DIR: track 0.00 -> 70.4 mm, vias 0 -> 1
- net M9_ENABLE: track 0.00 -> 69.2 mm, vias 0 -> 1
- net M9_STEP: track 0.00 -> 65.7 mm, vias 0 -> 1
- net M3_DIR: track 10.7 -> 63.6 mm, vias 0 -> 1
- net M8_STEP: track 0.00 -> 51.9 mm
- net M3_STEP: track 14.8 -> 62.9 mm, vias 0 -> 1
- net M8_ENABLE: track 0.00 -> 46.6 mm
- net MR_ENABLE: track 160.5 -> 206.3 mm
- net M3_ENABLE: track 13.6 -> 59.4 mm, vias 0 -> 1
- net M8_DIR: track 0.00 -> 45.7 mm
- net MR_DIR: track 135.6 -> 174.3 mm
- net M5_DIR: track 8.18 -> 44.0 mm
- net M5_STEP: track 11.4 -> 42.4 mm
- net M6_ENABLE: track 32.9 -> 63.5 mm, vias 0 -> 1
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Other:
- board text removed: "A"
- board text removed: "C"
- board text removed: "W F"
- board text removed: "X1"
- board text removed: "Y"
- board text removed: "Z"
