File: S7G2_Titan_6L/Titan_6L_v1p3.brd (EAGLE design)
At the start: 70 x 102 mm, 257 parts, among them J1 SD_CARD, J10 CONN_530470410_PICOBLADE_X_4, J12 10-pos, J13 CONN_530470410_PICOBLADE_X_4, J14 CONN_530470410_PICOBLADE_X_4, J15 CONN_530470410_PICOBLADE_X_4, J16 CONN_530470410_PICOBLADE_X_4, J17 CONN_530470410_PICOBLADE_X_4, J18 CONN_530470410_PICOBLADE_X_4, J19 CONN_530470410_PICOBLADE_X_4, J2 4-pos, J20 CONN_530470410_PICOBLADE_X_4, J21 CONN_530470410_PICOBLADE_X_4, J22 CONN_530470410_PICOBLADE_X_4, J24 CONN_530470410_PICOBLADE_X_4, J3 10-pos, J4 20-pos, J5 10-pos, J6 USB-A, J7 USB-B-Micro, U10 NPN, U11 NPN, U12 NPN, U13 NPN, U14 NPN, U15 NPN, U16 NPN, U17 NPN, U18 NPN, U19 NPN, U2 AP2151DWG-7, U20 NPN, U21 NPN, U22 NPN, U23 NPN, U24 NPN, U25 NPN, U26 NPN, U27 NPN, U28 NPN, U29 NPN, U3 S7G2LQFP176, U30 NPN, U31 NPN, U32 NPN, U33 NPN, U34 NPN, U35 NPN, U36 NPN, U37 NPN, U38 NPN, U39 NPN, U4 TVS-Diode, U40 NPN, U41 NPN, U42 NPN, U43 NPN, U44 NPN, U45 NPN, U46 NPN, U47 NPN, U48 NPN, U49 NPN, U5 TVS-Diode, U51 NPN, U52 NPN, U53 NPN, U54 NPN, U56 NPN, U57 NPN, U59 NPN, U6 KSZ8081RNACAQFN-24-M, U7 NPN, U8 NPN, U9 NPN, X2 24MHz, X3 32.768KHz

Commit message: Updated
Parts:
- moved J1 2.40 mm to (7.31, 70.2)
- moved C20 1.10 mm to (17.5, 65.3)
- moved C40 0.55 mm to (53.5, 56.3)
- moved R13 0.55 mm to (52.5, 56.3)
- moved C16 0.50 mm to (51.4, 56.3)
Routing:
- net GND: track 16.2 -> 187.3 mm, vias 209 -> 146
- net SD1_DAT3: track 28.2 -> 21.4 mm
- net SD1_DAT0: track 28.9 -> 23.0 mm
- net SD1_DAT1: track 30.5 -> 26.8 mm
- net SD1_DAT2: track 24.0 -> 20.7 mm
- net SD1_CMD: track 24.3 -> 21.0 mm
- net SD1_CD: track 24.7 -> 21.4 mm
- net ETH_IRQ14: track 39.2 -> 36.3 mm
- net RESET: track 37.5 -> 39.7 mm
- net SD1_WP: track 12.2 -> 10.1 mm
- net SD1_CLK: track 25.9 -> 27.8 mm
- net LS_04: track 53.6 -> 51.7 mm
- net M2_DIR: track 19.9 -> 20.6 mm
- net VDD: vias 37 -> 38
- removed copper zone on layer 1, net GND
- removed copper zone on layer 16, net GND

Commit message: updated
Parts:
- moved AFID1 6.32 mm to (60.0, 4.00)
- moved AFID4 6.32 mm to (60.0, 4.00)
Connections:
- new net GNDE: J2.P$4, J6.SHLD1, J6.SHLD2, J7.P$6, J7.P$7, J7.P$8, J7.P$9, U$2.13, U$2.14
- net GND: no longer J2.P$4, J6.SHLD1, J6.SHLD2, J7.P$6, J7.P$7, J7.P$8, J7.P$9, U$2.13, U$2.14
Routing:
- net GNDE: track 0.00 -> 61.9 mm
- net GND: track 187.3 -> 171.9 mm, vias 146 -> 144
- removed copper zone on layer 2, net GND
- removed copper zone on layer 15, net VDD
