File: S7G2_Titan_6L/Titan_6L_v1p3.sch (EAGLE design)
At the start: 257 parts, among them J1 SD_CARD, J10 CONN_530470410_PICOBLADE_X_4, J12 10-pos, J13 CONN_530470410_PICOBLADE_X_4, J14 CONN_530470410_PICOBLADE_X_4, J15 CONN_530470410_PICOBLADE_X_4, J16 CONN_530470410_PICOBLADE_X_4, J17 CONN_530470410_PICOBLADE_X_4, J18 CONN_530470410_PICOBLADE_X_4, J19 CONN_530470410_PICOBLADE_X_4, J2 4-pos, J20 CONN_530470410_PICOBLADE_X_4, J21 CONN_530470410_PICOBLADE_X_4, J22 CONN_530470410_PICOBLADE_X_4, J24 CONN_530470410_PICOBLADE_X_4, J3 10-pos, J4 20-pos, J5 10-pos, J6 USB-A, J7 USB-B-Micro, U10 NPN, U11 NPN, U12 NPN, U13 NPN, U14 NPN, U15 NPN, U16 NPN, U17 NPN, U18 NPN, U19 NPN, U2 AP2151DWG-7, U20 NPN, U21 NPN, U22 NPN, U23 NPN, U24 NPN, U25 NPN, U26 NPN, U27 NPN, U28 NPN, U29 NPN, U3 S7G2LQFP176, U30 NPN, U31 NPN, U32 NPN, U33 NPN, U34 NPN, U35 NPN, U36 NPN, U37 NPN, U38 NPN, U39 NPN, U4 TVS-Diode, U40 NPN, U41 NPN, U42 NPN, U43 NPN, U44 NPN, U45 NPN, U46 NPN, U47 NPN, U48 NPN, U49 NPN, U5 TVS-Diode, U51 NPN, U52 NPN, U53 NPN, U54 NPN, U56 NPN, U57 NPN, U59 NPN, U6 KSZ8081RNACAQFN-24-M, U7 NPN, U8 NPN, U9 NPN, X2 24MHz, X3 32.768KHz

Commit message: updated
Connections:
- new net GNDE: J2.P$4, J6.SHIELD_1, J6.SHIELD_2, J7.SHIELD1, J7.SHIELD2, J7.SHIELD3, J7.SHIELD4, U$2.GNDE0, U$2.GNDE1
- net GND: no longer J2.P$4, J6.SHIELD_1, J6.SHIELD_2, J7.SHIELD1, J7.SHIELD2, J7.SHIELD3, J7.SHIELD4, U$2.GNDE0, U$2.GNDE1
