File: S7G2_Titan_6L/Titan_6L_EoB_v1p4.sch (EAGLE design)
At the start: 249 parts, among them J1 SD_CARD, J10 CONN_530470410_PICOBLADE_X_4, J12 10-pos, J13 CONN_530470410_PICOBLADE_X_4, J14 CONN_530470410_PICOBLADE_X_4, J15 CONN_530470410_PICOBLADE_X_4, J16 CONN_530470410_PICOBLADE_X_4, J17 CONN_530470410_PICOBLADE_X_4, J18 CONN_530470410_PICOBLADE_X_4, J19 CONN_530470410_PICOBLADE_X_4, J2 4-pos, J20 CONN_530470410_PICOBLADE_X_4, J21 CONN_530470410_PICOBLADE_X_4, J22 CONN_530470410_PICOBLADE_X_4, J24 CONN_530470410_PICOBLADE_X_4, J3 10-pos, J6 USB-A, J7 USB-B-Micro, U10 NPN, U11 NPN, U12 NPN, U13 NPN, U14 NPN, U15 NPN, U16 NPN, U17 NPN, U18 NPN, U19 NPN, U2 AP2151DWG-7, U20 NPN, U21 NPN, U22 NPN, U23 NPN, U24 NPN, U25 NPN, U26 NPN, U27 NPN, U28 NPN, U29 NPN, U3 S7G2LQFP176, U30 NPN, U31 NPN, U32 NPN, U33 NPN, U34 NPN, U35 NPN, U36 NPN, U37 NPN, U38 NPN, U39 NPN, U4 TVS-Diode, U40 NPN, U41 NPN, U42 NPN, U43 NPN, U44 NPN, U45 NPN, U46 NPN, U47 NPN, U48 NPN, U49 NPN, U5 TVS-Diode, U50 NPN, U51 NPN, U52 NPN, U53 NPN, U54 NPN, U55 NPN, U56 NPN, U7 NPN, U8 NPN, U9 NPN, X2 24MHz, X3 32.768KHz

Commit message: Update
Parts:
- added C15, C31, C47, C52: 0.1uF, 3D_MIG_Controller:C_0402
- added C44, C45: 24pF, 3D_MIG_Controller:C_0402
- added C46, C51: 22uF, 3D_MIG_Controller:C_0603
- added C48: 2.2uF, 3D_MIG_Controller:C_0402
- added C49: .1uF, 3D_MIG_Controller:C_0402
- added C50: 100pF, 3D_MIG_Controller:R_0402
- added FB2/2: (no value), 3D_MIG_Controller:FB_0805_120_OHM
- added R107, R108: 470, 3D_MIG_Controller:R_0402
- added R109: 6k49, 3D_MIG_Controller:R_0402
- added R110, R111: 10K, 3D_MIG_Controller:R_0402
- added R112, R113: 1K50, 3D_MIG_Controller:R_0402
- added R114, R115, R116, R117: 33, 3D_MIG_Controller:R_0402
- added U$2: (no value), 3D_MIG_Controller:RJ45_WITH_ELEC
- added U$3: (no value), 3D_MIG_Controller:XTAL_25_MHZ
- added U$4: 10uF, 3D_MIG_Controller:C_0402
- added U6: KSZ8081RNACAQFN-24-M, 3D_MIG_Controller:KSZ8081RNACAQFN-24-M
Connections:
- removed net ETH: U3.P7_1
- new net C58: C15.1, U$2.CT1
- new net C60: C31.1, U$2.CT2
- new net CRS_DV: R117.2, U6.CRS_DV/PHYAD[1:0]
- new net ETH_CLK: U3.P7_1, U6.REF_CLK
- new net LED1/SPEED: U$2.YLO, U6.LED0/ANEN_SPEED
- new net NC: U$2.P7
- new net R51: R107.1, U$2.YHI
- new net R52: R108.1, U$2.GHI
- new net REXT: C50.1, R109.2, U6.REXT
- new net RXD0: R115.2, U6.RXD0
- new net RXD1: R114.2, U6.RXD1
- new net RXER: R116.2, U6.RXER
- new net RXM: U$2.RD-, U6.RXM
- new net RXP: U$2.RD+, U6.RXP
- new net TXM: U$2.TD-, U6.TXM
- new net TXP: U$2.TD+, U6.TXP
- new net VDD_1.2: C48.1, C49.1, U6.VDD_1.2
- new net VDD_ENET1: C46.1, C47.1, FB2/2.P$2, U6.VDDA_3.3
- new net XII: C45.1, U$3.1, U6.XI
- new net XOO: C44.1, U$3.3, U6.XO
- net ETH_CRS_DV: now also R117.1
- net ETH_IRQ14: now also R110.1, U6.INTRP
- net ETH_MDC: now also R112.1, U6.MDC
- net ETH_MDIO: now also R113.1, U6.MDIO
- net ETH_RESET: now also R111.1, U$4.1, U6.!RST
- net ETH_RXD0: now also R115.1
- net ETH_RXD1: now also R114.1
- net ETH_RX_ER: now also R116.1
- net ETH_TXD0: now also U6.TXD0
- net ETH_TXD1: now also U6.TXD1
- net ETH_TXD_EN: now also U6.TXEN
- net GND: now also C15.2, C31.2, C44.2, C45.2, C46.2, C47.2, C48.2, C49.2, C50.2, C51.2, C52.2, R109.1, U$2.GLO, U$2.P8, U$3.2, U$3.4, U$4.2, U6.25, U6.GND
- net GNDS: now also U$2.GNDE0, U$2.GNDE1
- net VDD: now also C51.1, C52.1, FB2/2.P$1, R107.2, R108.2, R110.2, R111.2, R112.2, R113.2, U6.VDDIO
