File: Arduino_RC_Shield/Arduino_Shield_footprint.brd (EAGLE design)
At the start: 68.6 x 53.3 mm, 5 parts

Commit message: Update
Other:
- board outline removed
Changed lines of the file:
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@@
 <board>
 <plain>
-<wire x1="0" y1="0" x2="68.58" y2="0" width="0" layer="20"/>
-<wire x1="68.58" y1="0" x2="68.58" y2="53.34" width="0" layer="20"/>
-<wire x1="68.58" y1="53.34" x2="0" y2="53.34" width="0" layer="20"/>
-<wire x1="0" y1="53.34" x2="0" y2="0" width="0" layer="20"/>
+<wire x1="0" y1="0" x2="68.58" y2="0" width="0" layer="21"/>
+<wire x1="68.58" y1="0" x2="68.58" y2="53.34" width="0" layer="21"/>
+<wire x1="68.58" y1="53.34" x2="0" y2="53.34" width="0" layer="21"/>
+<wire x1="0" y1="53.34" x2="0" y2="0" width="0" layer="21"/>
 </plain>
 <attributes>
