File: Arduino_RC_Shield/Arduino_Shield_RC_Controller.sch (EAGLE design)
At the start: 6 parts

Commit message: Update
Parts:
- removed H1: (no value), 3D_MIG_Controller:1_X_6_HEADER_GENERIC_.1INCH
- removed H2, H3: (no value), 3D_MIG_Controller:1_X_8_HEADER_GENERIC_.1INCH
- removed U$1: 1_X_10_HEADER_GENERIC_.1INCH, 3D_MIG_Controller:1_X_10_HEADER_GENERIC_.1INCH
- added AR1: (no value), 3D_MIG_Controller:ARDUINO_R3
- added R1: (no value), 3D_MIG_Controller:R-TRIMM3103
- added R2, R3, R4: 10K0, 3D_MIG_Controller:R_0402_10K0
- added R5: 470R0, 3D_MIG_Controller:R_0402_470R0
- added SW1, SW2, SW3: PTS810SJG250SMTRLFS, 3D_MIG_Controller:PTS810SJG250SMTRLFS
Connections:
- new net A0: AR1.A0
- new net A1: AR1.A1
- new net A2: AR1.A2
- new net A3: AR1.A3
- new net A4: AR1.A4
- new net A5: AR1.A5
- new net AREF: AR1.AREF
- new net CIPO: AR1.CIPO/PB4, J1.1
- new net COPI: AR1.COPI/PB3, J1.4
- new net D4: AR1.8, LCD1.DB4
- new net D5: AR1.7, LCD1.DB5
- new net D6: AR1.4, LCD1.DB6
- new net D7: AR1.2, LCD1.DB7
- new net E: AR1.10, LCD1.E
- new net GND: AR1.GND0, AR1.GND1, AR1.GND2, AR1.GND3, J1.6, LCD1.K, LCD1.R/W, LCD1.VSS-GND, R1.E, SW1.3, SW1.4, SW2.3, SW2.4, SW3.3, SW3.4
- new net N$39: LCD1.A, R5.1
- new net NC: AR1.0-RX, AR1.1-TX, AR1.IOREF, AR1.NC, AR1.RESET, LCD1.DB0, LCD1.DB1, LCD1.DB2, LCD1.DB3
- new net PWM5: AR1.5
- new net PWM6: AR1.6
- new net PWM9: AR1.9
- new net RESET: AR1.RESET2, J1.5
- new net RS: AR1.11, LCD1.RS
- new net SCK: AR1.SCK/PB5, J1.3
- new net SCL: AR1.SCL
- new net SDA: AR1.SDA
- new net SW1: AR1.13, R4.2, SW1.1, SW1.2
- new net SW2: AR1.12, R3.2, SW2.1, SW2.2
- new net SW3: AR1.3, R2.2, SW3.1, SW3.2
- new net V0: LCD1.V0, R1.S
- new net VDD: AR1.3.3V
- new net VDD5: AR1.5V, AR1.VDD5, AR1.VIN, J1.2, LCD1.VDD5, R1.A, R2.1, R3.1, R4.1, R5.2
Other:
- moved on the sheet: J1

Commit message: Update
Parts:
- added C1: 0.1uF, 3D_MIG_Controller:C_0402_0.1UF
- added C2: CAP_470UF_RAD_TH, 3D_MIG_Controller:CAP_470UF_RAD_TH
- J1: device 3D_MIG_Controller:CONN_03X2 -> 3D_MIG_Controller:CONN_04X2
Connections:
- removed net CIPO: AR1.CIPO/PB4, J1.1
- removed net COPI: AR1.COPI/PB3, J1.4
- removed net PWM5: AR1.5
- removed net PWM6: AR1.6
- removed net RESET: AR1.RESET2, J1.5
- new net CSN: AR1.6, J1.4
- new net MISO: AR1.CIPO/PB4, J1.7
- new net MOSI: AR1.COPI/PB3, J1.6
- new net N$9: AR1.RESET2
- new net RCE: AR1.3, J1.3
- net GND: now also C1.1, C2.1, J1.1; no longer J1.6
- net NC: now also J1.8
- net SCK: now also J1.5; no longer J1.3
- net SW3: now also AR1.5; no longer AR1.3
- net VDD: now also C1.2, C2.2, J1.2
- net VDD5: no longer J1.2
