File: Arduino_RC_Shield/Arduino_Shield_RC_Controller_v2.brd (EAGLE design)
At the start: 135 x 100 mm, 10 parts, among them SW1 PTS810SJG250SMTRLFS, SW2 PTS810SJG250SMTRLFS, SW3 PTS810SJG250SMTRLFS

Commit message: updated
Parts:
- added SW4, SW5: PTS810SJG250SMTRLFS, 3D_MIG_Controller:PTS810
- moved AR1 82.6 mm to (129.8, 94.5), turned to 180 degrees
- moved R5 55.4 mm to (71.0, 34.2), flipped to the bottom, turned to 0 degrees
- moved R1 49.0 mm to (40.6, 45.2)
- moved C1 27.5 mm to (45.5, 91.0)
- moved J1 27.1 mm to (53.2, 90.7)
- moved C2 25.5 mm to (37.4, 87.7), turned to 90 degrees
- moved SW3 14.3 mm to (115.0, 84.0)
- moved SW1 14.0 mm to (16.8, 84.0)
- moved SW2 12.0 mm to (67.4, 58.4)
Connections:
- removed net A0: AR1.P30
- removed net A1: AR1.P29
- removed net A2: AR1.P28
- removed net A3: AR1.P27
- removed net A4: AR1.P26
- removed net A5: AR1.P25
- removed net AREF: AR1.P3
- removed net D4: AR1.P10, LCD1.P11
- removed net D5: AR1.P11, LCD1.P12
- removed net D6: AR1.P14, LCD1.P13
- removed net D7: AR1.P16, LCD1.P14
- removed net N$9: AR1.P23
- removed net PWM9: AR1.P9
- removed net SCL: AR1.P1
- removed net SDA: AR1.P2
- new net N$3: AR1.P11, LCD1.P14
- new net N$4: AR1.P12, LCD1.P13
- new net N$5: AR1.P13, LCD1.P12
- new net N$6: AR1.P14, LCD1.P11
- new net SW4: AR1.P27, SW4.1, SW4.2
- new net SW5: AR1.P28, SW5.1, SW5.2
- net CSN: now also AR1.P25; no longer AR1.P12
- net E: now also AR1.P16; no longer AR1.P8
- net GND: now also SW4.3, SW4.4, SW5.3, SW5.4; no longer AR1.P24
- net NC: no longer AR1.P36, AR1.P37, AR1.P38, J1.8, LCD1.P10, LCD1.P7, LCD1.P8, LCD1.P9
- net RCE: now also AR1.P26; no longer AR1.P15
- net RS: now also AR1.P15; no longer AR1.P7
- net SW1: now also AR1.P10; no longer AR1.P5
- net SW2: now also AR1.P9; no longer AR1.P6
- net SW3: now also AR1.P8; no longer AR1.P13
- net VDD5: no longer AR1.P20, AR1.P31
Routing:
- net VDD5: track 0.25 -> 161.0 mm, vias 0 -> 1
- net SW1: track 0.02 -> 90.6 mm, vias 0 -> 1
- net GND: track 0.18 -> 67.0 mm, vias 0 -> 2
- net VDD: track 0.14 -> 64.9 mm, vias 0 -> 1
- net SW3: track 0.00 -> 55.8 mm, vias 0 -> 1
- net RCE: track 0.00 -> 46.0 mm, vias 0 -> 1
- net RS: track 0.00 -> 44.2 mm, vias 0 -> 1
- net MOSI: track 0.00 -> 39.5 mm, vias 0 -> 1
- net MISO: track 0.00 -> 36.2 mm, vias 0 -> 1
- net SW2: track 0.01 -> 35.4 mm, vias 0 -> 1
- net E: track 0.00 -> 35.3 mm, vias 0 -> 1
- net CSN: track 0.00 -> 34.2 mm, vias 0 -> 1
- net SCK: track 0.00 -> 32.2 mm, vias 0 -> 1
- net N$5: track 0.00 -> 20.7 mm, vias 0 -> 1
- net N$4: track 0.00 -> 20.6 mm, vias 0 -> 1
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
Commit message: update
Routing:
- net GND: track 67.0 -> 72.7 mm
Changed lines of the file:
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@@
 <wire x1="69.025" y1="82.925" x2="73.175" y2="82.925" width="0.508" layer="1"/>
 <wire x1="79.925" y1="82.925" x2="84.075" y2="82.925" width="0.508" layer="1"/>
+<wire x1="45.5" y1="90.4" x2="45.5" y2="88.9" width="0.508" layer="1"/>
+<wire x1="37.4" y1="87.7" x2="39.5" y2="87.7" width="1.016" layer="1"/>
+<wire x1="37.4" y1="87.7" x2="35.3" y2="87.7" width="1.016" layer="1"/>
+<wire x1="99.3" y1="89.4" x2="112.925" y2="82.925" width="0" layer="19" extent="1-16"/>
+<wire x1="84.075" y1="82.925" x2="96.8" y2="89.2" width="0" layer="19" extent="1-16"/>
+<wire x1="73.6" y1="82.8" x2="79.925" y2="82.925" width="0" layer="19" extent="1-16"/>
+<wire x1="73.175" y1="82.925" x2="73.5" y2="82.7" width="0" layer="19" extent="1-16"/>
+<wire x1="49.4" y1="86.9" x2="69.025" y2="82.925" width="0" layer="19" extent="1-16"/>
+<wire x1="45.5" y1="88.9" x2="46.7" y2="89.5" width="0" layer="19" extent="1-16"/>
+<wire x1="39.5" y1="87.7" x2="45.5" y2="88.9" width="0" layer="19" extent="1-1"/>
+<wire x1="20.5" y1="82.9" x2="35.3" y2="87.7" width="0" layer="19" extent="1-16"/>
+<wire x1="69.475" y1="57.325" x2="69.025" y2="82.925" width="0" layer="19" extent="1-1"/>
+<wire x1="73.6" y1="37.05" x2="69.45" y2="57.3" width="0" layer="19" extent="1-1"/>
+<wire x1="53.2" y1="34.5" x2="73.6" y2="37.05" width="0" layer="19" extent="1-1"/>
+<wire x1="45.66" y1="37.05" x2="53.2" y2="34.5" width="0" layer="19" extent="1-1"/>
+<wire x1="39.6" y1="46.425" x2="45.6" y2="39.3" width="0" layer="19" extent="1-16"/>
+<wire x1="35.5" y1="39.4" x2="36.9" y2="46.5" width="0" layer="19" extent="1-16"/>
+<wire x1="37" y1="30" x2="35.5" y2="34.8" width="0" layer="19" extent="1-1"/>
+<wire x1="103.38" y1="43.66" x2="76.2" y2="36.8" width="0" layer="19" extent="1-1"/>
 </signal>
 <signal name="SCK">

Commit message: Update
Connections:
- net SW4: now also SW5.1, SW5.2; no longer SW4.1, SW4.2
- net SW5: now also SW4.1, SW4.2; no longer SW5.1, SW5.2
Routing:
- net GND: track 72.7 -> 60.1 mm
- net CSN: track 34.2 -> 22.3 mm
- net RCE: track 46.0 -> 35.6 mm
- net VDD: track 64.9 -> 68.4 mm
- net SW5: track 14.0 -> 16.4 mm
- net VDD5: track 161.0 -> 159.9 mm
- net SW4: track 16.4 -> 15.6 mm
Changed lines of the file:
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@@
 <contactref element="R1" pad="1"/>
 <contactref element="R5" pad="P$2"/>
-<wire x1="94.24" y1="91.96" x2="94.24" y2="55.44" width="1.016" layer="1"/>
 <wire x1="86.1" y1="47.3" x2="86.1" y2="40.2" width="1.016" layer="1"/>
 <wire x1="86.1" y1="40.2" x2="86.1" y2="38.3" width="1.016" layer="1"/>
@@
 <wire x1="73.53" y1="33.54" x2="71.07" y2="33.54" width="0.508" layer="16"/>
 <wire x1="71.07" y1="33.54" x2="71.05" y2="33.56" width="0.508" layer="16"/>
-<wire x1="94.24" y1="55.44" x2="86.1" y2="47.3" width="1.016" layer="1"/>
+<wire x1="91.25" y1="52.45" x2="86.1" y2="47.3" width="1.016" layer="1"/>
 <wire x1="86.1" y1="40.2" x2="52.2" y2="40.2" width="1.016" layer="1"/>
 <wire x1="46" y1="46.4" x2="44" y2="46.4" width="1.016" layer="1"/>
@@
 <wire x1="71.89" y1="31.9" x2="40.6" y2="31.9" width="1.016" layer="16"/>
 <wire x1="40.6" y1="31.9" x2="38.04" y2="34.46" width="1.016" layer="16"/>
+<wire x1="91.7" y1="91.96" x2="91.7" y2="52.9" width="1.016" layer="1"/>
+<wire x1="91.7" y1="52.9" x2="91.25" y2="52.45" width="1.016" layer="1"/>
 </signal>
 <signal name="GND">
@@
 <wire x1="103.38" y1="43.66" x2="103.38" y2="46.42" width="1.016" layer="16"/>
 <wire x1="103.38" y1="46.42" x2="103.3" y2="46.5" width="1.016" layer="16"/>
-<wire x1="96.78" y1="91.96" x2="96.78" y2="89.22" width="1.016" layer="16"/>
-<wire x1="96.78" y1="89.22" x2="96.8" y2="89.2" width="1.016" layer="16"/>
-<wire x1="99.32" y1="91.96" x2="99.32" y2="89.42" width="1.016" layer="16"/>
-<wire x1="99.32" y1="89.42" x2="99.3" y2="89.4" width="1.016" layer="16"/>
 <wire x1="49.39" y1="89.43" x2="49.4" y2="89.42" width="1.016" layer="16"/>
 <wire x1="49.4" y1="89.42" x2="49.4" y2="86.9" width="1.016" layer="16"/>
@@
 <wire x1="103.38" y1="43.66" x2="103.38" y2="46.32" width="1.016" layer="1"/>
 <wire x1="103.38" y1="46.32" x2="103.2" y2="46.5" width="1.016" layer="1"/>
-<wire x1="96.78" y1="91.96" x2="99.32" y2="91.96" width="1.016" layer="1"/>
-<wire x1="96.78" y1="91.96" x2="96.78" y2="89.42" width="1.016" layer="1"/>
-<wire x1="96.78" y1="89.42" x2="96.8" y2="89.4" width="1.016" layer="1"/>
-<wire x1="99.32" y1="91.96" x2="99.32" y2="89.88" width="1.016" layer="1"/>
-<wire x1="99.32" y1="89.88" x2="99.4" y2="89.8" width="1.016" layer="1"/>
 <wire x1="69.025" y1="82.925" x2="73.175" y2="82.925" width="0.508" layer="1"/>
 <wire x1="79.925" y1="82.925" x2="84.075" y2="82.925" width="0.508" layer="1"/>
@@
 <wire x1="37.4" y1="87.7" x2="39.5" y2="87.7" width="1.016" layer="1"/>
 <wire x1="37.4" y1="87.7" x2="35.3" y2="87.7" width="1.016" layer="1"/>
-<wire x1="99.3" y1="89.4" x2="112.925" y2="82.925" width="0" layer="19" extent="1-16"/>
-<wire x1="84.075" y1="82.925" x2="96.8" y2="89.2" width="0" layer="19" extent="1-16"/>
+<wire x1="89.16" y1="91.96" x2="112.925" y2="82.925" width="0" layer="19" extent="1-1"/>
+<wire x1="86.62" y1="91.96" x2="89.16" y2="91.96" width="0" layer="19" extent="1-1"/>
+<wire x1="84.075" y1="82.925" x2="86.62" y2="91.96" width="0" layer="19" extent="1-1"/>
 <wire x1="73.6" y1="82.8" x2="79.925" y2="82.925" width="0" layer="19" extent="1-16"/>
 <wire x1="73.175" y1="82.925" x2="73.5" y2="82.7" width="0" layer="19" extent="1-16"/>
@@
 <wire x1="45.5" y1="91.6" x2="38.5038" y2="91.6" width="0.508" layer="1"/>
 <wire x1="38.5038" y1="91.6" x2="37.4" y2="92.7038" width="0.508" layer="1"/>
-<wire x1="91.7" y1="91.96" x2="86.56" y2="97.1" width="1.016" layer="1"/>
+<wire x1="94.24" y1="91.96" x2="94.24" y2="93.56" width="1.016" layer="1"/>
+<wire x1="94.24" y1="93.56" x2="90.7" y2="97.1" width="1.016" layer="1"/>
 <wire x1="48.3" y1="97.1" x2="45.5" y2="94.3" width="1.016" layer="1"/>
-<wire x1="86.56" y1="97.1" x2="48.3" y2="97.1" width="1.016" layer="1"/>
+<wire x1="90.7" y1="97.1" x2="48.3" y2="97.1" width="1.016" layer="1"/>
 <wire x1="49.39" y1="91.97" x2="49.02" y2="91.6" width="0.508" layer="16"/>
 <wire x1="49.02" y1="91.6" x2="46.7" y2="91.6" width="0.508" layer="16"/>
@@
 <contactref element="AR1" pad="P26"/>
 <wire x1="51.93" y1="89.43" x2="51.93" y2="80.27" width="0.508" layer="16"/>
-<wire x1="52.9" y1="79.3" x2="75.2" y2="79.3" width="0.508" layer="16"/>
-<wire x1="75.2" y1="79.3" x2="76.5" y2="80.6" width="0.508" layer="16"/>
-<wire x1="76.5" y1="80.6" x2="76.5" y2="89.6" width="0.508" layer="16"/>
-<via x="76.5" y="89.6" extent="1-16" drill="0.35"/>
-<wire x1="76.5" y1="89.6" x2="76.46" y2="89.64" width="0.508" layer="1"/>
-<wire x1="76.46" y1="89.64" x2="76.46" y2="91.96" width="0.508" layer="1"/>
-<wire x1="51.93" y1="80.27" x2="52.9" y2="79.3" width="0.508" layer="16"/>
+<via x="65" y="88.2" extent="1-16" drill="0.35"/>
+<wire x1="65" y1="88.2" x2="65" y2="81.5" width="0.508" layer="16"/>
+<wire x1="68.84" y1="91.96" x2="65.08" y2="88.2" width="0.508" layer="1"/>
+<wire x1="65" y1="88.2" x2="65.08" y2="88.2" width="0.508" layer="1"/>
+<wire x1="52.9" y1="79.3" x2="51.93" y2="80.27" width="0.508" layer="16"/>
+<wire x1="65" y1="81.5" x2="62.8" y2="79.3" width="0.508" layer="16"/>
+<wire x1="62.8" y1="79.3" x2="52.9" y2="79.3" width="0.508" layer="16"/>
 </signal>
 <signal name="MISO">
@@
 <wire x1="51.93" y1="91.97" x2="51.93" y2="95.33" width="0.508" layer="16"/>
 <wire x1="51.93" y1="95.33" x2="53.3" y2="96.7" width="0.508" layer="16"/>
-<wire x1="53.3" y1="96.7" x2="76.4" y2="96.7" width="0.508" layer="16"/>
-<wire x1="76.4" y1="96.7" x2="79" y2="94.1" width="0.508" layer="16"/>
-<via x="79" y="94.1" extent="1-16" drill="0.35"/>
-<wire x1="79" y1="94.1" x2="79" y2="91.96" width="0.508" layer="1"/>
+<wire x1="53.3" y1="96.7" x2="65" y2="96.7" width="0.508" layer="16"/>
+<wire x1="65" y1="96.7" x2="66.3" y2="95.4" width="0.508" layer="16"/>
+<via x="66.3" y="95.4" extent="1-16" drill="0.35"/>
+<wire x1="66.3" y1="95.4" x2="66.3" y2="91.96" width="0.508" layer="1"/>
 </signal>
 <signal name="MOSI">
@@
 <wire x1="60.9" y1="38.8" x2="63.9" y2="41.8" width="0.508" layer="16"/>
 </signal>
-<signal name="SW4">
+<signal name="SW5">
 <contactref element="SW4" pad="2"/>
 <contactref element="SW4" pad="1"/>
-<contactref element="AR1" pad="P27"/>
 <wire x1="84.075" y1="85.075" x2="79.925" y2="85.075" width="0.508" layer="1"/>
-<wire x1="79.925" y1="85.075" x2="77.525" y2="85.075" width="0.508" layer="1"/>
-<wire x1="73.92" y1="88.68" x2="73.92" y2="91.96" width="0.508" layer="1"/>
-<wire x1="77.525" y1="85.075" x2="73.92" y2="88.68" width="0.508" layer="1"/>
+<wire x1="77.525" y1="85.075" x2="79.925" y2="85.075" width="0.508" layer="1"/>
 <wire x1="84.075" y1="85.075" x2="85.575" y2="85.075" width="0.508" layer="1"/>
-</signal>
-<signal name="SW5">
+<contactref element="AR1" pad="P28"/>
+<wire x1="73.92" y1="91.96" x2="73.92" y2="88.68" width="0.508" layer="1"/>
+<wire x1="73.92" y1="88.68" x2="77.525" y2="85.075" width="0.508" layer="1"/>
+</signal>
+<signal name="SW4">
 <contactref element="SW5" pad="2"/>
 <contactref element="SW5" pad="1"/>
-<contactref element="AR1" pad="P28"/>
-<wire x1="69.025" y1="85.075" x2="71.4" y2="85.075" width="0.508" layer="1"/>
-<wire x1="71.4" y1="85.075" x2="73.175" y2="85.075" width="0.508" layer="1"/>
-<wire x1="71.38" y1="91.96" x2="71.4" y2="91.94" width="0.508" layer="1"/>
-<wire x1="71.4" y1="91.94" x2="71.4" y2="85.075" width="0.508" layer="1"/>
+<wire x1="69.025" y1="85.075" x2="71.7" y2="85.075" width="0.508" layer="1"/>
+<wire x1="73.175" y1="85.075" x2="74.6" y2="85.075" width="0.508" layer="1"/>
+<wire x1="71.7" y1="85.075" x2="73.175" y2="85.075" width="0.508" layer="1"/>
 <wire x1="69.025" y1="85.075" x2="67.225" y2="85.075" width="0.508" layer="1"/>
 <wire x1="73.175" y1="85.075" x2="74.375" y2="85.075" width="0.508" layer="1"/>
+<contactref element="AR1" pad="P27"/>
+<wire x1="71.38" y1="91.96" x2="71.38" y2="85.395" width="0.508" layer="1"/>
+<wire x1="71.38" y1="85.395" x2="71.7" y2="85.075" width="0.508" layer="1"/>
 </signal>
 </signals>
