File: Callisto_Limit_Switch_x_10/Callisto_LSOx10_v1p1.brd (EAGLE design)
At the start: 120 x 59.1 mm, 21 parts, among them J1 2-pos, J10 CRJ044-3-TH, J14 CRJ044-3-TH, J16 CRJ044-3-TH, J18 CRJ044-3-TH, J22 CRJ044-3-TH, J24 CRJ044-3-TH, J28 CRJ044-3-TH, J4 CRJ044-3-TH, J6 CRJ044-3-TH, J8 CRJ044-3-TH

Commit message: Update
Parts:
- renumbered J15 to LS_OUT
Connections:
- net GND: now also J11.2, J17.2, J19.2, J23.2, J25.2, J29.2, J5.2, J7.2, J9.2, LS_OUT.2; no longer J11.1, J17.1, J19.1, J23.1, J25.1, J29.1, J5.1, J7.1, J9.1, LS_OUT.1
- net LS_OUT: now also J11.1, J17.1, J19.1, J23.1, J25.1, J29.1, J5.1, J7.1, J9.1, LS_OUT.1; no longer J11.2, J17.2, J19.2, J23.2, J25.2, J29.2, J5.2, J7.2, J9.2, LS_OUT.2
Routing:
- net GND: track 0.00 -> 256.3 mm, vias 19 -> 21
- net LS_OUT: track 178.8 -> 178.3 mm
Other:
- board text added: "+12V"
- board text added: "E-Stop"
- board text added: "Gnd"
- board text added: "LSR"
- board text added: "LS_01"
- board text added: "LS_02"
- board text added: "LS_03"
- board text added: "LS_04"
- board text added: "LS_05"
- board text added: "LS_06"
- board text added: "LS_07"
- board text added: "LS_08"
- board text added: "LS_09"
