File: R7FS5D37A3A01CFM/R7FS5D37A3A01CFM.brd (EAGLE design)
At the start: 160 x 100 mm, 8 parts, among them J1 CONN_530470410_PICOBLADE_X_4, U1 R7FS5D37A3A01CFPAA0, U5 NPN, U6 NPN, U7 NPN

Commit message: Updates
Parts:
- removed U5, U6, U7: NPN, 3D_MIG_Controller:SOT323
- added C1, C10, C3, C4, C5, C6, C7, C8, C9: 0.1uF, 3D_MIG_Controller:0402
- added C11: 1uF, 3D_MIG_Controller:0402
- added C16: 10uF, 3D_MIG_Controller:0402
- added C17, C18: 10pF, 3D_MIG_Controller:0402
- added C32, C37: 12pF, 3D_MIG_Controller:0402
- added J11, J13, J16, J17, J20, J21, J4, J6, J7, J9: (no value), 3D_MIG_Controller:CON_530470210_MOL
- added J2, J5: CONN_530470410_PICOBLADE_X_4, 3D_MIG_Controller:CON_530470410_MOL
- added J3: 10-pos, 3D_MIG_Controller:2X5
- added LED11, LED12, LED15, LED16, LED2, LED4, LED6, LED8: Green, 3D_MIG_Controller:0805
- added R1, R10, R11, R12, R2, R3, R9: 33R0, 3D_MIG_Controller:0402
- added R13, R41, R44, R53, R56: 10K0, 3D_MIG_Controller:0402
- added R19, R23, R27, R31: 500R0, 3D_MIG_Controller:0402
- added R20, R24, R28, R32, R40, R43, R52, R55: 470R0, 3D_MIG_Controller:0402
- added R39, R42, R51, R54: 2.2K, 3D_MIG_Controller:0402
- added U10, U11, U12, U17, U19, U2, U21, U23, U25, U28, U29, U3, U32, U33, U4, U9: NPN, 3D_MIG_Controller:SOT323
- added X3: 32.768KHz, 3D_MIG_Controller:SMD_X_2_PADS
- added Y1: XTAL_12MHZ_ABM8G-12.000MHZ-B4Y-T, 3D_MIG_Controller:CRYSTAL_ABM8G_ABR
- J1: value CONN_530470410_PICOBLADE_X_4 -> (none); device 3D_MIG_Controller:CON_530470410_MOL -> 3D_MIG_Controller:CON_530470210_MOL
- R5, R6: value 33R0 -> (none)
- U1: value R7FS5D37A3A01CFPAA0 -> RENESAS_R7FS5D37A3A01CFM#AA0PLQP0064KB-C_REN-M; device 3D_MIG_Controller:PLQP0100KB-B_REN -> 3D_MIG_Controller:PLQP0064KB-C_REN-M
- moved J1 74.4 mm to (11.8, -5.00), turned to 0 degrees
- moved R6 57.8 mm to (8.45, -5.70), turned to 180 degrees
- moved R5 53.7 mm to (12.2, 1.35), turned to 270 degrees
- moved R4 32.0 mm to (-1.81, 30.1), turned to 0 degrees
- moved U1 26.1 mm to (0.00, 0.00), turned to 270 degrees
Connections:
- net VCC_3 renamed SCLK
- net VCC_4 renamed DFI_02
- net VCC_USB_LDO renamed DFO_01
- net VSS_3 renamed SSL0
- net VSS_USB renamed N$76
- removed net AVCC0: U1.88
- removed net AVSS0: U1.89
- removed net DIR: R5.P$1
- removed net ENABLE: R6.P$1
- removed net N$5: R6.P$2, U7.1
- removed net N$6: R4.P$2, U5.1
- removed net STEP: R4.P$1
- removed net VCC: U1.82
- removed net VCC_2: U1.15
- removed net VCC_USB: U1.29
- removed net VCL: U1.64
- removed net VREFH: U1.87
- removed net VREFH0: U1.91
- removed net VREFL: U1.86
- removed net VREFL0: U1.90
- removed net VSS: U1.83
- removed net VSS_2: U1.12
- removed net VSS_4: U1.63
- new net A1M0_DIR: R2.P$1, U1.15
- new net A1M0_ENABLE: R3.P$1, U1.14
- new net A1M0_HLFB: U1.13, U9.2
- new net A1M0_STEP: R1.P$1, U1.16
- new net A1M1_DIR: R10.P$1, U1.3
- new net A1M1_ENABLE: R11.P$1, U1.2
- new net A1M1_HLFB: U1.1, U17.2
- new net A1M1_STEP: R9.P$1, U1.12
- new net AN07: J4.2, R5.P$2, U1.61
- new net AN16: J1.2, R6.P$2, U1.49
- new net DAC: J6.2, U1.54
- new net DFI_01: U1.50
- new net DFO_02: U1.41
- new net DFO_03: U1.42
- new net ESTOP: U1.27
- new net HLFB_RETURN: J2.1, J5.1, R12.P$1, R4.P$1
- new net LS_01: R40.P$2, R41.P$2, U1.23, U28.2
- new net LS_02: R43.P$2, R44.P$2, U1.53, U29.2
- new net LS_03: R52.P$2, R53.P$2, U1.64, U32.2
- new net LS_04: R55.P$2, R56.P$2, U1.63, U33.2
- new net LS_RET: J16.2, J17.2, J20.2, J21.2, R39.P$1, R42.P$1, R51.P$1, R54.P$1
- new net MISO: U1.48
- new net MOSI: U1.47
- new net N$1: R2.P$2, U3.1
- new net N$10: R11.P$2, U12.1
- new net N$11: R9.P$2, U10.1
- new net N$12: R12.P$2, U17.1
- new net N$2: R3.P$2, U4.1
- new net N$20: R19.P$2, U19.1
- new net N$21: J7.2, LED2.2, U19.3
- new net N$22: LED2.1, R20.P$1
- new net N$26: R23.P$2, U21.1
- new net N$27: J9.2, LED4.2, U21.3
- new net N$28: LED4.1, R24.P$1
- new net N$32: R27.P$2, U23.1
- new net N$33: J11.2, LED6.2, U23.3
- new net N$34: LED6.1, R28.P$1
- new net N$38: R31.P$2, U25.1
- new net N$39: J13.2, LED8.2, U25.3
- new net N$4: R4.P$2, U9.1
- new net N$40: LED8.1, R32.P$1
- new net N$45: R39.P$2, U28.1
- new net N$46: LED11.1, R40.P$1
- new net N$47: R42.P$2, U29.1
- new net N$48: LED12.1, R43.P$1
- new net N$53: R51.P$2, U32.1
- new net N$54: LED15.1, R52.P$1
- new net N$55: R54.P$2, U33.1
- new net N$56: LED16.1, R55.P$1
- new net N$69: U1.18
- new net N$70: U1.19
- new net N$82: U1.36
- new net N$83: U1.37
- new net N$86: U1.40
- new net N$89: U1.43
- new net N$9: R10.P$2, U11.1
- new net N$90: U1.44
- new net RELAY_1: R19.P$1, U1.24
- new net RELAY_2: R23.P$1, U1.21
- new net RELAY_3: R27.P$1, U1.22
- new net RELAY_4: R31.P$1, U1.31
- new net RESET: C16.P$1, J3.9, R13.P$1, U1.25
- new net TCK: J3.7, U1.32
- new net TDI: J3.1, U1.35
- new net TDO: J3.3, U1.34
- new net TMS: J3.5, U1.33
- new net VDD: C1.P$1, C10.P$1, C11.P$1, C3.P$1, C4.P$1, C5.P$1, C7.P$2, C8.P$1, C9.P$1, J3.2, J3.4, R13.P$2, R5.P$1, R6.P$1, U1.11, U1.20, U1.29, U1.38, U1.51, U1.56, U1.57, U1.60, U17.3, U28.3, U29.3, U32.3, U33.3, U9.3
- new net VDD5: J11.1, J13.1, J7.1, J9.1, R20.P$2, R24.P$2, R28.P$2, R32.P$2
- new net XCIN: C32.P$1, U1.6, X3.P$1
- new net XCOUT: C37.P$1, U1.7, X3.P$2
- new net XTAL1: C17.P$1, U1.9, Y1.3
- new net XTAL2: C18.P$1, U1.10, Y1.1
- net GND: now also C1.P$2, C10.P$2, C11.P$2, C16.P$2, C17.P$2, C18.P$2, C3.P$2, C32.P$2, C37.P$2, C4.P$2, C5.P$2, C6.P$1, C7.P$1, C8.P$2, C9.P$2, J16.1, J17.1, J20.1, J21.1, J3.10, J3.6, J3.8, J4.1, J6.1, LED11.2, LED12.2, LED15.2, LED16.2, R41.P$1, R44.P$1, R53.P$1, R56.P$1, U1.17, U1.28, U1.39, U1.52, U1.55, U1.58, U1.59, U1.8, U10.2, U11.2, U12.2, U19.2, U2.2, U21.2, U23.2, U25.2, U3.2, U4.2, Y1.2, Y1.4; no longer U5.2, U6.2, U7.2
- net MO_DIR: now also J2.3, J5.3, U11.3, U3.3; no longer J1.3, U6.3
- net MO_ENABLE: now also J2.2, J5.2, U12.3, U4.3; no longer J1.2, U7.3
- net MO_STEP: now also J2.4, J5.4, U10.3, U2.3; no longer J1.4, U5.3
- net N$3: now also R1.P$2, U2.1; no longer R5.P$2, U6.1
- net VBATT: now also U1.4; no longer U1.8
- net VCL0: now also C6.P$2, U1.5; no longer U1.9
Routing:
- net VDD: track 0.00 -> 196.7 mm, vias 0 -> 10
- net VDD5: track 0.00 -> 80.3 mm, vias 0 -> 1
- net LS_01: track 0.00 -> 46.6 mm, vias 0 -> 2
- net RELAY_2: track 0.00 -> 39.3 mm, vias 0 -> 2
- net RELAY_1: track 0.00 -> 33.7 mm
- net LS_02: track 0.00 -> 32.4 mm, vias 0 -> 2
- net DAC: track 0.00 -> 29.9 mm, vias 0 -> 1
- net RELAY_4: track 0.00 -> 29.7 mm
- net A1M0_STEP: track 0.00 -> 26.4 mm, vias 0 -> 2
- net A1M0_HLFB: track 0.00 -> 24.8 mm, vias 0 -> 2
- net A1M0_DIR: track 0.00 -> 23.2 mm, vias 0 -> 2
- net HLFB_RETURN: track 0.00 -> 22.8 mm
- net A1M1_STEP: track 0.00 -> 22.7 mm, vias 0 -> 2
- net A1M1_HLFB: track 0.00 -> 22.6 mm, vias 0 -> 2
- net A1M0_ENABLE: track 0.00 -> 21.1 mm, vias 0 -> 2
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Other:
- board outline removed
- board text added: "10pf"
- board text added: "12.0 MHz"
- board text added: "32.768KHz"
- board text added: "A/D 1"
- board text added: "A/D 2"
- board text added: "A1M0"
- board text added: "A1M1"
- board text added: "DAC 1"
- board text added: "JTAG"
- board text added: "LS_01"
- board text added: "LS_02"
- board text added: "LS_03"
- board text added: "LS_04"
- board text added: "Relay 1"
- board text added: "Relay 2"
- board text added: "Relay 3"
- board text added: "Relay 4"
- board text added: "Reset"
- board text added: "TCK"
- board text added: "TDI"
- board text added: "TDO"
- board text added: "TMS"

Commit message: Update
Parts:
- removed J3: 10-pos, 3D_MIG_Controller:2X5
- added J8: CONN_530470610_PICOBLADE_X_6, 3D_MIG_Controller:CON_530470610_MOL
- moved C16 6.22 mm to (-15.8, 3.30)
- moved C5 6.22 mm to (-17.9, 3.30)
- moved R13 6.22 mm to (-16.9, 3.30)
- moved C7 0.40 mm to (-2.94, 8.37)
- moved C3 0.22 mm to (-7.75, 3.20)
Connections:
- net A1M0_DIR renamed DIR_M0A1
- net A1M0_ENABLE renamed ENABLE_M0A1
- net A1M0_HLFB renamed HLFB_M0A1
- net A1M0_STEP renamed STEP_M0A1
- net A1M1_DIR renamed DIR_M1A1
- net A1M1_ENABLE renamed ENABLE_M1A1
- net A1M1_HLFB renamed HLFB_M1A1
- net A1M1_STEP renamed STEP_M1A1
- net AN07 renamed AN07_A1
- net AN16 renamed AN16_A1
- net DAC renamed DAC_A1
- net DFI_01 renamed DFI_01_A1
- net DFI_02 renamed DFI_02_A1
- net DFO_01 renamed DFO_01_A1
- net DFO_02 renamed DFO_02_A1
- net DFO_03 renamed DFO_03_A1
- net ESTOP renamed ESTOP_A1
- net LS_01 renamed LS_01_A1
- net LS_02 renamed LS_02_A1
- net LS_03 renamed LS_03_A1
- net LS_04 renamed LS_04_A1
- net RELAY_1 renamed RELAY_1_A1
- net RELAY_2 renamed RELAY_2_A1
- net RELAY_3 renamed RELAY_3_A1
- net RELAY_4 renamed RELAY_4_A1
- net SSL0 renamed SSL0_A1
- net VBATT renamed VBATT_M1A1
- net VCL0 renamed VCL0_A1
- net XCIN renamed XCIN_A1
- net XCOUT renamed XCOUT_A1
- net XTAL1 renamed XTAL1_A1
- net XTAL2 renamed XTAL2_A1
- removed net HLFB_RETURN: J2.1, J5.1, R12.P$1, R4.P$1
- removed net LS_RET: J16.2, J17.2, J20.2, J21.2, R39.P$1, R42.P$1, R51.P$1, R54.P$1
- removed net MO_DIR: J2.3, J5.3, U11.3, U3.3
- removed net MO_ENABLE: J2.2, J5.2, U12.3, U4.3
- removed net MO_STEP: J2.4, J5.4, U10.3, U2.3
- removed net RESET: C16.P$1, J3.9, R13.P$1, U1.25
- removed net TCK: J3.7, U1.32
- removed net TDI: J3.1, U1.35
- removed net TDO: J3.3, U1.34
- removed net TMS: J3.5, U1.33
- new net HLFB_RETURN_M0_A1: J2.1, R4.P$1
- new net HLFB_RETURN_M1_A1: J5.1, R12.P$1
- new net LS_01_RET_A1: J16.2, R39.P$1
- new net LS_02_RET_A1: J17.2, R42.P$1
- new net LS_03_RET_A1: J20.2, R51.P$1
- new net LS_04_RET_A1: J21.2, R54.P$1
- new net MO_DIR_M0_A1: J2.3, U3.3
- new net MO_DIR_M1_A1: J5.3, U11.3
- new net MO_ENABLE_M0_A1: J2.2, U4.3
- new net MO_ENABLE_M1_A1: J5.2, U12.3
- new net MO_STEP_M0_A1: J2.4, U2.3
- new net MO_STEP_M1_A1: J5.4, U10.3
- new net RESET_A1: C16.P$1, J8.2, R13.P$1, U1.25
- new net TCK_A1: J8.6, U1.32
- new net TDI_A1: J8.3, U1.35
- new net TDO_A1: J8.4, U1.34
- new net TMS_A1: J8.5, U1.33
- net GND: now also J8.1; no longer J3.10, J3.6, J3.8
- net VDD: no longer J3.2, J3.4
Routing:
- net MO_ENABLE: track 35.8 -> 0.00 mm
- net HLFB_RETURN: track 22.8 -> 0.00 mm
- net TDI_A1: track 0.00 -> 18.8 mm
- net MO_ENABLE_M1_A1: track 0.00 -> 17.9 mm
- net MO_ENABLE_M0_A1: track 0.00 -> 17.9 mm
- net MO_DIR: track 17.8 -> 0.00 mm
- net RESET_A1: track 0.00 -> 17.0 mm
- net TMS: track 16.6 -> 0.00 mm
- net RESET: track 16.6 -> 0.00 mm
- net TDO: track 16.2 -> 0.00 mm
- net TDO_A1: track 0.00 -> 16.0 mm
- net TDI: track 14.9 -> 0.00 mm
- net TMS_A1: track 0.00 -> 13.5 mm
- net TCK: track 13.3 -> 0.00 mm
- net HLFB_RETURN_M1_A1: track 0.00 -> 11.4 mm
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Other:
- board text added: "Limit Sw 1"
- board text added: "Limit Sw 2"
- board text added: "Limit Sw 3"
- board text added: "Limit Sw 4"
- board text added: "Th 1"
- board text added: "Th 2"
- board text removed: "10pf"
- board text removed: "A/D 1"
- board text removed: "A/D 2"
- board text removed: "LS_01"
- board text removed: "LS_02"
- board text removed: "LS_03"
- board text removed: "LS_04"

Commit message: Update
Parts:
- added J25: (no value), 3D_MIG_Controller:CON_530470210_MOL
- added J29: (no value), 3D_MIG_Controller:2X5
- J1: value (none) -> 4-pos; device 3D_MIG_Controller:CON_530470210_MOL -> 3D_MIG_Controller:1X4_3.81MM_PITCH
- R22, R26, R30, R34: value 500R0 -> 470R0
- R36, R45, R48, R57: value 2.2K -> 2K2
- R60, R61: value (none) -> 100K0
- moved J1 50.2 mm to (8.60, 45.1), turned to 180 degrees
- renumbered C1 to C15, C10 to C26, C11 to C27, C16 to C28, C17 to C13, C18 to C14, C3 to C19, C32 to C2, C37 to C12, C4 to C20, C5 to C21, C6 to C22, C7 to C23, C8 to C24, C9 to C25, J11 to J15, J13 to J18, J16 to J19, J17 to J22, J2 to J3, J20 to J23, J21 to J24, J4 to J26, J5 to J10, J6 to J27, J7 to J12, J8 to J28, J9 to J14, LED11 to LED9, LED12 to LED10, LED15 to LED13, LED16 to LED14, LED2 to LED1, LED4 to LED3, LED6 to LED5, LED8 to LED7, R1 to R7, R10 to R17, R11 to R18, R12 to R21, R13 to R62, R19 to R22, R2 to R8, R20 to R25, R23 to R26, R24 to R29, R27 to R30, R28 to R33, R3 to R14, R31 to R34, R32 to R35, R39 to R36, R4 to R15, R40 to R37, R41 to R38, R42 to R45, R43 to R46, R44 to R47, R5 to R60, R51 to R48, R52 to R49, R53 to R50, R54 to R57, R55 to R58, R56 to R59, R6 to R61, R9 to R16, U1 to U5, U10 to U14, U11 to U15, U12 to U16, U17 to U18, U19 to U20, U2 to U6, U21 to U22, U23 to U24, U25 to U26, U28 to U27, U29 to U30, U3 to U7, U32 to U31, U33 to U34, U4 to U8, U9 to U13, X3 to X1, Y1 to Y2
Connections:
- new net VDD12: J1.P$4
- net AN16_A1: now also J25.2; no longer J1.2
- net GND: now also J1.P$1, J25.1, J29.1, J29.2; no longer J1.1
- net MISO: now also J29.10, J29.9
- net MOSI: now also J29.7, J29.8
- net SCLK: now also J29.5, J29.6
- net SSL0_A1: now also J29.3, J29.4
- net VDD: now also J1.P$2
- net VDD5: now also J1.P$3
Routing:
- net MISO: track 0.00 -> 9.34 mm
- net SSL0_A1: track 0.00 -> 8.13 mm
- net MOSI: track 0.00 -> 7.62 mm
- net SCLK: track 0.00 -> 7.29 mm
- net VDD5: track 80.3 -> 85.1 mm
- net VDD: track 203.7 -> 207.1 mm
Other:
- board outline added: 39 x 64 mm
