File: R7FS5D37A3A01CFM/R7FS5D37A3A01CFM.sch (EAGLE design)
At the start: 8 parts, among them J1 CONN_530470410_PICOBLADE_X_4, U1 R7FS5D37A3A01CFPAA0, U5 NPN, U6 NPN, U7 NPN

Commit message: Updates
Parts:
- removed U5, U6, U7: NPN, 3D_MIG_Controller:BC846BW
- added C1, C10, C3, C4, C5, C6, C7, C8, C9: 0.1uF, 3D_MIG_Controller:C_0402_0.1UF
- added C11: 1uF, 3D_MIG_Controller:C_0402_1UF
- added C16: 10uF, 3D_MIG_Controller:C_0402_10UF
- added C17, C18: 10pF, 3D_MIG_Controller:C_0402
- added C32, C37: 12pF, 3D_MIG_Controller:C_0402_12PF
- added J11, J13, J16, J17, J20, J21, J4, J6, J7, J9: (no value), 3D_MIG_Controller:CONN_530470210_PICOBLADE_X_2
- added J2, J5: CONN_530470410_PICOBLADE_X_4, 3D_MIG_Controller:CONN_530470410_PICOBLADE_X_4
- added J3: 10-pos, 3D_MIG_Controller:CONN_05X2_RAPTH
- added LED11, LED12, LED15, LED16, LED2, LED4, LED6, LED8: Green, 3D_MIG_Controller:LED_0805_GREEN
- added R1, R10, R11, R12, R2, R3, R9: 33R0, 3D_MIG_Controller:R_0402_33R0
- added R13, R41, R44, R53, R56: 10K0, 3D_MIG_Controller:R_0402_10K0
- added R19, R23, R27, R31: 500R0, 3D_MIG_Controller:R_0402
- added R20, R24, R28, R32, R40, R43, R52, R55: 470R0, 3D_MIG_Controller:R_0402_470R0
- added R39, R42, R51, R54: 2.2K, 3D_MIG_Controller:R_0402
- added U10, U11, U12, U17, U19, U2, U21, U23, U25, U28, U29, U3, U32, U33, U4, U9: NPN, 3D_MIG_Controller:BC846BW
- added X3: 32.768KHz, 3D_MIG_Controller:XTAL_32.768KHZ
- added Y1: XTAL_12MHZ_ABM8G-12.000MHZ-B4Y-T, 3D_MIG_Controller:XTAL_12MHZ_ABM8G-12.000MHZ-B4Y-T
- J1: value CONN_530470410_PICOBLADE_X_4 -> (none); device 3D_MIG_Controller:CONN_530470410_PICOBLADE_X_4 -> 3D_MIG_Controller:CONN_530470210_PICOBLADE_X_2
- R5, R6: value 33R0 -> (none); device 3D_MIG_Controller:R_0402_33R0 -> 3D_MIG_Controller:R_0402
- U1: value R7FS5D37A3A01CFPAA0 -> RENESAS_R7FS5D37A3A01CFM#AA0PLQP0064KB-C_REN-M; device 3D_MIG_Controller:R7FS5D37A3A01CFPAA0 -> 3D_MIG_Controller:RENESAS_R7FS5D37A3A01CFM#AA0PLQP0064KB-C_REN-M
Connections:
- removed net DIR: R5.1
- removed net ENABLE: R6.1
- removed net N$5: R6.2, U7.B(2)
- removed net N$6: R4.2, U5.B(2)
- removed net STEP: R4.1
- new net A1M0_DIR: R2.1, U1.15/P408
- new net A1M0_ENABLE: R3.1, U1.14/P409
- new net A1M0_HLFB: U1.13/P410, U9.E(1)
- new net A1M0_STEP: R1.1, U1.16/P407
- new net A1M1_DIR: R10.1, U1.3/P402
- new net A1M1_ENABLE: R11.1, U1.2/P401
- new net A1M1_HLFB: U1.1/P400, U17.E(1)
- new net A1M1_STEP: R9.1, U1.12/P411
- new net AN07: J4.2, R5.2, U1.61/P003
- new net AN16: J1.2, R6.2, U1.49/P500
- new net DAC: J6.2, U1.54/P014
- new net DFI_01: U1.50/P501
- new net DFI_02: U1.62/P002
- new net DFO_01: U1.30/P302
- new net DFO_02: U1.41/P107
- new net DFO_03: U1.42/P106
- new net ESTOP: U1.27/P200
- new net HLFB_RETURN: J2.1, J5.1, R12.1, R4.1
- new net LS_01: R40.2, R41.2, U1.23/P205, U28.E(1)
- new net LS_02: R43.2, R44.2, U1.53/P015, U29.E(1)
- new net LS_03: R52.2, R53.2, U1.64/P000, U32.E(1)
- new net LS_04: R55.2, R56.2, U1.63/P001, U33.E(1)
- new net LS_RET: J16.2, J17.2, J20.2, J21.2, R39.1, R42.1, R51.1, R54.1
- new net MISO: U1.48/P100
- new net MOSI: U1.47/P101
- new net N$1: R2.2, U3.B(2)
- new net N$10: R11.2, U12.B(2)
- new net N$11: R9.2, U10.B(2)
- new net N$12: R12.2, U17.B(2)
- new net N$2: R3.2, U4.B(2)
- new net N$20: R19.2, U19.B(2)
- new net N$21: J7.2, LED2.C, U19.C(3)
- new net N$22: LED2.A, R20.1
- new net N$26: R23.2, U21.B(2)
- new net N$27: J9.2, LED4.C, U21.C(3)
- new net N$28: LED4.A, R24.1
- new net N$32: R27.2, U23.B(2)
- new net N$33: J11.2, LED6.C, U23.C(3)
- new net N$34: LED6.A, R28.1
- new net N$38: R31.2, U25.B(2)
- new net N$39: J13.2, LED8.C, U25.C(3)
- new net N$4: R4.2, U9.B(2)
- new net N$40: LED8.A, R32.1
- new net N$45: R39.2, U28.B(2)
- new net N$46: LED11.A, R40.1
- new net N$47: R42.2, U29.B(2)
- new net N$48: LED12.A, R43.1
- new net N$53: R51.2, U32.B(2)
- new net N$54: LED15.A, R52.1
- new net N$55: R54.2, U33.B(2)
- new net N$56: LED16.A, R55.1
- new net N$69: U1.18/USB_DM
- new net N$70: U1.19/USB_DP
- new net N$76: U1.26/P201/MD
- new net N$82: U1.36/P111
- new net N$83: U1.37/P112
- new net N$86: U1.40/VCL
- new net N$89: U1.43/P105
- new net N$9: R10.2, U11.B(2)
- new net N$90: U1.44/P104
- new net RELAY_1: R19.1, U1.24/P204
- new net RELAY_2: R23.1, U1.21/P207
- new net RELAY_3: R27.1, U1.22/P206
- new net RELAY_4: R31.1, U1.31/P301
- new net RESET: C16.1, J3.9, R13.1, U1.25/RES
- new net SCLK: U1.46/P102
- new net SSL0: U1.45/P103
- new net TCK: J3.7, U1.32/P300/TCK/SWCLK
- new net TDI: J3.1, U1.35/P110/TDI
- new net TDO: J3.3, U1.34/P109/TDO/SWO
- new net TMS: J3.5, U1.33/P108/TMS/SWDIO
- new net VBATT: U1.4/VBATT
- new net VCL0: C6.2, U1.5/VCL0
- new net VDD: C1.1, C10.1, C11.1, C3.1, C4.1, C5.1, C7.2, C8.1, C9.1, J3.2, J3.4, R13.2, R5.1, R6.1, U1.11/VCC, U1.20/VCC_USB, U1.29/VCC, U1.38/VCC, U1.51/VCC, U1.56/VREFH, U1.57/AVCC0, U1.60/VREFH0, U17.C(3), U28.C(3), U29.C(3), U32.C(3), U33.C(3), U9.C(3)
- new net VDD5: J11.1, J13.1, J7.1, J9.1, R20.2, R24.2, R28.2, R32.2
- new net XCIN: C32.1, U1.6/XCIN, X3.P$1
- new net XCOUT: C37.1, U1.7/XCOUT, X3.P$2
- new net XTAL1: C17.1, U1.9/XTAL, Y1.3
- new net XTAL2: C18.1, U1.10/EXTAL, Y1.1
- net GND: now also C1.2, C10.2, C11.2, C16.2, C17.2, C18.2, C3.2, C32.2, C37.2, C4.2, C5.2, C6.1, C7.1, C8.2, C9.2, J16.1, J17.1, J20.1, J21.1, J3.10, J3.6, J3.8, J4.1, J6.1, LED11.C, LED12.C, LED15.C, LED16.C, R41.1, R44.1, R53.1, R56.1, U1.17/VSS_USB, U1.28/VSS, U1.39/VSS, U1.52/VSS, U1.55/VREFL, U1.58/AVSS0, U1.59/VREFL0, U1.8/VSS, U10.E(1), U11.E(1), U12.E(1), U19.E(1), U2.E(1), U21.E(1), U23.E(1), U25.E(1), U3.E(1), U4.E(1), Y1.2, Y1.4; no longer U5.E(1), U6.E(1), U7.E(1)
- net MO_DIR: now also J2.3, J5.3, U11.C(3), U3.C(3); no longer J1.3, U6.C(3)
- net MO_ENABLE: now also J2.2, J5.2, U12.C(3), U4.C(3); no longer J1.2, U7.C(3)
- net MO_STEP: now also J2.4, J5.4, U10.C(3), U2.C(3); no longer J1.4, U5.C(3)
- net N$3: now also R1.2, U2.B(2); no longer R5.2, U6.B(2)
Other:
- note added: "JTAG"
- moved on the sheet: R4, R5, R6

Commit message: Update
Parts:
- removed J3: 10-pos, 3D_MIG_Controller:CONN_05X2_RAPTH
- added J8: CONN_530470610_PICOBLADE_X_6, 3D_MIG_Controller:CONN_530470610_PICOBLADE_X_6
Connections:
- net A1M0_DIR renamed DIR_M0A1
- net A1M0_ENABLE renamed ENABLE_M0A1
- net A1M0_HLFB renamed HLFB_M0A1
- net A1M0_STEP renamed STEP_M0A1
- net A1M1_DIR renamed DIR_M1A1
- net A1M1_ENABLE renamed ENABLE_M1A1
- net A1M1_HLFB renamed HLFB_M1A1
- net A1M1_STEP renamed STEP_M1A1
- net AN07 renamed AN07_A1
- net AN16 renamed AN16_A1
- net DAC renamed DAC_A1
- net DFI_01 renamed DFI_01_A1
- net DFI_02 renamed DFI_02_A1
- net DFO_01 renamed DFO_01_A1
- net DFO_02 renamed DFO_02_A1
- net DFO_03 renamed DFO_03_A1
- net ESTOP renamed ESTOP_A1
- net LS_01 renamed LS_01_A1
- net LS_02 renamed LS_02_A1
- net LS_03 renamed LS_03_A1
- net LS_04 renamed LS_04_A1
- net RELAY_1 renamed RELAY_1_A1
- net RELAY_2 renamed RELAY_2_A1
- net RELAY_3 renamed RELAY_3_A1
- net RELAY_4 renamed RELAY_4_A1
- net SSL0 renamed SSL0_A1
- net VBATT renamed VBATT_M1A1
- net VCL0 renamed VCL0_A1
- net XCIN renamed XCIN_A1
- net XCOUT renamed XCOUT_A1
- net XTAL1 renamed XTAL1_A1
- net XTAL2 renamed XTAL2_A1
- removed net HLFB_RETURN: J2.1, J5.1, R12.1, R4.1
- removed net LS_RET: J16.2, J17.2, J20.2, J21.2, R39.1, R42.1, R51.1, R54.1
- removed net MO_DIR: J2.3, J5.3, U11.C(3), U3.C(3)
- removed net MO_ENABLE: J2.2, J5.2, U12.C(3), U4.C(3)
- removed net MO_STEP: J2.4, J5.4, U10.C(3), U2.C(3)
- removed net RESET: C16.1, J3.9, R13.1, U1.25/RES
- removed net TCK: J3.7, U1.32/P300/TCK/SWCLK
- removed net TDI: J3.1, U1.35/P110/TDI
- removed net TDO: J3.3, U1.34/P109/TDO/SWO
- removed net TMS: J3.5, U1.33/P108/TMS/SWDIO
- new net HLFB_RETURN_M0_A1: J2.1, R4.1
- new net HLFB_RETURN_M1_A1: J5.1, R12.1
- new net LS_01_RET_A1: J16.2, R39.1
- new net LS_02_RET_A1: J17.2, R42.1
- new net LS_03_RET_A1: J20.2, R51.1
- new net LS_04_RET_A1: J21.2, R54.1
- new net MO_DIR_M0_A1: J2.3, U3.C(3)
- new net MO_DIR_M1_A1: J5.3, U11.C(3)
- new net MO_ENABLE_M0_A1: J2.2, U4.C(3)
- new net MO_ENABLE_M1_A1: J5.2, U12.C(3)
- new net MO_STEP_M0_A1: J2.4, U2.C(3)
- new net MO_STEP_M1_A1: J5.4, U10.C(3)
- new net RESET_A1: C16.1, J8.2, R13.1, U1.25/RES
- new net TCK_A1: J8.6, U1.32/P300/TCK/SWCLK
- new net TDI_A1: J8.3, U1.35/P110/TDI
- new net TDO_A1: J8.4, U1.34/P109/TDO/SWO
- new net TMS_A1: J8.5, U1.33/P108/TMS/SWDIO
- net GND: now also J8.1; no longer J3.10, J3.6, J3.8
- net VDD: no longer J3.2, J3.4
Other:
- moved on the sheet: C16, C5, R13

Commit message: Update
Parts:
- removed C1, C10, C3, C4, C5, C6, C7, C8, C9: 0.1uF, 3D_MIG_Controller:C_0402_0.1UF
- removed C11: 1uF, 3D_MIG_Controller:C_0402_1UF
- removed C16: 10uF, 3D_MIG_Controller:C_0402_10UF
- removed C17, C18: 10pF, 3D_MIG_Controller:C_0402
- removed C32, C37: 12pF, 3D_MIG_Controller:C_0402_12PF
- removed J11, J13, J16, J17, J20, J21, J4, J6, J7, J9: (no value), 3D_MIG_Controller:CONN_530470210_PICOBLADE_X_2
- removed J2, J5: CONN_530470410_PICOBLADE_X_4, 3D_MIG_Controller:CONN_530470410_PICOBLADE_X_4
- removed J8: CONN_530470610_PICOBLADE_X_6, 3D_MIG_Controller:CONN_530470610_PICOBLADE_X_6
- removed LED11, LED12, LED15, LED16, LED2, LED4, LED6, LED8: Green, 3D_MIG_Controller:LED_0805_GREEN
- removed R1, R10, R11, R12, R2, R3, R4, R9: 33R0, 3D_MIG_Controller:R_0402_33R0
- removed R13, R41, R44, R53, R56: 10K0, 3D_MIG_Controller:R_0402_10K0
- removed R19, R23, R27, R31: 500R0, 3D_MIG_Controller:R_0402
- removed R20, R24, R28, R32, R40, R43, R52, R55: 470R0, 3D_MIG_Controller:R_0402_470R0
- removed R39, R42, R51, R54: 2.2K, 3D_MIG_Controller:R_0402
- removed R5, R6: (no value), 3D_MIG_Controller:R_0402
- removed U1: RENESAS_R7FS5D37A3A01CFM#AA0PLQP0064KB-C_REN-M, 3D_MIG_Controller:RENESAS_R7FS5D37A3A01CFM#AA0PLQP0064KB-C_REN-M
- removed U10, U11, U12, U17, U19, U2, U21, U23, U25, U28, U29, U3, U32, U33, U4, U9: NPN, 3D_MIG_Controller:BC846BW
- removed X3: 32.768KHz, 3D_MIG_Controller:XTAL_32.768KHZ
- removed Y1: XTAL_12MHZ_ABM8G-12.000MHZ-B4Y-T, 3D_MIG_Controller:XTAL_12MHZ_ABM8G-12.000MHZ-B4Y-T
- added C12, C2: 12pF, 3D_MIG_Controller:C_0402_12PF
- added C13, C14: 10pF, 3D_MIG_Controller:C_0402_10PF
- added C15, C19, C20, C21, C22, C23, C24, C25, C26: 0.1uF, 3D_MIG_Controller:C_0402_0.1UF
- added C27: 1uF, 3D_MIG_Controller:C_0402_1UF
- added C28: 10uF, 3D_MIG_Controller:C_0402_10UF
- added J10, J3: CONN_530470410_PICOBLADE_X_4, 3D_MIG_Controller:CONN_530470410_PICOBLADE_X_4
- added J12, J14, J15, J18, J19, J22, J23, J24, J25, J26, J27: (no value), 3D_MIG_Controller:CONN_530470210_PICOBLADE_X_2
- added J28: CONN_530470610_PICOBLADE_X_6, 3D_MIG_Controller:CONN_530470610_PICOBLADE_X_6
- added J29: (no value), 3D_MIG_Controller:CONN_05X2PTH
- added LED1, LED10, LED13, LED14, LED3, LED5, LED7, LED9: Green, 3D_MIG_Controller:LED_0805_GREEN
- added R14, R15, R16, R17, R18, R21, R7, R8: 33R0, 3D_MIG_Controller:R_0402_33R0
- added R22, R25, R26, R29, R30, R33, R34, R35, R37, R46, R49, R58: 470R0, 3D_MIG_Controller:R_0402_470R0
- added R36, R45, R48, R57: 2K2, 3D_MIG_Controller:R_0402_2K2
- added R38, R47, R50, R59, R62: 10K0, 3D_MIG_Controller:R_0402_10K0
- added R60, R61: 100K0, 3D_MIG_Controller:R_0402_100K0
- added U13, U14, U15, U16, U18, U20, U22, U24, U26, U27, U30, U31, U34, U6, U7, U8: NPN, 3D_MIG_Controller:BC846BW
- added U5: RENESAS_R7FS5D37A3A01CFM#AA0PLQP0064KB-C_REN-M, 3D_MIG_Controller:RENESAS_R7FS5D37A3A01CFM#AA0PLQP0064KB-C_REN-M
- added X1: 32.768KHz, 3D_MIG_Controller:XTAL_32.768KHZ
- added Y2: XTAL_12MHZ_ABM8G-12.000MHZ-B4Y-T, 3D_MIG_Controller:XTAL_12MHZ_ABM8G-12.000MHZ-B4Y-T
- J1: value (none) -> 4-pos; device 3D_MIG_Controller:CONN_530470210_PICOBLADE_X_2 -> 3D_MIG_Controller:3.81MM_1_X_4_RT_ANGLE_PLUG_HEADER
Connections:
- removed net N$1: R2.2, U3.B(2)
- removed net N$10: R11.2, U12.B(2)
- removed net N$11: R9.2, U10.B(2)
- removed net N$12: R12.2, U17.B(2)
- removed net N$2: R3.2, U4.B(2)
- removed net N$20: R19.2, U19.B(2)
- removed net N$21: J7.2, LED2.C, U19.C(3)
- removed net N$22: LED2.A, R20.1
- removed net N$26: R23.2, U21.B(2)
- removed net N$27: J9.2, LED4.C, U21.C(3)
- removed net N$28: LED4.A, R24.1
- removed net N$3: R1.2, U2.B(2)
- removed net N$32: R27.2, U23.B(2)
- removed net N$33: J11.2, LED6.C, U23.C(3)
- removed net N$34: LED6.A, R28.1
- removed net N$38: R31.2, U25.B(2)
- removed net N$39: J13.2, LED8.C, U25.C(3)
- removed net N$4: R4.2, U9.B(2)
- removed net N$40: LED8.A, R32.1
- removed net N$45: R39.2, U28.B(2)
- removed net N$46: LED11.A, R40.1
- removed net N$47: R42.2, U29.B(2)
- removed net N$48: LED12.A, R43.1
- removed net N$53: R51.2, U32.B(2)
- removed net N$54: LED15.A, R52.1
- removed net N$55: R54.2, U33.B(2)
- removed net N$56: LED16.A, R55.1
- removed net N$9: R10.2, U11.B(2)
- new net N$14: R7.2, U6.B(2)
- new net N$15: R15.2, U13.B(2)
- new net N$16: R17.2, U15.B(2)
- new net N$17: R18.2, U16.B(2)
- new net N$18: R16.2, U14.B(2)
- new net N$19: R21.2, U18.B(2)
- new net N$23: R22.2, U20.B(2)
- new net N$24: J12.2, LED1.C, U20.C(3)
- new net N$25: LED1.A, R25.1
- new net N$29: R26.2, U22.B(2)
- new net N$30: J14.2, LED3.C, U22.C(3)
- new net N$31: LED3.A, R29.1
- new net N$35: R30.2, U24.B(2)
- new net N$36: J15.2, LED5.C, U24.C(3)
- new net N$37: LED5.A, R33.1
- new net N$41: R34.2, U26.B(2)
- new net N$42: J18.2, LED7.C, U26.C(3)
- new net N$43: LED7.A, R35.1
- new net N$44: R36.2, U27.B(2)
- new net N$49: LED9.A, R37.1
- new net N$50: R45.2, U30.B(2)
- new net N$51: LED10.A, R46.1
- new net N$52: R48.2, U31.B(2)
- new net N$57: LED13.A, R49.1
- new net N$58: R57.2, U34.B(2)
- new net N$59: LED14.A, R58.1
- new net N$6: R8.2, U7.B(2)
- new net N$7: R14.2, U8.B(2)
- new net VDD12: J1.P$4
- net AN07_A1: now also J26.2, R60.2, U5.61/P003; no longer J4.2, R5.2, U1.61/P003
- net AN16_A1: now also J25.2, R61.2, U5.49/P500; no longer J1.2, R6.2, U1.49/P500
- net DAC_A1: now also J27.2, U5.54/P014; no longer J6.2, U1.54/P014
- net DFI_01_A1: now also U5.50/P501; no longer U1.50/P501
- net DFI_02_A1: now also U5.62/P002; no longer U1.62/P002
- net DFO_01_A1: now also U5.30/P302; no longer U1.30/P302
- net DFO_02_A1: now also U5.41/P107; no longer U1.41/P107
- net DFO_03_A1: now also U5.42/P106; no longer U1.42/P106
- net DIR_M0A1: now also R8.1, U5.15/P408; no longer R2.1, U1.15/P408
- net DIR_M1A1: now also R17.1, U5.3/P402; no longer R10.1, U1.3/P402
- net ENABLE_M0A1: now also R14.1, U5.14/P409; no longer R3.1, U1.14/P409
- net ENABLE_M1A1: now also R18.1, U5.2/P401; no longer R11.1, U1.2/P401
- net ESTOP_A1: now also U5.27/P200; no longer U1.27/P200
- net GND: now also C12.2, C13.2, C14.2, C15.2, C19.2, C2.2, C20.2, C21.2, C22.1, C23.1, C24.2, C25.2, C26.2, C27.2, C28.2, J1.P$1, J19.1, J22.1, J23.1, J24.1, J25.1, J26.1, J27.1, J28.1, J29.1, J29.2, LED10.C, LED13.C, LED14.C, LED9.C, R38.1, R47.1, R50.1, R59.1, U14.E(1), U15.E(1), U16.E(1), U20.E(1), U22.E(1), U24.E(1), U26.E(1), U5.17/VSS_USB, U5.28/VSS, U5.39/VSS, U5.52/VSS, U5.55/VREFL, U5.58/AVSS0, U5.59/VREFL0, U5.8/VSS, U6.E(1), U7.E(1), U8.E(1), Y2.2, Y2.4; no longer C1.2, C10.2, C11.2, C16.2, C17.2, C18.2, C3.2, C32.2, C37.2, C4.2, C5.2, C6.1, C7.1, C8.2, C9.2, J1.1, J16.1, J17.1, J20.1, J21.1, J4.1, J6.1, J8.1, LED11.C, LED12.C, LED15.C, LED16.C, R41.1, R44.1, R53.1, R56.1, U1.17/VSS_USB, U1.28/VSS, U1.39/VSS, U1.52/VSS, U1.55/VREFL, U1.58/AVSS0, U1.59/VREFL0, U1.8/VSS, U10.E(1), U11.E(1), U12.E(1), U19.E(1), U2.E(1), U21.E(1), U23.E(1), U25.E(1), U3.E(1), U4.E(1), Y1.2, Y1.4
- net HLFB_M0A1: now also U13.E(1), U5.13/P410; no longer U1.13/P410, U9.E(1)
- net HLFB_M1A1: now also U18.E(1), U5.1/P400; no longer U1.1/P400, U17.E(1)
- net HLFB_RETURN_M0_A1: now also J3.1, R15.1; no longer J2.1, R4.1
- net HLFB_RETURN_M1_A1: now also J10.1, R21.1; no longer J5.1, R12.1
- net LS_01_A1: now also R37.2, R38.2, U27.E(1), U5.23/P205; no longer R40.2, R41.2, U1.23/P205, U28.E(1)
- net LS_01_RET_A1: now also J19.2, R36.1; no longer J16.2, R39.1
- net LS_02_A1: now also R46.2, R47.2, U30.E(1), U5.53/P015; no longer R43.2, R44.2, U1.53/P015, U29.E(1)
- net LS_02_RET_A1: now also J22.2, R45.1; no longer J17.2, R42.1
- net LS_03_A1: now also R49.2, R50.2, U31.E(1), U5.64/P000; no longer R52.2, R53.2, U1.64/P000, U32.E(1)
- net LS_03_RET_A1: now also J23.2, R48.1; no longer J20.2, R51.1
- net LS_04_A1: now also R58.2, R59.2, U34.E(1), U5.63/P001; no longer R55.2, R56.2, U1.63/P001, U33.E(1)
- net LS_04_RET_A1: now also J24.2, R57.1; no longer J21.2, R54.1
- net MISO: now also J29.10, J29.9, U5.48/P100; no longer U1.48/P100
- net MOSI: now also J29.7, J29.8, U5.47/P101; no longer U1.47/P101
- net MO_DIR_M0_A1: now also J3.3, U7.C(3); no longer J2.3, U3.C(3)
- net MO_DIR_M1_A1: now also J10.3, U15.C(3); no longer J5.3, U11.C(3)
- net MO_ENABLE_M0_A1: now also J3.2, U8.C(3); no longer J2.2, U4.C(3)
- net MO_ENABLE_M1_A1: now also J10.2, U16.C(3); no longer J5.2, U12.C(3)
- net MO_STEP_M0_A1: now also J3.4, U6.C(3); no longer J2.4, U2.C(3)
- net MO_STEP_M1_A1: now also J10.4, U14.C(3); no longer J5.4, U10.C(3)
- net N$69: now also U5.18/USB_DM; no longer U1.18/USB_DM
- net N$70: now also U5.19/USB_DP; no longer U1.19/USB_DP
- net N$76: now also U5.26/P201/MD; no longer U1.26/P201/MD
- net N$82: now also U5.36/P111; no longer U1.36/P111
- net N$83: now also U5.37/P112; no longer U1.37/P112
- net N$86: now also U5.40/VCL; no longer U1.40/VCL
- net N$89: now also U5.43/P105; no longer U1.43/P105
- net N$90: now also U5.44/P104; no longer U1.44/P104
- net RELAY_1_A1: now also R22.1, U5.24/P204; no longer R19.1, U1.24/P204
- net RELAY_2_A1: now also R26.1, U5.21/P207; no longer R23.1, U1.21/P207
- net RELAY_3_A1: now also R30.1, U5.22/P206; no longer R27.1, U1.22/P206
- net RELAY_4_A1: now also R34.1, U5.31/P301; no longer R31.1, U1.31/P301
- net RESET_A1: now also C28.1, J28.2, R62.1, U5.25/RES; no longer C16.1, J8.2, R13.1, U1.25/RES
- net SCLK: now also J29.5, J29.6, U5.46/P102; no longer U1.46/P102
- net SSL0_A1: now also J29.3, J29.4, U5.45/P103; no longer U1.45/P103
- net STEP_M0A1: now also R7.1, U5.16/P407; no longer R1.1, U1.16/P407
- net STEP_M1A1: now also R16.1, U5.12/P411; no longer R9.1, U1.12/P411
- net TCK_A1: now also J28.6, U5.32/P300/TCK/SWCLK; no longer J8.6, U1.32/P300/TCK/SWCLK
- net TDI_A1: now also J28.3, U5.35/P110/TDI; no longer J8.3, U1.35/P110/TDI
- net TDO_A1: now also J28.4, U5.34/P109/TDO/SWO; no longer J8.4, U1.34/P109/TDO/SWO
- net TMS_A1: now also J28.5, U5.33/P108/TMS/SWDIO; no longer J8.5, U1.33/P108/TMS/SWDIO
- net VBATT_M1A1: now also U5.4/VBATT; no longer U1.4/VBATT
- net VCL0_A1: now also C22.2, U5.5/VCL0; no longer C6.2, U1.5/VCL0
- net VDD: now also C15.1, C19.1, C20.1, C21.1, C23.2, C24.1, C25.1, C26.1, C27.1, J1.P$2, R60.1, R61.1, R62.2, U13.C(3), U18.C(3), U27.C(3), U30.C(3), U31.C(3), U34.C(3), U5.11/VCC, U5.20/VCC_USB, U5.29/VCC, U5.38/VCC, U5.51/VCC, U5.56/VREFH, U5.57/AVCC0, U5.60/VREFH0; no longer C1.1, C10.1, C11.1, C3.1, C4.1, C5.1, C7.2, C8.1, C9.1, R13.2, R5.1, R6.1, U1.11/VCC, U1.20/VCC_USB, U1.29/VCC, U1.38/VCC, U1.51/VCC, U1.56/VREFH, U1.57/AVCC0, U1.60/VREFH0, U17.C(3), U28.C(3), U29.C(3), U32.C(3), U33.C(3), U9.C(3)
- net VDD5: now also J1.P$3, J12.1, J14.1, J15.1, J18.1, R25.2, R29.2, R33.2, R35.2; no longer J11.1, J13.1, J7.1, J9.1, R20.2, R24.2, R28.2, R32.2
- net XCIN_A1: now also C2.1, U5.6/XCIN, X1.P$1; no longer C32.1, U1.6/XCIN, X3.P$1
- net XCOUT_A1: now also C12.1, U5.7/XCOUT, X1.P$2; no longer C37.1, U1.7/XCOUT, X3.P$2
- net XTAL1_A1: now also C13.1, U5.9/XTAL, Y2.3; no longer C17.1, U1.9/XTAL, Y1.3
- net XTAL2_A1: now also C14.1, U5.10/EXTAL, Y2.1; no longer C18.1, U1.10/EXTAL, Y1.1
Other:
- note added: "SPI"
