File: SPI_Test/SPI_Test.brd (EAGLE design)
At the start: 120 x 145 mm, 164 parts, among them J1 10-pos, J10 10-pos, J12 10-pos, J13 4-pos, J16 10-pos, J4 10-pos, J6 10-pos, J8 10-pos, U1 RENESAS_R7FS5D37A3A01CFM#AA0P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, U2 S7G2LQFP176, U3 RENESAS_R7FS5D37A3A01CFM#AA0P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, U4 RENESAS_R7FS5D37A3A01CFM#AA0P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, U6 RENESAS_R7FS5D37A3A01CFM#AA0P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, U7 RENESAS_R7FS5D37A3A01CFM#AA0P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, U9 RENESAS_R7FS5D37A3A01CFM#AA0P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, X10 32.768KHz, X2 32.768KHz, X3 32.768KHz, X4 24MHz, X5 32.768KHz, X6 32.768KHz, X7 32.768KHz, X8 32.768KHz, Y1 XTAL_12MHZ_ABM8G-12.000MHZ-B4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, Y3 XTAL_12MHZ_ABM8G-12.000MHZ-B4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, Y4 XTAL_12MHZ_ABM8G-12.000MHZ-B4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, Y5 XTAL_12MHZ_ABM8G-12.000MHZ-B4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, Y6 XTAL_12MHZ_ABM8G-12.000MHZ-B4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, Y8 XTAL_12MHZ_ABM8G-12.000MHZ-B4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

Commit message: Update
Parts:
- removed C102, C132, C38, C72, C86: 10pF, 3D_MIG_Controller:0402
- removed C103, C104, C105, C106, C107, C108, C109, C110, C111, C133, C134, C135, C136, C137, C138, C139, C140, C141, C73, C74, C75, C76, C77, C78, C79, C80, C81: 0.1uF, 3D_MIG_Controller:0402
- removed C112, C142, C82: 1uF, 3D_MIG_Controller:0402
- removed C113, C143, C83: 10uF, 3D_MIG_Controller:0402
- removed C36, C37, C84, C85: 12pF, 3D_MIG_Controller:0402
- removed J11, J7: (no value), 3D_MIG_Controller:2X5
- removed J12, J16, J8: 10-pos, 3D_MIG_Controller:2X5
- removed R11, R7, R9: 10K0, 3D_MIG_Controller:0402
- removed U4, U7, U9: RENESAS_R7FS5D37A3A01CFM#AA0PLQP0064KB-C_REN-M, 3D_MIG_Controller:PLQP0064KB-C_REN-M
- removed X10, X6, X8: 32.768KHz, 3D_MIG_Controller:SMD_X_2_PADS
- removed Y4, Y6, Y8: XTAL_12MHZ_ABM8G-12.000MHZ-B4Y-T, 3D_MIG_Controller:CRYSTAL_ABM8G_ABR
- added C117, C118, C147, C148, C177, C178: 12pF, 3D_MIG_Controller:0402
- added C119, C120, C149, C150, C179, C180: 10pF, 3D_MIG_Controller:0402
- added C121, C122, C123, C124, C125, C126, C127, C128, C151, C152, C153, C154, C155, C156, C157, C158, C159, C181, C182, C183, C184, C185, C186, C187, C188, C189: 0.1uF, 3D_MIG_Controller:0402
- added C160, C190: 1uF, 3D_MIG_Controller:0402
- added C161, C191: 10uF, 3D_MIG_Controller:0402
- added J14, J18, J22: (no value), 3D_MIG_Controller:2X5
- added J19, J23: 10-pos, 3D_MIG_Controller:2X5
- added R10, R13, R15: 10K0, 3D_MIG_Controller:0402
- added U10, U12, U8: RENESAS_R7FS5D37A3A01CFM#AA0PLQP0064KB-C_REN-M, 3D_MIG_Controller:PLQP0064KB-C_REN-M
- added X11, X13, X9: 32.768KHz, 3D_MIG_Controller:SMD_X_2_PADS
- added Y11, Y7, Y9: XTAL_12MHZ_ABM8G-12.000MHZ-B4Y-T, 3D_MIG_Controller:CRYSTAL_ABM8G_ABR
- C100, C130, C55, C70: value 12pF -> 1uF
- C101, C131, C56, C71: value 10pF -> 10uF
- C129, C54, C69, C99: value 12pF -> 0.1uF
- C39, C57, C87: value 10pF -> 12pF
- C40, C58, C88: value 0.1uF -> 12pF
- C41, C42, C59, C60, C89, C90: value 0.1uF -> 10pF
- C52, C67, C97: value 1uF -> 0.1uF
- C53, C68, C98: value 10uF -> 0.1uF
- J15: value (none) -> 10-pos
- moved C101 86.3 mm to (85.2, 131.9), turned to 180 degrees
- moved C99 81.9 mm to (89.0, 124.3), turned to 180 degrees
- moved C129 80.4 mm to (101.6, 92.8), turned to 90 degrees
- moved C131 79.9 mm to (109.2, 96.5), turned to 90 degrees
- moved C100 79.0 mm to (108.3, 126.6), turned to 90 degrees
- moved J15 78.8 mm to (94.9, 96.8), turned to 0 degrees
- moved C90 62.2 mm to (91.9, 135.6), turned to 270 degrees
- moved C95 59.6 mm to (102.3, 133.8), turned to 270 degrees
- moved C94 59.0 mm to (83.2, 131.9)
- moved C130 58.4 mm to (103.9, 73.5), turned to 0 degrees
- moved X7 58.3 mm to (100.5, 137.6), turned to 270 degrees
- moved C69 58.1 mm to (48.0, 124.3), turned to 180 degrees
- moved C71 56.6 mm to (44.4, 131.9), turned to 180 degrees
- moved C54 56.3 mm to (11.1, 124.2), turned to 180 degrees
- moved C56 54.8 mm to (7.35, 131.8), turned to 180 degrees
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Connections:
- removed net GNDS: J13.P$4
- removed net VDD5: J13.P$3
- net DFI_01_A1: now also U10.50, U12.50, U8.50; no longer U4.50, U7.50, U9.50
- net DFI_02_A1: now also U10.62, U12.62, U8.62; no longer U4.62, U7.62, U9.62
- net DFO_01_A1: now also U10.30, U12.30, U8.30; no longer U4.30, U7.30, U9.30
- net DFO_02_A1: now also U10.41, U12.41, U8.41; no longer U4.41, U7.41, U9.41
- net DFO_03_A1: now also U10.42, U12.42, U8.42; no longer U4.42, U7.42, U9.42
- net DIR_M0A1: now also U10.15, U12.15, U8.15; no longer U4.15, U7.15, U9.15
- net DIR_M1A1: now also U10.3, U12.3, U8.3; no longer U4.3, U7.3, U9.3
- net ENABLE_M0A1: now also U10.14, U12.14, U8.14; no longer U4.14, U7.14, U9.14
- net ENABLE_M1A1: now also U10.2, U12.2, U8.2; no longer U4.2, U7.2, U9.2
- net ESTOP_A1: now also U10.27, U12.27, U8.27; no longer U4.27, U7.27, U9.27
- net GND: now also C117.P$2, C118.P$2, C119.P$2, C120.P$2, C121.P$2, C122.P$2, C123.P$2, C124.P$2, C125.P$1, C126.P$1, C127.P$2, C128.P$2, C147.P$2, C148.P$2, C149.P$2, C150.P$2, C151.P$2, C152.P$2, C153.P$2, C154.P$2, C155.P$1, C156.P$1, C157.P$2, C158.P$2, C159.P$2, C160.P$2, C161.P$2, C177.P$2, C178.P$2, C179.P$2, C180.P$2, C181.P$2, C182.P$2, C183.P$2, C184.P$2, C185.P$1, C186.P$1, C187.P$2, C188.P$2, C189.P$2, C190.P$2, C191.P$2, C47.P$2, C48.P$2, C50.P$1, C51.P$1, C62.P$2, C63.P$2, C65.P$1, C66.P$1, C92.P$2, C93.P$2, C95.P$1, C96.P$1, J13.P$3, J13.P$4, J14.1, J14.2, J15.10, J15.6, J15.8, J18.1, J18.2, J19.10, J19.6, J19.8, J22.1, J22.2, J23.10, J23.6, J23.8, U10.17, U10.28, U10.39, U10.55, U10.58, U10.59, U10.8, U12.17, U12.28, U12.39, U12.55, U12.58, U12.59, U12.8, U8.17, U8.28, U8.39, U8.55, U8.58, U8.59, U8.8, Y11.2, Y11.4, Y7.2, Y7.4, Y9.2, Y9.4; no longer C102.P$2, C103.P$2, C104.P$2, C105.P$2, C106.P$2, C107.P$1, C108.P$1, C109.P$2, C110.P$2, C111.P$2, C112.P$2, C113.P$2, C132.P$2, C133.P$2, C134.P$2, C135.P$2, C136.P$2, C137.P$1, C138.P$1, C139.P$2, C140.P$2, C141.P$2, C142.P$2, C143.P$2, C36.P$2, C37.P$2, C38.P$2, C47.P$1, C48.P$1, C50.P$2, C51.P$2, C62.P$1, C63.P$1, C65.P$2, C66.P$2, C72.P$2, C73.P$2, C74.P$2, C75.P$2, C76.P$2, C77.P$1, C78.P$1, C79.P$2, C80.P$2, C81.P$2, C82.P$2, C83.P$2, C84.P$2, C85.P$2, C86.P$2, C92.P$1, C93.P$1, C95.P$2, C96.P$2, J11.1, J11.2, J12.10, J12.6, J12.8, J15.1, J15.2, J16.10, J16.6, J16.8, J7.1, J7.2, J8.10, J8.6, J8.8, U4.17, U4.28, U4.39, U4.55, U4.58, U4.59, U4.8, U7.17, U7.28, U7.39, U7.55, U7.58, U7.59, U7.8, U9.17, U9.28, U9.39, U9.55, U9.58, U9.59, U9.8, Y4.2, Y4.4, Y6.2, Y6.4, Y8.2, Y8.4
- net HLFB_M0A1: now also U10.13, U12.13, U8.13; no longer U4.13, U7.13, U9.13
- net HLFB_M1A1: now also U10.1, U12.1, U8.1; no longer U4.1, U7.1, U9.1
- net LS_01_A1: now also U10.23, U12.23, U8.23; no longer U4.23, U7.23, U9.23
- net LS_02_A1: now also U10.53, U12.53, U8.53; no longer U4.53, U7.53, U9.53
- net LS_03_A1: now also U10.64, U12.64, U8.64; no longer U4.64, U7.64, U9.64
- net LS_04_A1: now also U10.63, U12.63, U8.63; no longer U4.63, U7.63, U9.63
- net MISO: now also J14.10, J14.9, J18.10, J18.9, J22.10, J22.9, U10.48, U12.48, U8.48; no longer J11.10, J11.9, J15.10, J15.9, J7.10, J7.9, U4.48, U7.48, U9.48
- net MOSI: now also J14.7, J14.8, J18.7, J18.8, J22.7, J22.8, U10.47, U12.47, U8.47; no longer J11.7, J11.8, J15.7, J15.8, J7.7, J7.8, U4.47, U7.47, U9.47
- net N$69: now also U10.18, U12.18, U8.18; no longer U4.18, U7.18, U9.18
- net N$70: now also U10.19, U12.19, U8.19; no longer U4.19, U7.19, U9.19
- net N$76: now also U10.26, U12.26, U8.26; no longer U4.26, U7.26, U9.26
- net N$82: now also U10.36, U12.36, U8.36; no longer U4.36, U7.36, U9.36
- net N$83: now also U10.37, U12.37, U8.37; no longer U4.37, U7.37, U9.37
- net N$86: now also U10.40, U12.40, U8.40; no longer U4.40, U7.40, U9.40
- net N$89: now also U10.43, U12.43, U8.43; no longer U4.43, U7.43, U9.43
- net N$90: now also U10.44, U12.44, U8.44; no longer U4.44, U7.44, U9.44
- net RELAY_1_A1: now also U10.24, U12.24, U8.24; no longer U4.24, U7.24, U9.24
- net RELAY_2_A1: now also U10.21, U12.21, U8.21; no longer U4.21, U7.21, U9.21
- net RELAY_3_A1: now also U10.22, U12.22, U8.22; no longer U4.22, U7.22, U9.22
- net RELAY_4_A1: now also U10.31, U12.31, U8.31; no longer U4.31, U7.31, U9.31
- net RESET_A1: now also C101.P$1, C131.P$1, C161.P$1, C191.P$1, C56.P$1, C71.P$1, J15.9, J19.9, J23.9, R10.P$1, R13.P$1, R15.P$1, U10.25, U12.25, U8.25; no longer C113.P$1, C143.P$1, C53.P$1, C68.P$1, C83.P$1, C98.P$1, J12.9, J16.9, J8.9, R11.P$1, R7.P$1, R9.P$1, U4.25, U7.25, U9.25
- net SCLK: now also J14.5, J14.6, J18.5, J18.6, J22.5, J22.6, U10.46, U12.46, U8.46; no longer J11.5, J11.6, J15.5, J15.6, J7.5, J7.6, U4.46, U7.46, U9.46
- net SSL0_A1_03: now also J9.3, J9.4, U6.45; no longer J7.3, J7.4, U4.45
- net SSL0_A1_04: now also J14.3, J14.4, U8.45; no longer J9.3, J9.4, U6.45
- net SSL0_A1_05: now also J18.3, J18.4, U10.45; no longer J11.3, J11.4, U7.45
- net SSL0_A1_06: now also J22.3, J22.4, U12.45; no longer J15.3, J15.4, U9.45
- net STEP_M0A1: now also U10.16, U12.16, U8.16; no longer U4.16, U7.16, U9.16
- net STEP_M1A1: now also U10.12, U12.12, U8.12; no longer U4.12, U7.12, U9.12
- net TCK: now also J15.7, J19.7, J23.7, U10.32, U12.32, U8.32; no longer J12.7, J16.7, J8.7, U4.32, U7.32, U9.32
- net TDI: now also J15.1, J19.1, J23.1, U10.35, U12.35, U8.35; no longer J12.1, J16.1, J8.1, U4.35, U7.35, U9.35
- net TDO: now also J15.3, J19.3, J23.3, U10.34, U12.34, U8.34; no longer J12.3, J16.3, J8.3, U4.34, U7.34, U9.34
- net TMS: now also J15.5, J19.5, J23.5, U10.33, U12.33, U8.33; no longer J12.5, J16.5, J8.5, U4.33, U7.33, U9.33
- net VBATT_M1A1: now also U10.4, U12.4, U8.4; no longer U4.4, U7.4, U9.4
- net VCL0_A1: now also C125.P$2, C155.P$2, C185.P$2, C50.P$2, C65.P$2, C95.P$2, U10.5, U12.5, U8.5; no longer C107.P$2, C137.P$2, C47.P$2, C62.P$2, C77.P$2, C92.P$2, U4.5, U7.5, U9.5
- net VDD: now also C100.P$1, C121.P$1, C122.P$1, C123.P$1, C124.P$1, C126.P$2, C127.P$1, C128.P$1, C129.P$1, C130.P$1, C151.P$1, C152.P$1, C153.P$1, C154.P$1, C156.P$2, C157.P$1, C158.P$1, C159.P$1, C160.P$1, C181.P$1, C182.P$1, C183.P$1, C184.P$1, C186.P$2, C187.P$1, C188.P$1, C189.P$1, C190.P$1, C47.P$1, C48.P$1, C51.P$2, C53.P$1, C54.P$1, C55.P$1, C62.P$1, C63.P$1, C66.P$2, C68.P$1, C69.P$1, C70.P$1, C92.P$1, C93.P$1, C96.P$2, C98.P$1, C99.P$1, J15.2, J15.4, J19.2, J19.4, J23.2, J23.4, R10.P$2, R13.P$2, R15.P$2, U10.11, U10.20, U10.29, U10.38, U10.51, U10.56, U10.57, U10.60, U12.11, U12.20, U12.29, U12.38, U12.51, U12.56, U12.57, U12.60, U8.11, U8.20, U8.29, U8.38, U8.51, U8.56, U8.57, U8.60; no longer C103.P$1, C104.P$1, C105.P$1, C106.P$1, C108.P$2, C109.P$1, C110.P$1, C111.P$1, C112.P$1, C133.P$1, C134.P$1, C135.P$1, C136.P$1, C138.P$2, C139.P$1, C140.P$1, C141.P$1, C142.P$1, C40.P$1, C41.P$1, C42.P$1, C48.P$2, C50.P$1, C51.P$1, C58.P$1, C59.P$1, C60.P$1, C63.P$2, C65.P$1, C66.P$1, C73.P$1, C74.P$1, C75.P$1, C76.P$1, C78.P$2, C79.P$1, C80.P$1, C81.P$1, C82.P$1, C88.P$1, C89.P$1, C90.P$1, C93.P$2, C95.P$1, C96.P$1, J12.2, J12.4, J16.2, J16.4, J8.2, J8.4, R11.P$2, R7.P$2, R9.P$2, U4.11, U4.20, U4.29, U4.38, U4.51, U4.56, U4.57, U4.60, U7.11, U7.20, U7.29, U7.38, U7.51, U7.56, U7.57, U7.60, U9.11, U9.20, U9.29, U9.38, U9.51, U9.56, U9.57, U9.60
- net XCIN_A1: now also C117.P$1, C147.P$1, C177.P$1, C39.P$1, C57.P$1, C87.P$1, U10.6, U12.6, U8.6, X11.P$1, X13.P$1, X9.P$1; no longer C129.P$1, C36.P$1, C54.P$1, C69.P$1, C84.P$1, C99.P$1, U4.6, U7.6, U9.6, X10.P$1, X6.P$1, X8.P$1
- net XCOUT_A1: now also C118.P$1, C148.P$1, C178.P$1, C40.P$1, C58.P$1, C88.P$1, U10.7, U12.7, U8.7, X11.P$2, X13.P$2, X9.P$2; no longer C100.P$1, C130.P$1, C37.P$1, C55.P$1, C70.P$1, C85.P$1, U4.7, U7.7, U9.7, X10.P$2, X6.P$2, X8.P$2
- net XTAL1_A1: now also C119.P$1, C149.P$1, C179.P$1, C41.P$1, C59.P$1, C89.P$1, U10.9, U12.9, U8.9, Y11.3, Y7.3, Y9.3; no longer C101.P$1, C131.P$1, C38.P$1, C56.P$1, C71.P$1, C86.P$1, U4.9, U7.9, U9.9, Y4.3, Y6.3, Y8.3
- net XTAL2_A1: now also C120.P$1, C150.P$1, C180.P$1, C42.P$1, C60.P$1, C90.P$1, U10.10, U12.10, U8.10, Y11.1, Y7.1, Y9.1; no longer C102.P$1, C132.P$1, C39.P$1, C57.P$1, C72.P$1, C87.P$1, U4.10, U7.10, U9.10, Y4.1, Y6.1, Y8.1
Routing:
- net VDD: track 1063.3 -> 1112.3 mm, vias 50 -> 63
- net MISO: track 309.4 -> 340.0 mm, vias 13 -> 6
- net RESET: track 6.32 -> 34.9 mm, vias 1 -> 0
- net TDO: track 122.1 -> 93.6 mm, vias 7 -> 0
- net TMS: track 120.3 -> 92.6 mm, vias 7 -> 0
- net TDI: track 122.2 -> 96.3 mm, vias 7 -> 0
- net TCK: track 97.5 -> 76.7 mm, vias 7 -> 0
- net XTAL2_A1: track 61.5 -> 74.4 mm
- net MOSI: track 299.1 -> 311.9 mm, vias 13 -> 12
- net VCL0_A1: track 10.8 -> 22.8 mm
- net SCLK: track 295.2 -> 286.9 mm, vias 11 -> 6
- net RESET_A1: track 85.8 -> 93.1 mm
- net SSL0_A1_02: track 75.4 -> 81.1 mm
- net XCIN_A1: track 51.7 -> 47.1 mm
- net SSL0_A1_06: track 134.6 -> 138.9 mm
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