File: SPI_Test/SPI_Test_2xMCUs.brd (EAGLE design)
At the start: 120 x 145 mm, 80 parts, among them J1 10-pos, J13 4-pos, J4 10-pos, J8 10-pos, U1 RENESAS_R7FS5D37A3A01CFM#AA0P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, U2 S7G2LQFP176, U4 RENESAS_R7FS5D37A3A01CFM#AA0P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, X2 32.768KHz, X3 32.768KHz, X4 24MHz, X6 32.768KHz, Y1 XTAL_12MHZ_ABM8G-12.000MHZ-B4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, Y4 XTAL_12MHZ_ABM8G-12.000MHZ-B4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

Commit message: Update
Parts:
- removed C39, C72, C73: 12pF, 3D_MIG_Controller:0402
- removed C74, C75: 10pF, 3D_MIG_Controller:0402
- removed C76, C77, C78, C79, C80, C81, C82, C83, C84: 0.1uF, 3D_MIG_Controller:0402
- removed C85: 1uF, 3D_MIG_Controller:0402
- removed C86: 10uF, 3D_MIG_Controller:0402
- removed J7: (no value), 3D_MIG_Controller:2X5
- removed J8: 10-pos, 3D_MIG_Controller:2X5
- removed R7: 10K0, 3D_MIG_Controller:0402
- removed U4: RENESAS_R7FS5D37A3A01CFM#AA0PLQP0064KB-C_REN-M, 3D_MIG_Controller:PLQP0064KB-C_REN-M
- removed X6: 32.768KHz, 3D_MIG_Controller:SMD_X_2_PADS
- removed Y4: XTAL_12MHZ_ABM8G-12.000MHZ-B4Y-T, 3D_MIG_Controller:CRYSTAL_ABM8G_ABR
- added C203, C204: 12pF, 3D_MIG_Controller:0402
- added C205, C206: 10pF, 3D_MIG_Controller:0402
- added C207, C208, C209, C210, C211, C212, C213, C214, C215, C218, C58: 0.1uF, 3D_MIG_Controller:0402
- added C216: 1uF, 3D_MIG_Controller:0402
- added C217, C57: 10uF, 3D_MIG_Controller:0402
- added J24: (no value), 3D_MIG_Controller:2X5
- added J25: 10-pos, 3D_MIG_Controller:2X5
- added R16: 10K0, 3D_MIG_Controller:0402
- added U13: RENESAS_R7FS5D37A3A01CFM#AA0PLQP0064KB-C_REN-M, 3D_MIG_Controller:PLQP0064KB-C_REN-M
- added X14: 32.768KHz, 3D_MIG_Controller:SMD_X_2_PADS
- added Y12: XTAL_12MHZ_ABM8G-12.000MHZ-B4Y-T, 3D_MIG_Controller:CRYSTAL_ABM8G_ABR
- C41: value 10pF -> 12pF
- C43: value 0.1uF -> 10pF
- C55: value 1uF -> 0.1uF
- C56: value 10uF -> 1uF
- moved C49 30.9 mm to (31.3, 121.4), turned to 90 degrees
- moved C56 27.8 mm to (31.3, 124.8), turned to 90 degrees
- moved C54 22.5 mm to (31.3, 123.7), turned to 90 degrees
- moved C47 20.9 mm to (17.7, 112.8), turned to 0 degrees
- moved C43 18.1 mm to (14.9, 133.8), turned to 270 degrees
- moved C55 17.8 mm to (11.9, 122.5), turned to 180 degrees
- moved C50 17.4 mm to (6.25, 130.1), turned to 0 degrees
- moved C48 15.3 mm to (13.1, 126.8), turned to 180 degrees
- moved C51 14.3 mm to (25.3, 131.9), turned to 270 degrees
- moved C52 13.8 mm to (15.6, 132.4)
- moved C42 9.47 mm to (20.1, 133.6), turned to 90 degrees
- moved C40 7.57 mm to (25.3, 133.9), turned to 90 degrees
- moved C41 7.01 mm to (21.4, 132.6), turned to 270 degrees
- moved C53 6.37 mm to (31.3, 122.6)
- moved J3 6.12 mm to (23.3, 109.2)
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Connections:
- removed net DFO_01_A1: U1.30, U4.30
- removed net P400: U4.1
- removed net RELAY_4_A1: U1.31, U4.31
- new net 21/P207: U1.21, U13.21
- new net 4/VBATT: U1.4, U13.4
- new net N$19: C218.P$1, U13.40
- new net N$5: C58.P$1, U1.40
- new net N$69: U1.18, U13.18
- new net N$70: U1.19, U13.19
- new net N$82: U1.36, U13.36
- new net N$83: U1.37, U13.37
- net GND: now also C203.P$2, C204.P$2, C205.P$2, C206.P$2, C207.P$2, C208.P$2, C209.P$2, C210.P$2, C211.P$1, C212.P$1, C213.P$2, C214.P$2, C215.P$2, C216.P$2, C217.P$2, C218.P$2, C50.P$2, C52.P$1, C57.P$2, C58.P$2, J24.1, J24.2, J25.10, J25.6, J25.8, U13.17, U13.28, U13.39, U13.55, U13.58, U13.59, U13.8, Y12.2, Y12.4; no longer C39.P$2, C50.P$1, C52.P$2, C72.P$2, C73.P$2, C74.P$2, C75.P$2, C76.P$2, C77.P$2, C78.P$2, C79.P$2, C80.P$1, C81.P$1, C82.P$2, C83.P$2, C84.P$2, C85.P$2, C86.P$2, J7.1, J7.2, J8.10, J8.6, J8.8, U1.12, U1.13, U1.14, U1.15, U1.18, U1.19, U1.2, U1.21, U1.22, U1.23, U1.24, U1.26, U1.27, U1.3, U1.4, U1.40, U1.41, U1.42, U1.43, U1.44, U1.49, U1.50, U1.52, U1.53, U1.54, U1.61, U1.62, U1.63, U4.12, U4.13, U4.14, U4.15, U4.17, U4.18, U4.19, U4.2, U4.21, U4.22, U4.23, U4.24, U4.26, U4.27, U4.28, U4.3, U4.39, U4.4, U4.40, U4.41, U4.42, U4.43, U4.44, U4.49, U4.50, U4.52, U4.53, U4.54, U4.55, U4.58, U4.59, U4.61, U4.62, U4.63, U4.8, Y4.2, Y4.4
- net MISO: now also J24.10, J24.9, U13.48; no longer J7.10, J7.9, U4.48
- net MOSI: now also J24.7, J24.8, U13.47; no longer J7.7, J7.8, U4.47
- net RESET_A1: now also C217.P$1, C57.P$1, J25.9, R16.P$1, U13.25; no longer C56.P$1, C86.P$1, J8.9, R7.P$1, U4.25
- net SCLK: now also J24.5, J24.6, U13.46; no longer J7.5, J7.6, U4.46
- net SSL0_A1_06: now also J24.3, J24.4, U13.45; no longer J7.3, J7.4, U4.45
- net TCK: now also J25.7, U13.32; no longer J8.7, U4.32
- net TDI: now also J25.1, U13.35; no longer J8.1, U4.35
- net TDO: now also J25.3, U13.34; no longer J8.3, U4.34
- net TMS: now also J25.5, U13.33; no longer J8.5, U4.33
- net VCL0_A1: now also C211.P$2, C51.P$2, U13.5; no longer C50.P$2, C80.P$2, U4.5
- net VDD: now also C207.P$1, C208.P$1, C209.P$1, C210.P$1, C212.P$2, C213.P$1, C214.P$1, C215.P$1, C216.P$1, C50.P$1, C52.P$2, C56.P$1, J25.2, J25.4, R16.P$2, U13.11, U13.20, U13.29, U13.38, U13.51, U13.56, U13.57, U13.60; no longer C43.P$1, C51.P$2, C52.P$1, C76.P$1, C77.P$1, C78.P$1, C79.P$1, C81.P$2, C82.P$1, C83.P$1, C84.P$1, C85.P$1, J8.2, J8.4, R7.P$2, U4.11, U4.20, U4.29, U4.38, U4.51, U4.56, U4.57, U4.60
- net XCIN_A1: now also C203.P$1, C40.P$1, U13.6, X14.P$1; no longer C39.P$1, C72.P$1, U4.6, X6.P$1
- net XCOUT_A1: now also C204.P$1, C41.P$1, U13.7, X14.P$2; no longer C40.P$1, C73.P$1, U4.7, X6.P$2
- net XTAL1_A1: now also C205.P$1, C42.P$1, U13.9, Y12.3; no longer C41.P$1, C74.P$1, U4.9, Y4.3
- net XTAL2_A1: now also C206.P$1, C43.P$1, U13.10, Y12.1; no longer C42.P$1, C75.P$1, U4.10, Y4.1
Routing:
- net VDD: track 708.6 -> 825.1 mm, vias 33 -> 1
- net MISO: track 225.0 -> 233.4 mm
- net MOSI: track 216.7 -> 224.3 mm, vias 4 -> 2
- net SCLK: track 208.1 -> 214.9 mm, vias 4 -> 2
- net SSL0_A1_01: track 56.2 -> 49.8 mm, vias 2 -> 1
- net N$5: track 0.00 -> 4.18 mm
- net N$19: track 0.00 -> 3.94 mm
- net SSL0_A1_06: track 140.3 -> 144.2 mm, vias 2 -> 1
- net TDI: track 43.0 -> 42.0 mm
- net VCL_F(FLASH): track 5.46 -> 4.58 mm
- net GND: vias 0 -> 1
