File: SPI_Test/SPI_Test_2xMCUs.sch (EAGLE design)
At the start: 80 parts, among them J1 10-pos, J13 4-pos, J4 10-pos, J8 10-pos, U1 RENESAS_R7FS5D37A3A01CFM#AA0P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, U2 S7G2LQFP176, U4 RENESAS_R7FS5D37A3A01CFM#AA0P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, X2 32.768KHz, X3 32.768KHz, X4 24MHz, X6 32.768KHz, Y1 XTAL_12MHZ_ABM8G-12.000MHZ-B4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, Y4 XTAL_12MHZ_ABM8G-12.000MHZ-B4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

Commit message: Update
Parts:
- removed C39, C72, C73: 12pF, 3D_MIG_Controller:C_0402_12PF
- removed C74, C75: 10pF, 3D_MIG_Controller:C_0402_10PF
- removed C76, C77, C78, C79, C80, C81, C82, C83, C84: 0.1uF, 3D_MIG_Controller:C_0402_0.1UF
- removed C85: 1uF, 3D_MIG_Controller:C_0402_1UF
- removed C86: 10uF, 3D_MIG_Controller:C_0402_10UF
- removed J7: (no value), 3D_MIG_Controller:CONN_05X2PTH
- removed J8: 10-pos, 3D_MIG_Controller:CONN_05X2_RAPTH
- removed R7: 10K0, 3D_MIG_Controller:R_0402_10K0
- removed U4: RENESAS_R7FS5D37A3A01CFM#AA0PLQP0064KB-C_REN-M, 3D_MIG_Controller:RENESAS_R7FS5D37A3A01CFM#AA0PLQP0064KB-C_REN-M
- removed X6: 32.768KHz, 3D_MIG_Controller:XTAL_32.768KHZ
- removed Y4: XTAL_12MHZ_ABM8G-12.000MHZ-B4Y-T, 3D_MIG_Controller:XTAL_12MHZ_ABM8G-12.000MHZ-B4Y-T
- added C203, C204: 12pF, 3D_MIG_Controller:C_0402_12PF
- added C205, C206: 10pF, 3D_MIG_Controller:C_0402_10PF
- added C207, C208, C209, C210, C211, C212, C213, C214, C215, C218, C58: 0.1uF, 3D_MIG_Controller:C_0402_0.1UF
- added C216: 1uF, 3D_MIG_Controller:C_0402_1UF
- added C217, C57: 10uF, 3D_MIG_Controller:C_0402_10UF
- added J24: (no value), 3D_MIG_Controller:CONN_05X2PTH
- added J25: 10-pos, 3D_MIG_Controller:CONN_05X2_RAPTH
- added R16: 10K0, 3D_MIG_Controller:R_0402_10K0
- added U13: RENESAS_R7FS5D37A3A01CFM#AA0PLQP0064KB-C_REN-M, 3D_MIG_Controller:RENESAS_R7FS5D37A3A01CFM#AA0PLQP0064KB-C_REN-M
- added X14: 32.768KHz, 3D_MIG_Controller:XTAL_32.768KHZ
- added Y12: XTAL_12MHZ_ABM8G-12.000MHZ-B4Y-T, 3D_MIG_Controller:XTAL_12MHZ_ABM8G-12.000MHZ-B4Y-T
- C41: value 10pF -> 12pF; device 3D_MIG_Controller:C_0402_10PF -> 3D_MIG_Controller:C_0402_12PF
- C43: value 0.1uF -> 10pF; device 3D_MIG_Controller:C_0402_0.1UF -> 3D_MIG_Controller:C_0402_10PF
- C55: value 1uF -> 0.1uF; device 3D_MIG_Controller:C_0402_1UF -> 3D_MIG_Controller:C_0402_0.1UF
- C56: value 10uF -> 1uF; device 3D_MIG_Controller:C_0402_10UF -> 3D_MIG_Controller:C_0402_1UF
Connections:
- removed net DFO_01_A1: U1.30/P302, U4.30/P302
- removed net P400: U4.1/P400
- removed net RELAY_4_A1: U1.31/P301, U4.31/P301
- new net N$19: C218.1, U13.40/VCL
- new net N$5: C58.1, U1.40/VCL
- new net N$69: U1.18/USB_DM, U13.18/USB_DM
- new net N$70: U1.19/USB_DP, U13.19/USB_DP
- new net N$82: U1.36/P111, U13.36/P111
- new net N$83: U1.37/P112, U13.37/P112
- net GND: now also C203.2, C204.2, C205.2, C206.2, C207.2, C208.2, C209.2, C210.2, C211.1, C212.1, C213.2, C214.2, C215.2, C216.2, C217.2, C218.2, C50.2, C52.1, C57.2, C58.2, J24.1, J24.2, J25.10, J25.6, J25.8, U13.17/VSS_USB, U13.28/VSS, U13.39/VSS, U13.55/VREFL, U13.58/AVSS0, U13.59/VREFL0, U13.8/VSS, Y12.2, Y12.4; no longer C39.2, C50.1, C52.2, C72.2, C73.2, C74.2, C75.2, C76.2, C77.2, C78.2, C79.2, C80.1, C81.1, C82.2, C83.2, C84.2, C85.2, C86.2, J7.1, J7.2, J8.10, J8.6, J8.8, U1.12/P411, U1.13/P410, U1.14/P409, U1.15/P408, U1.18/USB_DM, U1.19/USB_DP, U1.2/P401, U1.21/P207, U1.22/P206, U1.23/P205, U1.24/P204, U1.26/P201/MD, U1.27/P200, U1.3/P402, U1.4/VBATT, U1.40/VCL, U1.41/P107, U1.42/P106, U1.43/P105, U1.44/P104, U1.49/P500, U1.50/P501, U1.52/VSS, U1.53/P015, U1.54/P014, U1.61/P003, U1.62/P002, U1.63/P001, U4.12/P411, U4.13/P410, U4.14/P409, U4.15/P408, U4.17/VSS_USB, U4.18/USB_DM, U4.19/USB_DP, U4.2/P401, U4.21/P207, U4.22/P206, U4.23/P205, U4.24/P204, U4.26/P201/MD, U4.27/P200, U4.28/VSS, U4.3/P402, U4.39/VSS, U4.4/VBATT, U4.40/VCL, U4.41/P107, U4.42/P106, U4.43/P105, U4.44/P104, U4.49/P500, U4.50/P501, U4.52/VSS, U4.53/P015, U4.54/P014, U4.55/VREFL, U4.58/AVSS0, U4.59/VREFL0, U4.61/P003, U4.62/P002, U4.63/P001, U4.8/VSS, Y4.2, Y4.4
- net MISO: now also J24.10, J24.9, U13.48/P100; no longer J7.10, J7.9, U4.48/P100
- net MOSI: now also J24.7, J24.8, U13.47/P101; no longer J7.7, J7.8, U4.47/P101
- net RESET_A1: now also C217.1, C57.1, J25.9, R16.1, U13.25/RES; no longer C56.1, C86.1, J8.9, R7.1, U4.25/RES
- net SCLK: now also J24.5, J24.6, U13.46/P102; no longer J7.5, J7.6, U4.46/P102
- net SSL0_A1_06: now also J24.3, J24.4, U13.45/P103; no longer J7.3, J7.4, U4.45/P103
- net TCK: now also J25.7, U13.32/P300/TCK/SWCLK; no longer J8.7, U4.32/P300/TCK/SWCLK
- net TDI: now also J25.1, U13.35/P110/TDI; no longer J8.1, U4.35/P110/TDI
- net TDO: now also J25.3, U13.34/P109/TDO/SWO; no longer J8.3, U4.34/P109/TDO/SWO
- net TMS: now also J25.5, U13.33/P108/TMS/SWDIO; no longer J8.5, U4.33/P108/TMS/SWDIO
- net VCL0_A1: now also C211.2, C51.2, U13.5/VCL0; no longer C50.2, C80.2, U4.5/VCL0
- net VDD: now also C207.1, C208.1, C209.1, C210.1, C212.2, C213.1, C214.1, C215.1, C216.1, C50.1, C52.2, C56.1, J25.2, J25.4, R16.2, U13.11/VCC, U13.20/VCC_USB, U13.29/VCC, U13.38/VCC, U13.51/VCC, U13.56/VREFH, U13.57/AVCC0, U13.60/VREFH0; no longer C43.1, C51.2, C52.1, C76.1, C77.1, C78.1, C79.1, C81.2, C82.1, C83.1, C84.1, C85.1, J8.2, J8.4, R7.2, U4.11/VCC, U4.20/VCC_USB, U4.29/VCC, U4.38/VCC, U4.51/VCC, U4.56/VREFH, U4.57/AVCC0, U4.60/VREFH0
- net XCIN_A1: now also C203.1, C40.1, U13.6/XCIN, X14.P$1; no longer C39.1, C72.1, U4.6/XCIN, X6.P$1
- net XCOUT_A1: now also C204.1, C41.1, U13.7/XCOUT, X14.P$2; no longer C40.1, C73.1, U4.7/XCOUT, X6.P$2
- net XTAL1_A1: now also C205.1, C42.1, U13.9/XTAL, Y12.3; no longer C41.1, C74.1, U4.9/XTAL, Y4.3
- net XTAL2_A1: now also C206.1, C43.1, U13.10/EXTAL, Y12.1; no longer C42.1, C75.1, U4.10/EXTAL, Y4.1
Other:
- moved on the sheet: C40, C41, C42, C43, C47, C48, C49, C50, C51, C52, C53, C54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
