File: Crutch_Light/Crutch_Light_v1p01.sch (EAGLE design)
At the start: 7 parts, among them J2 2-pos

Commit message: update
Parts:
- removed J2: 2-pos, 3D_MIG_Controller:3.81MM_1_X_2_RT_ANGLE_PLUG_HEADER
- added B1: BH-25C-1, 3D_MIG_Controller:BH-25C-1
- added J1: (no value), 3D_MIG_Controller:CONN_530470310_PICOBLADE_X_3
Connections:
- new net N$4: B1.2, J1.2
- net GND: now also B1.1; no longer J2.P$1
- net VDD: now also J1.1, J1.3; no longer J2.P$2
Changed lines of the file:
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@@
 <part name="LED3" library="3D_MIG_Controller" deviceset="LED_0805_GREEN" device="" value="Green"/>
 <part name="R3" library="3D_MIG_Controller" deviceset="R_0402_1K0" device="" value="1K0"/>
-<part name="J2" library="3D_MIG_Controller" deviceset="3.81MM_1_X_2_RT_ANGLE_PLUG_HEADER" device="" value="2-pos"/>
+<part name="B1" library="3D_MIG_Controller" deviceset="BH-25C-1" device=""/>
+<part name="J1" library="3D_MIG_Controller" deviceset="CONN_530470310_PICOBLADE_X_3" device=""/>
 </parts>
 <sheets>
@@
 <attribute name="VALUE" x="84.582" y="57.15" size="1.778" layer="96" rot="R90"/>
 </instance>
-<instance part="J2" gate="A" x="106.68" y="66.04" smashed="yes">
-<attribute name="NAME" x="100.076" y="74.168" size="1.778" layer="125"/>
+<instance part="B1" gate="A" x="144.78" y="60.96" smashed="yes">
+<attribute name="NAME" x="141.7066" y="63.0428" size="3.4798" layer="95" ratio="10" rot="SR0"/>
+<attribute name="VALUE" x="140.6398" y="55.4228" size="3.4798" layer="96" ratio="10" rot="SR0"/>
+</instance>
+<instance part="J1" gate="A" x="119.38" y="66.04" smashed="yes" rot="R270">
+<attribute name="NAME" x="124.6886" y="61.8744" size="2.0828" layer="95" ratio="6" rot="SR270"/>
 </instance>
 </instances>
@@
 <segment>
 <pinref part="R2" gate="G$1" pin="2"/>
-<pinref part="J2" gate="A" pin="P$2"/>
 <wire x1="50.8" y1="66.04" x2="50.8" y2="71.12" width="0.1524" layer="91"/>
 <wire x1="50.8" y1="71.12" x2="66.04" y2="71.12" width="0.1524" layer="91"/>
 <pinref part="R1" gate="G$1" pin="2"/>
 <wire x1="66.04" y1="71.12" x2="81.28" y2="71.12" width="0.1524" layer="91"/>
-<wire x1="81.28" y1="71.12" x2="101.6" y2="71.12" width="0.1524" layer="91"/>
 <wire x1="66.04" y1="66.04" x2="66.04" y2="71.12" width="0.1524" layer="91"/>
 <junction x="66.04" y="71.12"/>
 <pinref part="R3" gate="G$1" pin="2"/>
 <wire x1="81.28" y1="66.04" x2="81.28" y2="71.12" width="0.1524" layer="91"/>
+<label x="50.8" y="71.12" size="1.016" layer="95" rot="R180" xref="yes"/>
+<pinref part="J1" gate="A" pin="3"/>
+<wire x1="114.3" y1="66.04" x2="114.3" y2="71.12" width="0.1524" layer="91"/>
+<wire x1="114.3" y1="71.12" x2="81.28" y2="71.12" width="0.1524" layer="91"/>
 <junction x="81.28" y="71.12"/>
-<label x="50.8" y="71.12" size="1.016" layer="95" rot="R180" xref="yes"/>
+<pinref part="J1" gate="A" pin="1"/>
+<wire x1="119.38" y1="66.04" x2="119.38" y2="71.12" width="0.1524" layer="91"/>
+<wire x1="119.38" y1="71.12" x2="114.3" y2="71.12" width="0.1524" layer="91"/>
+<junction x="114.3" y="71.12"/>
 </segment>
 </net>
@@
 <wire x1="50.8" y1="38.1" x2="66.04" y2="38.1" width="0.1524" layer="91"/>
 <wire x1="66.04" y1="38.1" x2="81.28" y2="38.1" width="0.1524" layer="91"/>
-<wire x1="81.28" y1="38.1" x2="93.98" y2="38.1" width="0.1524" layer="91"/>
-<wire x1="93.98" y1="38.1" x2="93.98" y2="66.04" width="0.1524" layer="91"/>
-<pinref part="J2" gate="A" pin="P$1"/>
-<wire x1="93.98" y1="66.04" x2="101.6" y2="66.04" width="0.1524" layer="91"/>
 <pinref part="LED2" gate="G$1" pin="C"/>
 <wire x1="66.04" y1="45.72" x2="66.04" y2="38.1" width="0.1524" layer="91"/>
@@
 <junction x="81.28" y="38.1"/>
 <label x="50.8" y="38.1" size="1.016" layer="95" rot="R180" xref="yes"/>
+<pinref part="B1" gate="A" pin="1"/>
+<wire x1="154.94" y1="60.96" x2="160.02" y2="60.96" width="0.1524" layer="91"/>
+<wire x1="160.02" y1="60.96" x2="160.02" y2="38.1" width="0.1524" layer="91"/>
+<wire x1="160.02" y1="38.1" x2="81.28" y2="38.1" width="0.1524" layer="91"/>
 </segment>
 </net>
+<net name="N$4" class="0">
+<segment>
+<pinref part="J1" gate="A" pin="2"/>
+<wire x1="116.84" y1="66.04" x2="116.84" y2="73.66" width="0.1524" layer="91"/>
+<wire x1="116.84" y1="73.66" x2="137.16" y2="73.66" width="0.1524" layer="91"/>
+<pinref part="B1" gate="A" pin="2"/>
+<wire x1="137.16" y1="73.66" x2="137.16" y2="60.96" width="0.1524" layer="91"/>
+<wire x1="137.16" y1="60.96" x2="144.78" y2="60.96" width="0.1524" layer="91"/>
+</segment>
+</net>
