File: Flight Mill Controller/Flight-Mill-Controller.brd (EAGLE design)
At the start: 160 x 100 mm, 49 parts, among them IC1 STM32G0B1RET6, IC2 CSTNE8M00G520000R0, IC3 MCP6001UT, J1 1050170001, J2 61300411121, Q1 BC817, X1 B2B-XH-AM(LF)(SN), X2 B2B-XH-AM(LF)(SN), X3 WF2549-2WS05S0B01, X4 MICROMATCH-16, X6 282834-2

Commit message: Changes on going
Parts:
- added C10, C11, C12, C13, C14, C15: 100nF/50V, Labops_Lib_AH:EIA0603
- added D1: SS14, Labops_Lib_AH:SMA
- added D14: MMBZ4696-HE3-18, Labops_Lib_AH:SOT23-3
- added IC4, IC5, IC6: LMV641, Labops_Lib_AH:SOT-23-5
- added Q2: UT2955G-AA3-R, Labops_Lib_AH:SOT223
- added Q3: 2N7002, Labops_Lib_AH:SOT23
- added R26, R27, R28, R30, R31, R32, R33, R34, R37, R38, R39: 10K 1%, 3D_MIG_Controller:0603
- added R29, R35, R36, R41, R43: 100R 1%, 3D_MIG_Controller:0603
- added R40, R42: 1.5K 1%, 3D_MIG_Controller:0603
- added R44: 0R 1%, 3D_MIG_Controller:0603
- added X5, X7: 726386-2TE_726386-2, Labops_Lib_AH:TE_726386-2
Connections:
- new net AIR_PUMP+: D1.1, Q2.2, Q2.4, R30.2, X5.1, X5.1-2
- new net AI_O2_SENSOR: IC5.1, R37.1, R38.1, R38.2, R39.1, R40.1, R44.1
- new net DO_V_AIR_PUMP_ON: R29.2
- new net N$12: Q3.1, R28.2, R29.1
- new net N$14: IC5.4, R35.1, R37.2
- new net N$15: C13.2, R40.2, R41.1
- new net N$16: C11.2, R33.1, R34.2
- new net N$17: IC4.4, R33.2
- new net N$18: IC6.3, R41.2
- new net N$19: IC5.3, R36.1
- new net N$2: D14.1, Q2.1, R26.1, R27.2
- new net N$20: IC6.4, R43.2
- new net N$21: C14.1, R42.2, R43.1
- new net N$22: IC6.1, R44.2
- new net N$9: Q3.3, R27.1
- new net O2_SENSOR_C: C11.1, IC4.1
- new net O2_SENSOR_R: R34.1
- new net O2_SENSOR_S: R35.2
- new net VREF_O2: IC4.3, R31.2, R32.1, R36.2, R42.1
- new net V_12V0: D14.3, Q2.3, R26.2
- net GND: now also C10.2, C12.2, C13.1, C14.2, C15.2, D1.2, IC4.2, IC5.2, IC6.2, Q3.2, R28.1, R30.1, R31.1, R39.2, X7.1, X7.1-2
- net V5V0: now also C10.1, C12.1, C15.1, IC4.5, IC5.5, IC6.5, R32.2
