File: Organic Crystals Driver/Crystal_Driver.sch (EAGLE design)
At the start: 22 parts, among them T1 SIHG039N60EF2, T2 SIHG039N60EF2, X1 726386-2TE_726386-2, X2 726386-2TE_726386-2, X3 2304-6111-TP, X4 726386-2TE_726386-2, X5 726386-2TE_726386-2, X6 2304-6111-TP

Commit message: HW01.01 Ongoing
After Test Modifications..
Parts:
- R1, R3: value 470R 1% -> 220R 1%
Changed lines of the file:
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@@
 <part name="T1" library="Labops_Lib_AH" deviceset="SIHG039N60EF" device="2"/>
 <part name="GND1" library="Labops_Lib_AH" deviceset="GND" device=""/>
-<part name="R1" library="Labops_Lib_AH" deviceset="R_1206" device="EIA1206" value="470R 1%"/>
+<part name="R1" library="Labops_Lib_AH" deviceset="R_1206" device="EIA1206" value="220R 1%"/>
 <part name="R2" library="Labops_Lib_AH" deviceset="R_0603" device="" value="1K 1%"/>
 <part name="D1" library="Labops_Lib_AH" deviceset="FEP30DP-E3/45" device="TO-247AD"/>
@@
 <part name="T2" library="Labops_Lib_AH" deviceset="SIHG039N60EF" device="2"/>
 <part name="GND2" library="Labops_Lib_AH" deviceset="GND" device=""/>
-<part name="R3" library="Labops_Lib_AH" deviceset="R_1206" device="EIA1206" value="470R 1%"/>
+<part name="R3" library="Labops_Lib_AH" deviceset="R_1206" device="EIA1206" value="220R 1%"/>
 <part name="R4" library="Labops_Lib_AH" deviceset="R_0603" device="" value="1K 1%"/>
 <part name="D2" library="Labops_Lib_AH" deviceset="FEP30DP-E3/45" device="TO-247AD"/>
