File: Flight Mill Controller/Flight-Mill-AC/Flight-Mill-Controller.brd (EAGLE design)
At the start: 121.9 x 120 mm, 212 parts, among them IC1 STM32G0B1RET6, IC10 SN65HVD3082EDR, IC2 CSTNE8M00G520000R0, IC3 MCP6001UT, IC4 LMV641, IC5 LMV641, IC6 LMV641, IC7 LMV641, IC8 LMV641, IC9 LMV641, J1 1050170001, J2 61300411121, J3 615008148521, J4 61300411121, K1 RYA31012, K2 RYA31012, Q1 BC817, Q2 UT2955G-AA3-R, Q3 2N7002, Q4 UT2955G-AA3-R, Q5 2N7002, Q6 UT2955G-AA3-R, Q7 2N7002, Q8 UT2955G-AA3-R, Q9 2N7002, X1 B2B-XH-AM(LF)(SN), X10 MOLEX_206832-0601MOLEX_206832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, X11 726386-2TE_726386-2, X12 726386-2TE_726386-2, X13 726386-2TE_726386-2, X14 726386-2TE_726386-2, X15 726386-2TE_726386-2, X16 726386-2TE_726386-2, X17 282834-3, X18 282834-3, X19 726386-2TE_726386-2, X2 B2B-XH-AM(LF)(SN), X20 726386-2TE_726386-2, X21 726386-2TE_726386-2, X22 726386-2TE_726386-2, X23 282834-2, X24 282834-3, X3 WF2549-2WS05S0B01, X4 282834-2, X5 726386-2TE_726386-2, X6 282834-2, X7 726386-2TE_726386-2, X8 5-102203-3, X9 5-102203-3

Commit message: HW01.01 changes
Parts:
- removed IC3: MCP6001UT, Labops_Lib_AH:SOT-23-5
- R12: value 1K 1% -> n.P
- R14: value 47K 1% -> 0R 1%
Connections:
- net GND: no longer IC3.2
- net N$10: no longer IC3.4
- net N$6: no longer IC3.1
- net N$8: no longer IC3.3
- net V3V3: no longer IC3.5
Routing:
- net N$6: track 24.5 -> 17.7 mm
- net N$10: track 13.9 -> 11.0 mm
- net V3V3: track 335.3 -> 333.1 mm
- net N$8: track 5.16 -> 4.06 mm
