File: Flight Mill Controller/Flight-Mill-AC/Flight-Mill-Controller.sch (EAGLE design)
At the start: 212 parts, among them IC1 STM32G0B1RET6, IC10 SN65HVD3082EDR, IC2 CSTNE8M00G520000R0, IC3 MCP6001UT, IC4 LMV641, IC5 LMV641, IC6 LMV641, IC7 LMV641, IC8 LMV641, IC9 LMV641, J1 1050170001, J2 61300411121, J3 615008148521, J4 61300411121, K1 RYA31012, K2 RYA31012, Q1 BC817, Q2 UT2955G-AA3-R, Q3 2N7002, Q4 UT2955G-AA3-R, Q5 2N7002, Q6 UT2955G-AA3-R, Q7 2N7002, Q8 UT2955G-AA3-R, Q9 2N7002, X1 B2B-XH-AM(LF)(SN), X10 MOLEX_206832-0601MOLEX_206832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, X11 726386-2TE_726386-2, X12 726386-2TE_726386-2, X13 726386-2TE_726386-2, X14 726386-2TE_726386-2, X15 726386-2TE_726386-2, X16 726386-2TE_726386-2, X17 282834-3, X18 282834-3, X19 726386-2TE_726386-2, X2 B2B-XH-AM(LF)(SN), X20 726386-2TE_726386-2, X21 726386-2TE_726386-2, X22 726386-2TE_726386-2, X23 282834-2, X24 282834-3, X3 WF2549-2WS05S0B01, X4 282834-2, X5 726386-2TE_726386-2, X6 282834-2, X7 726386-2TE_726386-2, X8 5-102203-3, X9 5-102203-3

Commit message: HW01.01 changes
Parts:
- removed IC3: MCP6001UT, Labops_Lib_AH:MCP6001UT
- R12: value 1K 1% -> n.P
- R14: value 47K 1% -> 0R 1%
Connections:
- net GND: no longer IC3.NULL@2
- net N$10: no longer IC3.NULL@4
- net N$6: no longer IC3.NULL@1
- net N$8: no longer IC3.NULL@3
- net V3V3: no longer IC3.NULL@5
Changed lines of the file:
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@@
 <part name="X1" library="Labops_Lib_AH" deviceset="B2B-XH-AM(LF)(SN)" device=""/>
 <part name="X2" library="Labops_Lib_AH" deviceset="B2B-XH-AM(LF)(SN)" device=""/>
-<part name="IC3" library="Labops_Lib_AH" deviceset="MCP6001UT" device=""/>
 <part name="R7" library="Labops_Lib_AH" deviceset="R_0603" device="" value="47K 1%"/>
 <part name="R8" library="Labops_Lib_AH" deviceset="R_0603" device="" value="47K 1%"/>
@@
 <part name="R11" library="Labops_Lib_AH" deviceset="R_0603" device="" value="10K 1%"/>
 <part name="GND7" library="Labops_Lib_AH" deviceset="GND" device=""/>
-<part name="R12" library="Labops_Lib_AH" deviceset="R_0603" device="" value="1K 1%"/>
+<part name="R12" library="Labops_Lib_AH" deviceset="R_0603" device="" value="n.P"/>
 <part name="GND8" library="Labops_Lib_AH" deviceset="GND" device=""/>
 <part name="R13" library="Labops_Lib_AH" deviceset="R_0603" device="" value="n.p"/>
-<part name="GND9" library="Labops_Lib_AH" deviceset="GND" device=""/>
 <part name="C3" library="Labops_Lib_AH" deviceset="C_0603" device="EIA0603" value="100nF/50V"/>
 <part name="GND10" library="Labops_Lib_AH" deviceset="GND" device=""/>
-<part name="R14" library="Labops_Lib_AH" deviceset="R_0603" device="" value="47K 1%"/>
+<part name="R14" library="Labops_Lib_AH" deviceset="R_0603" device="" value="0R 1%"/>
 <part name="R15" library="Labops_Lib_AH" deviceset="R_0603" device="" value="100R 1%"/>
 <part name="X3" library="Labops_Lib_AH" deviceset="WF2549-2WS05S0B01" device=""/>
@@
 <attribute name="VALUE" x="207.518" y="64.77" size="1.778" layer="96" rot="R270"/>
 </instance>
-<instance part="IC3" gate="G$1" x="299.72" y="187.96" smashed="yes">
-<attribute name="NAME" x="310.388" y="193.294" size="1.27" layer="95"/>
-<attribute name="VALUE" x="310.388" y="190.754" size="1.27" layer="96"/>
-</instance>
 <instance part="R7" gate="G$1" x="274.32" y="190.5" smashed="yes">
 <attribute name="NAME" x="270.51" y="191.9986" size="1.778" layer="95"/>
@@
 <attribute name="VALUE" x="270.51" y="215.138" size="1.778" layer="96"/>
 </instance>
-<instance part="GND9" gate="1" x="299.72" y="175.26" smashed="yes"/>
 <instance part="C3" gate="G$1" x="304.8" y="203.2" smashed="yes" rot="R90">
 <attribute name="NAME" x="308.356" y="211.455" size="1.778" layer="95"/>
@@
 </segment>
 <segment>
-<pinref part="GND9" gate="1" pin="GND"/>
-<pinref part="IC3" gate="G$1" pin="NULL@2"/>
-<wire x1="299.72" y1="177.8" x2="299.72" y2="180.34" width="0.1524" layer="91"/>
-</segment>
-<segment>
 <pinref part="C3" gate="G$1" pin="2"/>
 <wire x1="308.356" y1="203.2" x2="312.42" y2="203.2" width="0.1524" layer="91"/>
@@
 <pinref part="R7" gate="G$1" pin="2"/>
 <wire x1="279.4" y1="180.34" x2="279.4" y2="190.5" width="0.1524" layer="91"/>
-<pinref part="IC3" gate="G$1" pin="NULL@1"/>
 <wire x1="279.4" y1="190.5" x2="281.94" y2="190.5" width="0.1524" layer="91"/>
 <junction x="279.4" y="190.5"/>
 <pinref part="R13" gate="G$1" pin="2"/>
-<wire x1="281.94" y1="190.5" x2="292.1" y2="190.5" width="0.1524" layer="91"/>
 <wire x1="279.4" y1="218.44" x2="281.94" y2="218.44" width="0.1524" layer="91"/>
 <wire x1="281.94" y1="218.44" x2="281.94" y2="190.5" width="0.1524" layer="91"/>
-<junction x="281.94" y="190.5"/>
 <pinref part="R14" gate="G$1" pin="1"/>
 <wire x1="292.1" y1="218.44" x2="281.94" y2="218.44" width="0.1524" layer="91"/>
@@
 <pinref part="R10" gate="G$1" pin="1"/>
 <wire x1="289.56" y1="157.48" x2="284.48" y2="157.48" width="0.1524" layer="91"/>
-<pinref part="IC3" gate="G$1" pin="NULL@3"/>
-<wire x1="292.1" y1="185.42" x2="289.56" y2="185.42" width="0.1524" layer="91"/>
-<wire x1="289.56" y1="185.42" x2="289.56" y2="157.48" width="0.1524" layer="91"/>
-<junction x="289.56" y="157.48"/>
 </segment>
 </net>
@@
 </segment>
 <segment>
-<pinref part="IC3" gate="G$1" pin="NULL@5"/>
-<wire x1="299.72" y1="195.58" x2="299.72" y2="203.2" width="0.1524" layer="91"/>
-<wire x1="299.72" y1="203.2" x2="294.64" y2="203.2" width="0.1524" layer="91"/>
+<wire x1="302.26" y1="203.2" x2="294.64" y2="203.2" width="0.1524" layer="91"/>
 <label x="294.64" y="203.2" size="1.778" layer="95" rot="R180" xref="yes"/>
 <pinref part="C3" gate="G$1" pin="1"/>
-<wire x1="299.72" y1="203.2" x2="302.26" y2="203.2" width="0.1524" layer="91"/>
-<junction x="299.72" y="203.2"/>
 </segment>
 <segment>
@@
 <wire x1="302.26" y1="218.44" x2="320.04" y2="218.44" width="0.1524" layer="91"/>
 <wire x1="320.04" y1="218.44" x2="320.04" y2="187.96" width="0.1524" layer="91"/>
-<pinref part="IC3" gate="G$1" pin="NULL@4"/>
-<wire x1="320.04" y1="187.96" x2="309.88" y2="187.96" width="0.1524" layer="91"/>
 <pinref part="R15" gate="G$1" pin="2"/>
 <wire x1="322.58" y1="187.96" x2="320.04" y2="187.96" width="0.1524" layer="91"/>
-<junction x="320.04" y="187.96"/>
-</segment>
-</net>
+</segment>
+</net>
